File: pic32mk.brd (EAGLE design)
At the start: 100 x 80 mm, 39 parts, among them IC1 PIC32MK1024MCF100-I_PT, IC2 ADM3095EBRZ, IC3 MC33931EK, IC4 MAX203ECWP, IC5 MC33931EK, IC6 TXB0101DCKR, IC7 TXB0101DCKR, IC8 TXB0101DCKR, X1 22-23-2101

Commit message: up
Parts:
- added C14, C15, C16, C17, C18, C19: 0.1, rcl:C0805
- added IC9: TXB0101DCKR, TXB0101DCKR:SOT65P210X110-6N
- added J1: 1-1586043-4, 1-1586043-4:TE_1-1586043-4
- added U1, U2: PMIC-MC33932VW(SOP44), PMIC-MC33932VW_SOP44_:SOP44-0.65-15.8X10.9MM
- IC3, IC5: value MC33931EK -> TXB0101DCKR; device MC33931EK:SOP65P1030X245-33N -> TXB0101DCKR:SOT65P210X110-6N
- moved IC3 72.0 mm to (15.2, 55.9)
- moved IC5 71.1 mm to (15.2, 61.0)
- moved L1 51.8 mm to (34.3, 12.7), turned to 180 degrees
- moved U$1 31.1 mm to (44.5, 39.4)
- moved IC4 30.2 mm to (61.0, 39.4)
- moved C7 17.0 mm to (88.9, 10.2), turned to 270 degrees
- moved C4 6.48 mm to (81.3, 20.3)
- moved C3 3.81 mm to (81.3, 17.8)
- turned C9 to 90 degrees
- turned R3 to 270 degrees
Connections:
- new net +24V: C18.1, C19.1, J1.14, U1.17, U1.18, U1.26, U1.27, U1.28, U1.39, U1.4, U1.40, U1.5, U1.6, U2.17, U2.18, U2.26, U2.27, U2.28, U2.39, U2.4, U2.40, U2.5, U2.6
- new net N$15: IC9.3, X1.6
- new net N$5: IC3.3, X1.4
- new net N$8: IC5.3, X1.5
- net +5V: now also C15.1, C17.1, IC3.6, IC5.6, IC9.6, J1.3, X1.7
- net RE8: now also IC3.5, IC5.5, IC9.5
- net VDD: now also C14.1, C16.1, IC3.1, IC5.1, IC9.1, J1.2
- net VSS: now also C14.2, C15.2, C16.2, C17.2, C18.2, C19.2, IC3.2, IC5.2, IC9.2, J1.1, J1.13, U1.10, U1.11, U1.12, U1.13, U1.32, U1.33, U1.34, U1.35, U2.10, U2.11, U2.12, U2.13, U2.32, U2.33, U2.34, U2.35, X1.10; no longer IC3.15, IC3.16, IC3.17, IC3.18, IC5.15, IC5.16, IC5.17, IC5.18
Routing:
- net +24V: track 0.00 -> 101.7 mm
- net VDD: track 220.9 -> 284.2 mm
- net N$6: track 69.1 -> 26.0 mm, vias 3 -> 0
- net +5V: track 126.9 -> 164.5 mm, vias 2 -> 1
- net VCC: track 83.4 -> 61.2 mm
- net RE8: track 44.3 -> 60.1 mm
- net N$15: track 0.00 -> 12.5 mm, vias 0 -> 1
- net +3V3: track 79.2 -> 68.2 mm
- net N$8: track 0.00 -> 10.4 mm, vias 0 -> 1
- net N$5: track 0.00 -> 9.73 mm, vias 0 -> 1
- net N$13: track 24.4 -> 33.3 mm
- net RPA0: track 22.3 -> 31.0 mm
- net N$14: track 17.0 -> 25.4 mm
- net RPA14: track 35.0 -> 26.6 mm
- net N$2: track 32.5 -> 36.5 mm
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
Commit message: up
Parts:
- moved IC8 7.62 mm to (15.2, 47.0)
- moved IC9 6.35 mm to (15.2, 59.7)
- moved IC6 5.08 mm to (15.2, 49.5)
- moved IC5 3.81 mm to (15.2, 57.1)
- moved C17 2.54 mm to (21.6, 62.2)
- moved IC3 1.27 mm to (15.2, 54.6)
- moved IC7 1.27 mm to (15.2, 52.1)
Connections:
- new net RPB1: IC1.25, IC3.4
- new net RPC1: IC1.33, IC5.4
- new net RPC10: IC1.71, IC9.4
Routing:
- net RPB1: track 0.00 -> 53.2 mm, vias 0 -> 2
- net RPC1: track 0.00 -> 48.8 mm, vias 0 -> 2
- net RPC10: track 0.00 -> 40.6 mm, vias 0 -> 2
- net RE8: track 60.1 -> 86.4 mm
- net N$6: track 26.0 -> 13.0 mm
- net VDD: track 284.2 -> 294.0 mm, vias 0 -> 5
- net N$13: track 33.3 -> 23.9 mm
- net RPB6: track 31.4 -> 38.5 mm
- net RPA14: track 26.6 -> 33.6 mm
- net +5V: track 164.5 -> 170.0 mm, vias 1 -> 6
- net N$15: track 12.5 -> 8.92 mm
- net VCC: track 61.2 -> 58.5 mm
- net N$10: track 11.1 -> 8.90 mm
- net N$8: track 10.4 -> 8.84 mm, vias 1 -> 0
- net N$11: track 9.98 -> 8.84 mm, vias 1 -> 0
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
Commit message: up
Parts:
- added C20, C21: 0.1, rcl:C0805
- added X3: 22-23-2101, con-molex:22-23-2101
- moved S3 75.6 mm to (11.4, 74.9)
- moved U$2 73.3 mm to (21.6, 72.4)
- moved U$1 30.0 mm to (62.2, 15.2), turned to 0 degrees
- moved IC4 11.4 mm to (66.0, 29.2), turned to 0 degrees
Connections:
- new net N$17: U$1.IN2, X3.2
- new net N$18: U$1.IN3, X3.3
- new net N$19: U$1.IN4, X3.4
- new net N$20: U$1.IN5, X3.5
- new net N$21: U$1.IN6, X3.6
- new net N$22: U$1.IN7, X3.7
- new net N$23: U$1.IN8, X3.8
- new net N$24: U2.7, U2.8, U2.9
- new net N$25: U2.36, U2.37, U2.38
- new net N$26: U2.14, U2.15, U2.16
- new net N$27: U2.29, U2.30, U2.31
- new net N$4: U$1.IN1, X3.1
- new net RD8: IC1.68, U$1.EN_L
- new net RPB7: IC1.72, U$1.CH_L
- new net U1O1: J1.12, U1.7, U1.8, U1.9
- new net U1O2: J1.11, U1.36, U1.37, U1.38
- new net U1O3: J1.10, U1.29, U1.30, U1.31
- new net U1O4: J1.9, U1.14, U1.15, U1.16
- net +24V: now also C20.1, C21.1
- net +5V: now also X3.10
- net VSS: now also C20.2, C21.2, X3.9
Routing:
- net U1O3: track 0.00 -> 54.9 mm
- net U1O2: track 0.00 -> 44.2 mm, vias 0 -> 1
- net U1O4: track 0.00 -> 38.8 mm
- net RPB7: track 0.00 -> 35.1 mm, vias 0 -> 2
- net RD8: track 0.00 -> 31.0 mm, vias 0 -> 2
- net U1O1: track 0.00 -> 28.4 mm
- net VCC: track 58.5 -> 32.2 mm, vias 0 -> 2
- net +5V: track 170.0 -> 193.5 mm, vias 6 -> 2
- net +24V: track 101.7 -> 119.8 mm
- net N$4: track 0.00 -> 16.1 mm
- net N$17: track 0.00 -> 14.2 mm
- net N$6: track 13.0 -> 26.0 mm
- net N$18: track 0.00 -> 12.4 mm
- net N$19: track 0.00 -> 10.4 mm
- net N$20: track 0.00 -> 8.55 mm
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
Commit message: up
Parts:
- added R10: 1k, rcl:M0805
- added R4, R7, R8, R9: 100, rcl:R0805
- turned C21 to 180 degrees
- turned U1 to 0 degrees
- turned U2 to 0 degrees
Connections:
- new net N$28: R4.2, U2.2
- new net N$29: R7.1, U2.24
- new net N$30: R9.2, U1.2
- new net N$31: R8.1, U1.24
- new net N$32: R10.2, S1.5
- new net PWM1H: IC1.4, U1.43
- new net PWM1L: IC1.5, U1.42
- new net PWM2H: IC1.98, U1.21
- new net PWM2L: IC1.99, U1.20
- new net RPG9: IC1.14, R10.1
- net VSS: now also R4.1, R7.2, R8.2, R9.1, S1.6, U1.EH@1, U1.EH@2, U1.EH@3, U2.EH@1, U2.EH@2, U2.EH@3
Routing:
- net PWM2H: track 0.00 -> 92.8 mm, vias 0 -> 2
- net PWM2L: track 0.00 -> 83.9 mm
- net PWM1H: track 0.00 -> 69.3 mm, vias 0 -> 2
- net PWM1L: track 0.00 -> 68.3 mm, vias 0 -> 4
- net RPG9: track 0.00 -> 24.0 mm, vias 0 -> 2
- net +24V: track 119.8 -> 135.4 mm, vias 0 -> 1
- net +5V: track 193.5 -> 208.9 mm, vias 2 -> 3
- net N$6: track 26.0 -> 13.1 mm, vias 0 -> 2
- net N$32: track 0.00 -> 11.7 mm, vias 0 -> 1
- net U1O4: track 38.8 -> 49.7 mm, vias 0 -> 1
- net U1O1: track 28.4 -> 38.8 mm
- net U1O3: track 54.9 -> 44.7 mm
- net U1O2: track 44.2 -> 34.5 mm, vias 1 -> 0
- net RPB1: track 52.7 -> 43.8 mm
- net N$30: track 0.00 -> 6.84 mm
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- added copper zone on layer 16, net VSS

Commit message: up
Parts:
- added C22, C23, C24, C25: 0.1, rcl:C0805
- added C26, C27: 22uf, rcl:C0805
- added LED1: led1, led:CHIPLED_1206
- added LED2: led2, led:CHIPLED_1206
- added LED3: led3, led:CHIPLED_1206
- added R11, R12, R13: 1k, rcl:M0805
- added TP2, TP3, TP5, TP6: TPB1,27, testpad:B1,27
- moved U$1 17.8 mm to (44.5, 15.2)
- moved C12 13.7 mm to (47.0, 31.8), turned to 180 degrees
- moved C2 12.5 mm to (39.4, 33.0), turned to 180 degrees
- moved OS2 6.48 mm to (39.4, 29.2)
- moved OS1 6.35 mm to (47.0, 26.7)
Connections:
- new net DERE: IC1.74, IC2.5, IC2.6
- new net IN1: IC1.47, U$1.OUT1
- new net IN2: IC1.48, U$1.OUT2
- new net IN3: IC1.49, U$1.OUT3
- new net IN4: IC1.50, U$1.OUT4
- new net IN5: IC1.61, U$1.OUT5
- new net N$33: IC1.95, R11.2
- new net N$34: IC1.96, R12.2
- new net N$35: IC1.97, R13.2
- new net N$36: LED1.A, R11.1
- new net N$37: LED2.A, R12.1
- new net N$38: LED3.A, R13.1
- new net N$39: IC2.14, TP5.TP
- new net N$40: IC2.11, TP6.TP
- new net N$41: IC4.10, IC4.17
- new net N$42: IC4.11, IC4.16
- new net N$43: IC4.12, IC4.15
- new net N$44: IC4.5, TP2.TP
- new net N$45: IC4.4, TP3.TP
- new net PWM3H: IC1.93, U2.43
- new net PWM3L: IC1.94, U2.42
- new net PWM4H: IC1.100, U2.21
- new net PWM4L: IC1.3, U2.20
- new net RPE0: IC1.52, U1.25, U1.3
- new net RPE1: IC1.53, U2.25, U2.3
- new net U1FS: IC1.41, U1.22, U1.44
- new net U201: J1.8, U2.7, U2.8, U2.9
- new net U202: J1.7, U2.36, U2.37, U2.38
- new net U203: J1.6, U2.29, U2.30, U2.31
- new net U204: J1.5, U2.14, U2.15, U2.16
- new net U2FS: IC1.42, U2.22, U2.44
- new net U3RX: IC1.78, IC4.3
- new net U3TX: IC1.77, IC4.2
- new net U6RX: IC1.67, IC2.7
- new net U6TX: IC1.51, IC2.4
- net +24V: now also C22.2, C23.1, C24.2, C25.2
- net +3V3: now also C27.1, J1.2; no longer SV2.3
- net +5V: now also C26.1; no longer C15.1, C17.1, C3.1, IC2.3, IC3.6, IC5.6, IC6.6, IC7.6, IC8.6, IC9.6, X1.7, X1.8, X3.10
- net N$16: now also IC1.73; no longer IC1.74
- net N$24: now also C22.1, U1.19; no longer U2.7, U2.8, U2.9
- net N$25: now also C23.2, U1.41; no longer U2.36, U2.37, U2.38
- net N$26: now also C24.1, U2.19; no longer U2.14, U2.15, U2.16
- net N$27: now also C25.1, U2.41; no longer U2.29, U2.30, U2.31
- net VCC: now also C15.1, C17.1, C3.1, IC2.3, IC3.6, IC5.6, IC6.6, IC7.6, IC8.6, IC9.6, SV2.3, X1.7, X1.8, X3.10
- net VDD: no longer J1.2
- net VSS: now also C26.2, C27.2, LED1.C, LED2.C, LED3.C, U1.1, U1.23, U2.1, U2.23
Routing:
- net VCC: track 32.2 -> 249.0 mm, vias 2 -> 3
- net U2FS: track 0.00 -> 142.6 mm, vias 0 -> 4
- net RPE0: track 0.00 -> 139.0 mm, vias 0 -> 2
- net +5V: track 208.9 -> 82.2 mm
- net RPE1: track 0.00 -> 114.6 mm, vias 0 -> 2
- net U1FS: track 0.00 -> 114.0 mm, vias 0 -> 4
- net PWM3L: track 0.00 -> 111.7 mm, vias 0 -> 4
- net PWM4L: track 0.00 -> 105.7 mm, vias 0 -> 4
- net U6RX: track 0.00 -> 90.0 mm, vias 0 -> 2
- net PWM4H: track 0.00 -> 89.9 mm, vias 0 -> 2
- net PWM3H: track 0.00 -> 77.7 mm, vias 0 -> 4
- net DERE: track 0.00 -> 60.9 mm, vias 0 -> 2
- net N$36: track 0.00 -> 59.6 mm, vias 0 -> 2
- net U203: track 0.00 -> 59.3 mm, vias 0 -> 1
- net U6TX: track 0.00 -> 57.1 mm, vias 0 -> 4
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
Commit message: up
Connections:
- net VCC: no longer U$1.VCC
- net VDD: now also U$1.VCC
Routing:
- net RPE0: track 139.0 -> 77.2 mm, vias 2 -> 5
- net PWM4L: track 105.7 -> 146.0 mm, vias 4 -> 2
- net PWM2H: track 77.8 -> 111.4 mm, vias 6 -> 4
- net PWM3L: track 111.7 -> 83.9 mm, vias 4 -> 2
- net PWM1H: track 77.6 -> 101.8 mm
- net U1O3: track 41.8 -> 64.6 mm
- net U2FS: track 142.6 -> 164.4 mm, vias 4 -> 2
- net U6TX: track 57.1 -> 76.1 mm, vias 4 -> 2
- net N$14: track 17.0 -> 35.5 mm
- net PWM3H: track 77.7 -> 95.1 mm
- net VCC: track 249.0 -> 232.0 mm
- net +3V3: track 72.9 -> 89.1 mm, vias 3 -> 1
- net U6RX: track 90.0 -> 74.2 mm
- net U1FS: track 114.0 -> 129.4 mm, vias 4 -> 2
- net VDD: track 274.4 -> 289.1 mm, vias 2 -> 0
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
Commit message: up
Routing:
- net VDD: track 289.1 -> 351.6 mm, vias 0 -> 5
- net U2FS: track 164.4 -> 124.5 mm, vias 2 -> 3
- net U1FS: track 129.4 -> 96.5 mm
- net PWM1H: track 101.8 -> 129.4 mm, vias 4 -> 2
- net PWM2H: track 111.4 -> 84.1 mm
- net U204: track 49.2 -> 74.0 mm, vias 1 -> 0
- net U1O3: track 64.6 -> 41.6 mm, vias 1 -> 0
- net +3V3: track 89.1 -> 66.6 mm, vias 1 -> 0
- net N$36: track 54.9 -> 77.2 mm, vias 2 -> 0
- net VCC: track 232.0 -> 213.2 mm, vias 3 -> 4
- net N$14: track 35.5 -> 16.9 mm
- net RD8: track 23.9 -> 41.2 mm, vias 2 -> 0
- net RPE0: track 77.2 -> 92.8 mm, vias 5 -> 2
- net U6TX: track 76.1 -> 60.8 mm
- net U6RX: track 74.2 -> 59.8 mm, vias 2 -> 4
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
Commit message: up
Parts:
- removed S3: JS202011SCQN, JS202011SCQN_fixed:SW_JS202011SCQN
- removed U$2: IRLML2502TRPBF, IRLML2502TRPBF:SOT23
- added U3: ULN2803ADW, maxim-10:SOIC127P1030X265-18N
Connections:
- net GND: now also U3.9
Changed lines of the file:
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@@
 <attribute name="VALUE" x="22.453009375" y="5.0367" size="1.27" layer="27" align="center"/>
-</element>
-<element name="S3" library="JS202011SCQN_fixed" package="SW_JS202011SCQN" value="JS202011SCQN" x="11.43" y="74.93" smashed="yes">
-<attribute name="AVAILABILITY" value="Unavailable" x="55.88" y="67.31" size="1.778" layer="27" display="off"/>
-<attribute name="DESCRIPTION" value=" JS Series DPDT On-On Gull Wing Surface Mount Subminiature Slide Switch " x="55.88" y="67.31" size="1.778" layer="27" display="off"/>
-<attribute name="MF" value="C&amp;K" x="55.88" y="67.31" size="1.778" layer="27" display="off"/>
-<attribute name="MP" value="JS202011SCQN" x="55.88" y="67.31" size="1.778" layer="27" display="off"/>
-<attribute name="NAME" x="7.423009375" y="79.93873125" size="1.01776875" layer="25"/>
-<attribute name="PACKAGE" value="None" x="55.88" y="67.31" size="1.778" layer="27" display="off"/>
-<attribute name="PRICE" value="None" x="55.88" y="67.31" size="1.778" layer="27" display="off"/>
-<attribute name="VALUE" x="7.425009375" y="68.922509375" size="1.01726875" layer="27"/>
 </element>
 <element name="SV2" library="con-lstb" library_urn="urn:adsk.eagle:library:162" package="MA06-1" package3d_urn="urn:adsk.eagle:package:8340/1" value="ICSP2" x="6.35" y="13.97" smashed="yes" rot="R90">
@@
 <attribute name="PRICE" value="None" x="63.5" y="-19.05" size="1.778" layer="27" display="off"/>
 <attribute name="VALUE" x="49.96058125" y="12.637940625" size="1.27105" layer="27" rot="R90"/>
-</element>
-<element name="U$2" library="IRLML2502TRPBF" package="SOT23" value="IRLML2502TRPBF" x="21.59" y="72.39" smashed="yes">
-<attribute name="DESCRIPTION" value=" Single N-Channel 20 V 0.08 Ohm 12 nC 1.25 W Silicon SMT Mosfet - SOT-23 " x="67.31" y="27.94" size="1.778" layer="27" display="off"/>
-<attribute name="DIGI-KEY_PART_NUMBER" value="IRLML2502TRPBFCT-ND" x="67.31" y="27.94" size="1.778" layer="27" display="off"/>
-<attribute name="DIGI-KEY_PURCHASE_URL" value="https://www.digikey.com/product-detail/en/infineon-technologies/IRLML2502TRPBF/IRLML2502TRPBFCT-ND/812502?utm_source=snapeda&amp;utm_medium=aggregator&amp;utm_campaign=symbol" x="67.31" y="27.94" size="1.778" layer="27" display="off"/>
-<attribute name="MF" value="Infineon" x="67.31" y="27.94" size="1.778" layer="27" display="off"/>
-<attribute name="MP" value="IRLML2502TRPBF" x="67.31" y="27.94" size="1.778" layer="27" display="off"/>
-<attribute name="NAME" x="19.678440625" y="74.301559375" size="1.27436875" layer="25"/>
-<attribute name="PACKAGE" value="SOT-23-3 Infineon" x="67.31" y="27.94" size="1.778" layer="27" display="off"/>
-<attribute name="VALUE" x="19.67896875" y="69.20495" size="1.27401875" layer="27"/>
 </element>
 <element name="C5" library="rcl" library_urn="urn:adsk.eagle:library:334" package="C0805" package3d_urn="urn:adsk.eagle:package:23617/2" value="0.1" x="12.7" y="22.86" smashed="yes" rot="R180">
@@
 <attribute name="SPICEPREFIX" value="C" x="36.83" y="54.61" size="1.778" layer="27" rot="R180" display="off"/>
 <attribute name="VALUE" x="38.1" y="57.15" size="1.27" layer="27" rot="R180"/>
+</element>
+<element name="U3" library="maxim-10" package="SOIC127P1030X265-18N" value="ULN2803ADW" x="16.51" y="72.39" smashed="yes" rot="R90">
+<attribute name="AVAILABILITY" value="Unavailable" x="16.51" y="72.39" size="1.778" layer="27" rot="R90" display="off"/>
+<attribute name="DESCRIPTION" value=" Bipolar (BJT) Transistor Array 8 NPN Darlington 50V 500mA Surface Mount 18-SOIC " x="16.51" y="72.39" size="1.778" layer="27" rot="R90" display="off"/>
+<attribute name="DIGIKEY-PURCHASE-URL" value="https://snapeda.com/shop?store=DigiKey&amp;id=38030" x="16.51" y="72.39" size="1.778" layer="27" rot="R90" display="off"/>
+<attribute name="MF" value="Texas Instruments" x="16.51" y="72.39" size="1.778" layer="27" rot="R90" display="off"/>
+<attribute name="MP" value="ULN2803ADW" x="16.51" y="72.39" size="1.778" layer="27" rot="R90" display="off"/>
+<attribute name="NAME" x="8.884390625" y="68.933059375" size="2.08433125" layer="25" ratio="10" rot="SR90"/>
+<attribute name="PACKAGE" value="SOIC-18 Texas Instruments" x="16.51" y="72.39" size="1.778" layer="27" rot="R90" display="off"/>
+<attribute name="PRICE" value="None" x="16.51" y="72.39" size="1.778" layer="27" rot="R90" display="off"/>
+<attribute name="VALUE" x="25.40215" y="68.93476875" size="2.0833" layer="27" ratio="10" rot="SR90"/>
 </element>
 </elements>
@@
 <via x="66.7512" y="21.5646" extent="1-16" drill="0.35"/>
 <via x="69.9516" y="22.6314" extent="1-16" drill="0.35"/>
+<contactref element="U3" pad="9"/>
+<wire x1="21.59" y1="67.7164" x2="47.375" y2="11.361" width="0" layer="19" extent="1-1"/>
 </signal>
 <signal name="VCC">
