File: pic32mk.brd (EAGLE design)
At the start: 108.9 x 85.1 mm, 85 parts, among them IC1 PIC32MK1024MCF100-I_PT, IC2 ADM3095EBRZ, IC3 TXB0101DCKR, IC4 MAX203ECWP, IC5 TXB0101DCKR, IC6 TXB0101DCKR, IC7 TXB0101DCKR, IC8 TXB0101DCKR, IC9 TXB0101DCKR, J1 1-1586043-4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

Commit message: up
Parts:
- turned RS485 to 0 degrees
Routing:
- net VSS: track 765.0 -> 773.4 mm
- net N$39: track 39.2 -> 33.9 mm
- net VCC: track 366.1 -> 361.6 mm, vias 13 -> 15
Other:
- board text added: "fgb@mchp vcan 1.01"
- board text removed: "fgb@mchp vcan 1.0"

Commit message: up
Connections:
- net VCC: no longer SV2.3
- net VDD: now also SV2.2
- net VSS: now also SV2.3; no longer SV2.2
Routing:
- net VCC: track 361.6 -> 351.1 mm
- net VDD: track 371.7 -> 379.9 mm
- net VSS: track 773.4 -> 775.7 mm, vias 17 -> 18
Other:
- board text added: "fgb@mchp vcan 1.02"
- board text removed: "fgb@mchp vcan 1.01"
Changed lines of the file:
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@@
 <hole x="1.27" y="-1.27" drill="2.3476"/>
 <hole x="45.72" y="38.1" drill="2.3476"/>
-<text x="73.66" y="-1.27" size="1.778" layer="1" font="vector" ratio="15">fgb@mchp vcan 1.01</text>
+<text x="73.66" y="-1.27" size="1.778" layer="1" font="vector" ratio="15">fgb@mchp vcan 1.02</text>
 </plain>
 <attributes>
@@
 <contactref element="X1" pad="7"/>
 <contactref element="DIN" pad="10"/>
-<contactref element="SV2" pad="3"/>
 <contactref element="RS485" pad="5"/>
 <contactref element="SPI" pad="7"/>
@@
 <wire x1="12.2682" y1="54.5592" x2="12.2682" y2="55.245" width="0.1524" layer="1"/>
 <wire x1="12.2682" y1="52.959" x2="12.2682" y2="54.5592" width="0.1524" layer="16"/>
-<wire x1="5.1054" y1="11.811" x2="5.1054" y2="11.43" width="0.1524" layer="16"/>
-<wire x1="6.858" y1="13.5636" x2="5.1054" y2="11.811" width="0.1524" layer="16"/>
-<wire x1="6.858" y1="21.1074" x2="6.858" y2="13.5636" width="0.1524" layer="16"/>
 <wire x1="5.1054" y1="22.86" x2="6.858" y2="21.1074" width="0.1524" layer="16"/>
 <wire x1="5.1054" y1="25.3746" x2="5.1054" y2="22.86" width="0.1524" layer="1"/>
@@
 <wire x1="10.1346" y1="36.4236" x2="9.6774" y2="36.8808" width="0.1524" layer="1"/>
 <wire x1="11.1252" y1="36.4236" x2="10.1346" y2="36.4236" width="0.1524" layer="1"/>
-<wire x1="5.1054" y1="11.43" x2="5.08" y2="11.43" width="0.1524" layer="16"/>
 <wire x1="31.3944" y1="45.72" x2="31.75" y2="45.72" width="0.1524" layer="16"/>
 <wire x1="29.4132" y1="47.7012" x2="31.3944" y2="45.72" width="0.1524" layer="16"/>
@@
 <wire x1="62.5602" y1="6.3246" x2="62.55" y2="6.35" width="0.1524" layer="1"/>
 <wire x1="80.01" y1="8.5344" x2="80.01" y2="8.57" width="0.1524" layer="1"/>
-<wire x1="10.2108" y1="2.9718" x2="10.2108" y2="2.5908" width="0.1524" layer="1"/>
+<wire x1="10.2108" y1="2.9718" x2="10.2108" y2="2.866275" width="0.1524" layer="1"/>
+<wire x1="10.2108" y1="2.866275" x2="10.2108" y2="2.5908" width="0.1524" layer="1"/>
 <wire x1="12.3444" y1="5.1054" x2="10.2108" y2="2.9718" width="0.1524" layer="1"/>
 <wire x1="16.764" y1="5.1054" x2="12.3444" y2="5.1054" width="0.1524" layer="1"/>
@@
 <via x="51.5112" y="14.3256" extent="1-16" drill="0.35"/>
 <via x="54.5592" y="17.3736" extent="1-16" drill="0.35"/>
+<wire x1="7.1374" y1="5.939675" x2="10.2108" y2="2.866275" width="0.1524" layer="1"/>
+<contactref element="SV2" pad="2"/>
+<wire x1="5.08" y1="8.89" x2="7.1374" y2="6.8326" width="0.1524" layer="1"/>
+<wire x1="7.1374" y1="6.8326" x2="7.1374" y2="5.939675" width="0.1524" layer="1"/>
 </signal>
 <signal name="VSS">
@@
 <contactref element="C10" pad="2"/>
 <contactref element="C11" pad="2"/>
-<contactref element="SV2" pad="2"/>
 <contactref element="OS2" pad="2"/>
 <contactref element="C12" pad="2"/>
@@
 <wire x1="19.9644" y1="3.81" x2="20" y2="3.81" width="0.1524" layer="1"/>
 <wire x1="17.3736" y1="6.3246" x2="19.8882" y2="3.81" width="0.1524" layer="1"/>
-<wire x1="10.2108" y1="6.3246" x2="17.3736" y2="6.3246" width="0.1524" layer="1"/>
+<wire x1="10.2108" y1="6.3246" x2="17.145" y2="6.3246" width="0.1524" layer="1"/>
+<wire x1="17.145" y1="6.3246" x2="17.3736" y2="6.3246" width="0.1524" layer="1"/>
 <wire x1="19.8882" y1="3.81" x2="20" y2="3.81" width="0.1524" layer="1"/>
 <wire x1="10.2108" y1="6.3246" x2="10.16" y2="6.35" width="0.1524" layer="1"/>
-<wire x1="7.5438" y1="8.8392" x2="5.1054" y2="8.8392" width="0.1524" layer="1"/>
-<wire x1="9.9822" y1="6.4008" x2="7.5438" y2="8.8392" width="0.1524" layer="1"/>
-<wire x1="10.1346" y1="6.4008" x2="9.9822" y2="6.4008" width="0.1524" layer="1"/>
-<wire x1="5.1054" y1="8.8392" x2="5.08" y2="8.89" width="0.1524" layer="1"/>
+<wire x1="9.9822" y1="6.4008" x2="10.00834375" y2="6.4008" width="0.1524" layer="1"/>
 <wire x1="10.1346" y1="6.4008" x2="10.16" y2="6.35" width="0.1524" layer="1"/>
 <wire x1="9.2202" y1="12.192" x2="9.2202" y2="12.6492" width="0.1524" layer="1"/>
-<wire x1="12.2682" y1="9.144" x2="9.2202" y2="12.192" width="0.1524" layer="1"/>
-<wire x1="13.8684" y1="9.144" x2="12.2682" y2="9.144" width="0.1524" layer="1"/>
-<wire x1="14.859" y1="10.1346" x2="13.8684" y2="9.144" width="0.1524" layer="1"/>
 <wire x1="9.2202" y1="12.6492" x2="9.21" y2="12.7" width="0.1524" layer="1"/>
 <wire x1="14.859" y1="10.1346" x2="14.92" y2="10.16" width="0.1524" layer="1"/>
@@
 <wire x1="9.144" y1="12.7254" x2="9.21" y2="12.7" width="0.1524" layer="1"/>
 <wire x1="6.0198" y1="24.0792" x2="6.03" y2="24.13" width="0.1524" layer="1"/>
-<wire x1="6.0198" y1="8.9154" x2="5.1054" y2="8.9154" width="0.1524" layer="16"/>
-<wire x1="7.7724" y1="10.668" x2="6.0198" y2="8.9154" width="0.1524" layer="16"/>
-<wire x1="9.2202" y1="12.1158" x2="7.7724" y2="10.668" width="0.1524" layer="1"/>
-<wire x1="5.1054" y1="8.9154" x2="5.08" y2="8.89" width="0.1524" layer="16"/>
 <wire x1="9.2202" y1="12.1158" x2="9.21" y2="12.7" width="0.1524" layer="1"/>
 <wire x1="38.1" y1="4.3434" x2="34.29" y2="4.3434" width="0.1524" layer="1"/>
@@
 <via x="8.8392" y="33.147" extent="1-16" drill="0.35"/>
 <via x="7.0866" y="30.6324" extent="1-16" drill="0.35"/>
-<via x="7.7724" y="10.668" extent="1-16" drill="0.35"/>
 <via x="41.4528" y="43.2054" extent="1-16" drill="0.35"/>
 <via x="31.6992" y="35.9664" extent="1-16" drill="0.35"/>
@@
 <wire x1="102.87" y1="11.43" x2="103.7844" y2="12.3444" width="0.1524" layer="1"/>
 <wire x1="97.8408" y1="20.2692" x2="97.79" y2="20.32" width="0.1524" layer="1"/>
+<wire x1="13.7922" y1="9.144" x2="14.7828" y2="10.1346" width="0.1524" layer="1"/>
+<wire x1="12.2682" y1="9.144" x2="13.7922" y2="9.144" width="0.1524" layer="1"/>
+<wire x1="9.2964" y1="12.1158" x2="12.2682" y2="9.144" width="0.1524" layer="1"/>
+<wire x1="14.7828" y1="10.1346" x2="14.92" y2="10.16" width="0.1524" layer="1"/>
+<wire x1="9.2964" y1="12.1158" x2="9.21" y2="12.7" width="0.1524" layer="1"/>
+<wire x1="9.144" y1="12.1158" x2="9.21" y2="12.7" width="0.1524" layer="1"/>
+<wire x1="17.145" y1="6.858" x2="17.145" y2="6.3246" width="0.1524" layer="1"/>
+<wire x1="17.145" y1="9.2964" x2="17.145" y2="6.858" width="0.1524" layer="16"/>
+<wire x1="16.383" y1="9.2964" x2="17.145" y2="9.2964" width="0.1524" layer="1"/>
+<wire x1="15.5448" y1="10.1346" x2="16.383" y2="9.2964" width="0.1524" layer="1"/>
+<wire x1="14.9352" y1="10.1346" x2="15.5448" y2="10.1346" width="0.1524" layer="1"/>
+<wire x1="14.9352" y1="10.1346" x2="14.92" y2="10.16" width="0.1524" layer="1"/>
+<via x="17.145" y="6.858" extent="1-16" drill="0.35"/>
+<via x="17.145" y="9.2964" extent="1-16" drill="0.35"/>
+<contactref element="SV2" pad="3"/>
+<wire x1="5.08" y1="11.43" x2="7.8232" y2="8.6868" width="0.1524" layer="1"/>
+<wire x1="7.8232" y1="8.6868" x2="7.8232" y2="8.58594375" width="0.1524" layer="1"/>
+<wire x1="7.8232" y1="8.58594375" x2="10.00834375" y2="6.4008" width="0.1524" layer="1"/>
+<wire x1="10.00834375" y1="6.4008" x2="10.1346" y2="6.4008" width="0.1524" layer="1"/>
 </signal>
 <signal name="+5V">
@@
 <wire x1="11.3538" y1="7.8486" x2="12.192" y2="8.6868" width="0.1524" layer="1"/>
 <wire x1="8.9916" y1="7.8486" x2="11.3538" y2="7.8486" width="0.1524" layer="1"/>
-<wire x1="6.858" y1="9.9822" x2="8.9916" y2="7.8486" width="0.1524" layer="1"/>
-<wire x1="6.858" y1="11.8872" x2="6.858" y2="9.9822" width="0.1524" layer="1"/>
-<wire x1="5.7912" y1="12.954" x2="6.858" y2="11.8872" width="0.1524" layer="1"/>
+<wire x1="8.128" y1="8.7122" x2="8.9916" y2="7.8486" width="0.1524" layer="1"/>
+<wire x1="8.128" y1="10.6172" x2="8.128" y2="8.7122" width="0.1524" layer="1"/>
+<wire x1="5.7912" y1="12.954" x2="8.128" y2="10.6172" width="0.1524" layer="1"/>
 <wire x1="3.8862" y1="12.954" x2="5.7912" y2="12.954" width="0.1524" layer="1"/>
 <wire x1="1.7526" y1="15.0876" x2="3.8862" y2="12.954" width="0.1524" layer="1"/>

Commit message: up
Connections:
- net VCC: now also C14.1, C16.1, IC3.1, IC5.1, IC6.1, IC7.1, IC8.1, IC9.1; no longer C15.1, C17.1, IC3.6, IC5.6, IC6.6, IC7.6, IC8.6, IC9.6
- net VDD: now also C15.1, C17.1, IC3.6, IC5.6, IC6.6, IC7.6, IC8.6, IC9.6; no longer C14.1, C16.1, IC3.1, IC5.1, IC6.1, IC7.1, IC8.1, IC9.1
Routing:
- net VCC: track 351.1 -> 369.0 mm, vias 15 -> 17
- net VDD: track 379.9 -> 367.7 mm, vias 25 -> 27

Commit message: up
Connections:
- net N$10: now also IC8.4; no longer IC8.3
- net N$11: now also IC6.4; no longer IC6.3
- net N$12: now also IC7.4; no longer IC7.3
- net N$15: now also IC9.4; no longer IC9.3
- net N$5: now also IC3.4; no longer IC3.3
- net N$8: now also IC5.4; no longer IC5.3
- net RPA0: now also IC8.3; no longer IC8.4
- net RPA14: now also IC6.3; no longer IC6.4
- net RPB1: now also IC3.3; no longer IC3.4
- net RPB6: now also IC7.3; no longer IC7.4
- net RPC1: now also IC5.3; no longer IC5.4
- net RPC10: now also IC9.3; no longer IC9.4
Routing:
- net RPC10: track 58.4 -> 87.2 mm
- net VCC: track 369.0 -> 395.9 mm
- net N$15: track 7.47 -> 31.5 mm, vias 0 -> 1
- net RPB1: track 79.6 -> 100.6 mm
- net N$8: track 8.74 -> 25.8 mm, vias 0 -> 1
- net RPA14: track 96.9 -> 82.7 mm, vias 8 -> 10
- net N$12: track 8.73 -> 20.5 mm, vias 0 -> 3
- net VSS: track 775.7 -> 787.0 mm, vias 18 -> 21
- net RPB6: track 40.5 -> 47.0 mm
- net N$11: track 7.81 -> 14.1 mm, vias 0 -> 1
- net VDD: track 367.7 -> 371.6 mm, vias 27 -> 25
- net RPA0: track 37.1 -> 40.8 mm
- net N$10: track 8.74 -> 12.3 mm
- net N$5: track 7.49 -> 9.88 mm, vias 0 -> 1
- net RPC1: track 47.0 -> 49.1 mm
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Other:
- board text added: "fgb@mchp vcan 1.03"
- board text removed: "fgb@mchp vcan 1.02"

Commit message: up
Connections:
- net RC11: now also SPI.9
- net RC2: now also SPI.6
- net VDD: now also SPI.10
Routing:
- net RC11: track 52.1 -> 70.1 mm, vias 4 -> 5
- net VDD: track 371.6 -> 384.0 mm, vias 25 -> 26
- net RC2: track 80.0 -> 87.7 mm, vias 2 -> 3
Changed lines of the file:
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@@
 <via x="11.1252" y="53.4924" extent="1-16" drill="0.35"/>
 <via x="13.335" y="46.1772" extent="1-16" drill="0.35"/>
+<contactref element="SPI" pad="10"/>
+<wire x1="46.9392" y1="10.2108" x2="46.9392" y2="8.9154" width="0.1524" layer="1"/>
+<wire x1="44.577" y1="12.573" x2="46.9392" y2="10.2108" width="0.1524" layer="1"/>
+<wire x1="49.7586" y1="12.573" x2="44.577" y2="12.573" width="0.1524" layer="16"/>
+<wire x1="51.5112" y1="14.3256" x2="49.7586" y2="12.573" width="0.1524" layer="16"/>
+<wire x1="46.9392" y1="8.9154" x2="46.99" y2="8.89" width="0.1524" layer="1"/>
+<via x="44.577" y="12.573" extent="1-16" drill="0.35"/>
 </signal>
 <signal name="VSS">
@@
 <wire x1="40.6908" y1="13.4874" x2="40.6908" y2="13.9446" width="0.1524" layer="1"/>
 <wire x1="42.9006" y1="11.2776" x2="40.6908" y2="13.4874" width="0.1524" layer="1"/>
-<wire x1="42.9006" y1="-0.0762" x2="42.9006" y2="11.2776" width="0.1524" layer="1"/>
+<wire x1="42.9006" y1="-0.0762" x2="42.9006" y2="5.715" width="0.1524" layer="1"/>
+<wire x1="42.9006" y1="5.715" x2="42.9006" y2="11.2776" width="0.1524" layer="1"/>
 <wire x1="41.6814" y1="-1.2954" x2="42.9006" y2="-0.0762" width="0.1524" layer="1"/>
 <wire x1="6.3246" y1="-1.2954" x2="41.6814" y2="-1.2954" width="0.1524" layer="1"/>
@@
 <via x="29.8704" y="17.8308" extent="1-16" drill="0.35"/>
 <via x="40.6908" y="13.9446" extent="1-16" drill="0.35"/>
+<contactref element="SPI" pad="6"/>
+<wire x1="36.8808" y1="8.3058" x2="36.8808" y2="8.8392" width="0.1524" layer="16"/>
+<wire x1="39.4716" y1="5.715" x2="36.8808" y2="8.3058" width="0.1524" layer="16"/>
+<wire x1="42.8244" y1="5.715" x2="39.4716" y2="5.715" width="0.1524" layer="16"/>
+<wire x1="42.9006" y1="5.715" x2="42.8244" y2="5.715" width="0.1524" layer="1"/>
+<wire x1="36.8808" y1="8.8392" x2="36.83" y2="8.89" width="0.1524" layer="16"/>
+<via x="42.8244" y="5.715" extent="1-16" drill="0.35"/>
 </signal>
 <signal name="RC11">
@@
 <via x="30.2514" y="6.858" extent="1-16" drill="0.35"/>
 <via x="22.2504" y="-0.6858" extent="1-16" drill="0.35"/>
+<contactref element="SPI" pad="9"/>
+<wire x1="44.4246" y1="6.4008" x2="44.4246" y2="8.8392" width="0.1524" layer="1"/>
+<wire x1="43.7388" y1="5.715" x2="44.4246" y2="6.4008" width="0.1524" layer="1"/>
+<wire x1="43.1292" y1="5.1054" x2="43.7388" y2="5.715" width="0.1524" layer="16"/>
+<wire x1="40.1574" y1="5.1054" x2="43.1292" y2="5.1054" width="0.1524" layer="16"/>
+<wire x1="39.8526" y1="5.4102" x2="40.1574" y2="5.1054" width="0.1524" layer="16"/>
+<wire x1="31.6992" y1="5.4102" x2="39.8526" y2="5.4102" width="0.1524" layer="16"/>
+<wire x1="30.2514" y1="6.858" x2="31.6992" y2="5.4102" width="0.1524" layer="16"/>
+<wire x1="44.4246" y1="8.8392" x2="44.45" y2="8.89" width="0.1524" layer="1"/>
+<via x="43.7388" y="5.715" extent="1-16" drill="0.35"/>
 </signal>
 <signal name="RG11">

Commit message: up
Connections:
- removed net DERE: IC1.74, IC2.5, IC2.6
- removed net N$16: IC1.73, OS2.3
- new net N$1: IC1.74, OS2.3
- new net SOSCI: IC1.73
- net RG11: now also IC2.5, IC2.6
Routing:
- net DERE: track 61.2 -> 0.00 mm, vias 6 -> 0
- net N$1: track 0.00 -> 13.4 mm, vias 0 -> 2
- net N$16: track 12.3 -> 0.00 mm, vias 2 -> 0
- net RG11: track 43.4 -> 46.8 mm
- net IN8: track 54.8 -> 55.9 mm
- net RPA14: track 82.7 -> 83.7 mm
- net VSS: track 787.0 -> 787.7 mm
Changed lines of the file:
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@@
 <wire x1="42.5196" y1="42.1386" x2="41.4528" y2="43.2054" width="0.1524" layer="1"/>
 <wire x1="42.5196" y1="42.1386" x2="42.23" y2="41.91" width="0.1524" layer="1"/>
-<wire x1="47.0154" y1="32.766" x2="37.2618" y2="32.766" width="0.1524" layer="1"/>
-<wire x1="47.244" y1="32.9946" x2="47.0154" y2="32.766" width="0.1524" layer="1"/>
-<wire x1="37.2618" y1="32.766" x2="37.218" y2="32.74" width="0.1524" layer="1"/>
-<wire x1="47.244" y1="32.9946" x2="47.31" y2="33.02" width="0.1524" layer="1"/>
+<wire x1="47.31" y1="33.02" x2="46.294" y2="34.036" width="0.1524" layer="1"/>
+<wire x1="46.294" y1="34.036" x2="41.540725" y2="34.036" width="0.1524" layer="1"/>
+<wire x1="41.540725" y1="34.036" x2="39.3574625" y2="32.74" width="0.1524" layer="1"/>
+<wire x1="39.3574625" y1="32.74" x2="37.218" y2="32.74" width="0.1524" layer="1"/>
 <wire x1="31.6992" y1="35.9664" x2="31.6992" y2="34.7472" width="0.1524" layer="1"/>
 <wire x1="31.6992" y1="34.1376" x2="31.6992" y2="35.9664" width="0.1524" layer="16"/>
@@
 <via x="11.5062" y="26.3652" extent="1-16" drill="0.35"/>
 </signal>
-<signal name="N$16">
-<contactref element="OS2" pad="3"/>
-<contactref element="IC1" pad="73"/>
-<wire x1="46.9392" y1="28.575" x2="47.3964" y2="28.575" width="0.1524" layer="1"/>
-<wire x1="46.2534" y1="29.2608" x2="46.9392" y2="28.575" width="0.1524" layer="1"/>
-<wire x1="46.2534" y1="30.4038" x2="46.2534" y2="29.2608" width="0.1524" layer="16"/>
-<wire x1="45.1104" y1="31.5468" x2="46.2534" y2="30.4038" width="0.1524" layer="16"/>
-<wire x1="44.6532" y1="31.5468" x2="45.1104" y2="31.5468" width="0.1524" layer="1"/>
-<wire x1="44.2722" y1="31.9278" x2="44.6532" y2="31.5468" width="0.1524" layer="1"/>
-<wire x1="37.2618" y1="31.9278" x2="44.2722" y2="31.9278" width="0.1524" layer="1"/>
-<wire x1="47.3964" y1="28.575" x2="47.41" y2="28.56" width="0.1524" layer="1"/>
-<wire x1="37.2618" y1="31.9278" x2="37.218" y2="31.94" width="0.1524" layer="1"/>
-<via x="46.2534" y="29.2608" extent="1-16" drill="0.35"/>
-<via x="45.1104" y="31.5468" extent="1-16" drill="0.35"/>
-</signal>
 <signal name="RE8">
 <contactref element="IC6" pad="5"/>
@@
 <wire x1="38.6334" y1="34.9758" x2="38.6334" y2="41.7576" width="0.1524" layer="1"/>
 <wire x1="42.672" y1="30.9372" x2="38.6334" y2="34.9758" width="0.1524" layer="16"/>
-<wire x1="40.6146" y1="30.9372" x2="42.672" y2="30.9372" width="0.1524" layer="1"/>
-<wire x1="38.862" y1="29.1846" x2="40.6146" y2="30.9372" width="0.1524" layer="1"/>
-<wire x1="37.2618" y1="29.1846" x2="38.862" y2="29.1846" width="0.1524" layer="1"/>
+<wire x1="42.672" y1="30.9372" x2="42.672" y2="29.1846" width="0.1524" layer="1"/>
+<wire x1="37.2618" y1="29.1846" x2="42.672" y2="29.1846" width="0.1524" layer="1"/>
 <wire x1="37.2618" y1="29.1846" x2="37.218" y2="29.14" width="0.1524" layer="1"/>
 <via x="22.7838" y="58.4454" extent="1-16" drill="0.35"/>
@@
 <via x="83.2866" y="15.0114" extent="1-16" drill="0.35"/>
 </signal>
-<signal name="DERE">
-<contactref element="IC2" pad="6"/>
-<contactref element="IC2" pad="5"/>
-<contactref element="IC1" pad="74"/>
-<wire x1="45.2628" y1="32.3088" x2="37.2618" y2="32.3088" width="0.1524" layer="1"/>
-<wire x1="46.0248" y1="31.5468" x2="45.2628" y2="32.3088" width="0.1524" layer="1"/>
-<wire x1="46.0248" y1="31.0896" x2="46.0248" y2="31.5468" width="0.1524" layer="16"/>
-<wire x1="47.9298" y1="29.1846" x2="46.0248" y2="31.0896" width="0.1524" layer="16"/>
-<wire x1="47.9298" y1="27.5082" x2="47.9298" y2="29.1846" width="0.1524" layer="16"/>
-<wire x1="50.2158" y1="27.5082" x2="47.9298" y2="27.5082" width="0.1524" layer="1"/>
-<wire x1="50.2158" y1="27.3558" x2="50.2158" y2="27.5082" width="0.1524" layer="16"/>
-<wire x1="49.4538" y1="26.5938" x2="50.2158" y2="27.3558" width="0.1524" layer="16"/>
-<wire x1="49.4538" y1="25.9842" x2="49.4538" y2="26.5938" width="0.1524" layer="16"/>
-<wire x1="49.911" y1="25.527" x2="49.4538" y2="25.9842" width="0.1524" layer="16"/>
-<wire x1="53.9496" y1="25.527" x2="49.911" y2="25.527" width="0.1524" layer="16"/>
-<wire x1="61.341" y1="18.1356" x2="53.9496" y2="25.527" width="0.1524" layer="16"/>
-<wire x1="61.341" y1="15.0876" x2="61.341" y2="18.1356" width="0.1524" layer="1"/>
-<wire x1="61.0362" y1="14.7828" x2="61.341" y2="15.0876" width="0.1524" layer="1"/>
-<wire x1="69.8754" y1="14.7828" x2="61.0362" y2="14.7828" width="0.1524" layer="16"/>
-<wire x1="73.0758" y1="17.9832" x2="69.8754" y2="14.7828" width="0.1524" layer="16"/>
-<wire x1="78.9432" y1="17.9832" x2="73.0758" y2="17.9832" width="0.1524" layer="16"/>
-<wire x1="79.248" y1="17.9832" x2="78.9432" y2="17.9832" width="0.1524" layer="1"/>
-<wire x1="79.5528" y1="18.288" x2="79.248" y2="17.9832" width="0.1524" layer="1"/>
-<wire x1="80.1624" y1="18.288" x2="79.5528" y2="18.288" width="0.1524" layer="1"/>
-<wire x1="81.915" y1="16.5354" x2="80.1624" y2="18.288" width="0.1524" layer="1"/>
-<wire x1="81.915" y1="16.383" x2="81.915" y2="16.5354" width="0.1524" layer="1"/>
-<wire x1="37.2618" y1="32.3088" x2="37.218" y2="32.34" width="0.1524" layer="1"/>
-<wire x1="81.915" y1="16.383" x2="83.1342" y2="16.383" width="0.1524" layer="1"/>
-<wire x1="83.1342" y1="16.383" x2="83.185" y2="16.338" width="0.1524" layer="1"/>
-<wire x1="81.915" y1="16.383" x2="81.915" y2="16.338" width="0.1524" layer="1"/>
-<via x="46.0248" y="31.5468" extent="1-16" drill="0.35"/>
-<via x="47.9298" y="27.5082" extent="1-16" drill="0.35"/>
-<via x="50.2158" y="27.5082" extent="1-16" drill="0.35"/>
-<via x="61.341" y="18.1356" extent="1-16" drill="0.35"/>
-<via x="61.0362" y="14.7828" extent="1-16" drill="0.35"/>
-<via x="78.9432" y="17.9832" extent="1-16" drill="0.35"/>
-</signal>
 <signal name="IN5">
 <contactref element="IC1" pad="61"/>
@@
 <wire x1="35.6616" y1="32.4612" x2="31.5468" y2="32.4612" width="0.1524" layer="1"/>
 <wire x1="36.7284" y1="33.528" x2="35.6616" y2="32.4612" width="0.1524" layer="1"/>
-<wire x1="44.4246" y1="33.528" x2="36.7284" y2="33.528" width="0.1524" layer="1"/>
-<wire x1="45.7962" y1="34.8996" x2="44.4246" y2="33.528" width="0.1524" layer="1"/>
+<wire x1="39.3446" y1="33.528" x2="36.7284" y2="33.528" width="0.1524" layer="1"/>
+<wire x1="45.7962" y1="34.8996" x2="44.5262" y2="36.1696" width="0.1524" layer="1"/>
+<wire x1="44.5262" y1="36.1696" x2="41.9862" y2="36.1696" width="0.1524" layer="1"/>
+<wire x1="41.9862" y1="36.1696" x2="39.3446" y2="33.528" width="0.1524" layer="1"/>
 <wire x1="50.0634" y1="39.1668" x2="45.7962" y2="34.8996" width="0.1524" layer="16"/>
 <wire x1="50.0634" y1="39.3954" x2="50.0634" y2="39.1668" width="0.1524" layer="16"/>
@@
 <via x="9.7536" y="20.3454" extent="1-16" drill="0.35"/>
 <via x="3.5814" y="10.287" extent="1-16" drill="0.35"/>
+<contactref element="IC2" pad="5"/>
+<contactref element="IC2" pad="6"/>
+<wire x1="81.915" y1="17.3736" x2="81.915" y2="16.338" width="0.1524" layer="1"/>
+<wire x1="81.9912" y1="17.4498" x2="81.915" y2="17.3736" width="0.1524" layer="1"/>
+<wire x1="83.1342" y1="17.4498" x2="81.9912" y2="17.4498" width="0.1524" layer="1"/>
+<wire x1="83.2104" y1="17.3736" x2="83.1342" y2="17.4498" width="0.1524" layer="1"/>
+<wire x1="83.2104" y1="16.383" x2="83.2104" y2="17.3736" width="0.1524" layer="1"/>
+<wire x1="83.2104" y1="16.383" x2="83.185" y2="16.338" width="0.1524" layer="1"/>
+<wire x1="30.48" y1="21.202" x2="81.915" y2="16.338" width="0" layer="19" extent="1-1"/>
 </signal>
 <signal name="RF13">
@@
 <via x="28.1178" y="31.623" extent="1-16" drill="0.35"/>
 </signal>
+<signal name="N$1">
+<contactref element="IC1" pad="74"/>
+<contactref element="OS2" pad="3"/>
+<wire x1="46.4058" y1="28.575" x2="47.3964" y2="28.575" width="0.1524" layer="1"/>
+<wire x1="46.2534" y1="28.7274" x2="46.4058" y2="28.575" width="0.1524" layer="1"/>
+<wire x1="46.2534" y1="29.2608" x2="46.2534" y2="28.7274" width="0.1524" layer="1"/>
+<wire x1="45.7962" y1="29.2608" x2="46.2534" y2="29.2608" width="0.1524" layer="16"/>
+<wire x1="45.4914" y1="29.5656" x2="45.7962" y2="29.2608" width="0.1524" layer="16"/>
+<wire x1="45.1104" y1="31.5468" x2="45.4914" y2="31.1658" width="0.1524" layer="16"/>
+<wire x1="45.4914" y1="31.1658" x2="45.4914" y2="29.5656" width="0.1524" layer="16"/>
+<wire x1="45.1104" y1="32.2072" x2="45.1104" y2="31.5468" width="0.1524" layer="1"/>
+<wire x1="45.0088" y1="32.3088" x2="45.1104" y2="32.2072" width="0.1524" layer="1"/>
+<wire x1="37.2618" y1="32.3088" x2="45.0088" y2="32.3088" width="0.1524" layer="1"/>
+<wire x1="47.3964" y1="28.575" x2="47.41" y2="28.56" width="0.1524" layer="1"/>
+<wire x1="37.2618" y1="32.3088" x2="37.218" y2="32.34" width="0.1524" layer="1"/>
+<via x="46.2534" y="29.2608" extent="1-16" drill="0.35"/>
+<via x="45.1104" y="31.5468" extent="1-16" drill="0.35"/>
+</signal>
+<signal name="SOSCI">
+<contactref element="IC1" pad="73"/>
+<wire x1="37.2618" y1="31.9278" x2="37.218" y2="31.94" width="0.1524" layer="1"/>
+</signal>
 </signals>
