File: pic32mk.brd (EAGLE design)
At the start: 108.9 x 85.1 mm, 85 parts, among them IC1 PIC32MK1024MCF100-I_PT, IC2 ADM3095EBRZ, IC3 TXB0101DCKR, IC4 MAX203ECWP, IC5 TXB0101DCKR, IC6 TXB0101DCKR, IC7 TXB0101DCKR, IC8 TXB0101DCKR, IC9 TXB0101DCKR, J1 1-1586043-4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

Commit message: up
Parts:
- removed JP1: vref-, pinhead:1X02
- removed JP2: vref+, pinhead:1X02
- added SPI_VOLTS: 1-2 3.3, 3-2 5.0, con-lstb:MA03-1
- moved R4 22.9 mm to (63.5, 19.1)
- moved C28 18.5 mm to (10.2, 17.8), turned to 180 degrees
- moved R7 16.1 mm to (72.4, 41.9)
- moved C29 12.5 mm to (10.2, 20.3), turned to 180 degrees
- moved R9 7.73 mm to (41.9, 49.5)
- moved JP4 7.73 mm to (35.6, 44.5)
- moved C8 6.48 mm to (41.9, 52.1)
- moved C16 6.48 mm to (8.89, 66.0), turned to 0 degrees
- moved C3 6.48 mm to (69.8, 8.89)
- moved C14 6.35 mm to (10.2, 44.5), turned to 0 degrees
- moved R8 6.35 mm to (72.4, 54.6)
- moved C17 6.35 mm to (8.89, 63.5), turned to 0 degrees
- moved C15 6.35 mm to (10.2, 41.9), turned to 0 degrees
- moved C4 5.68 mm to (77.5, 7.62), turned to 270 degrees
- moved C20 5.24 mm to (41.9, 54.6)
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Connections:
- removed net N$57: IC1.28, JP1.1
- removed net N$58: IC1.29, JP2.1
- new net N$16: SPI.7, SPI_VOLTS.2
- net REFOUT: now also IC1.29; no longer JP2.2
- net RG11: no longer JP3.3
- net VCC: now also SPI_VOLTS.3; no longer SPI.7
- net VDD: now also SPI_VOLTS.1
- net VSS: now also IC1.28; no longer JP1.2
Routing:
- net VSS: track 787.7 -> 403.3 mm, vias 21 -> 14
- net RF12: track 302.3 -> 94.4 mm, vias 9 -> 3
- net RF13: track 271.1 -> 109.1 mm, vias 6 -> 4
- net RE14: track 233.9 -> 80.7 mm, vias 10 -> 3
- net SPI_EN0: track 174.1 -> 29.9 mm, vias 3 -> 1
- net SPI_EN1: track 145.9 -> 26.6 mm, vias 5 -> 1
- net RG15: track 220.5 -> 103.9 mm, vias 12 -> 5
- net MCLEAR: track 245.0 -> 131.9 mm
- net REFOUT: track 196.6 -> 85.0 mm, vias 10 -> 2
- net N$34: track 140.4 -> 38.0 mm, vias 10 -> 2
- net VCC: track 395.9 -> 293.7 mm, vias 17 -> 6
- net +5V: track 205.4 -> 128.1 mm, vias 11 -> 3
- net PWM2L: track 110.3 -> 48.4 mm, vias 6 -> 2
- net VDD: track 384.0 -> 443.9 mm, vias 26 -> 10
- net RPB1: track 100.6 -> 43.4 mm, vias 8 -> 3
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- added copper zone on layer 2, net VSS
Other:
- board size 108.9 x 85.1 mm -> 110.2 x 85.1 mm
- board text added: "fgb@mchp vcan 1.04"
- board text removed: "fgb@mchp vcan 1.03"

Commit message: up
Parts:
- added C32, C33, C34, C35: 0.1, rcl:C0805
- added F3: 1206L050, polyfuse-smd_10:1206L
- added IC10: 5.0VDC, linear:TO220H
- added IC11: 3.3VDC, linear:TO220H
Connections:
- new net N$30: C32.1, C33.1, F3.2, IC10.1, IC11.1
- net +24V: now also F3.1
- net +3V3: now also C34.1, IC11.3
- net +5V: now also C35.1, IC10.3
- net RG11: now also JP3.3
- net VSS: now also C32.2, C33.2, C34.2, C35.2, IC10.2, IC11.2
Routing:
- net +3V3: track 73.1 -> 155.4 mm, vias 2 -> 3
- net +5V: track 128.1 -> 199.2 mm
- net N$6: track 77.9 -> 26.5 mm, vias 0 -> 2
- net RE8: track 98.4 -> 62.2 mm, vias 5 -> 7
- net GND: track 171.2 -> 137.7 mm, vias 3 -> 4
- net PWM2H: track 52.9 -> 86.2 mm, vias 3 -> 2
- net RG15: track 103.9 -> 136.7 mm, vias 5 -> 3
- net RG11: track 62.2 -> 93.9 mm, vias 2 -> 3
- net N$30: track 0.00 -> 30.1 mm
- net VCC: track 293.7 -> 322.6 mm
- net PWM1L: track 43.2 -> 71.6 mm
- net RA1: track 57.6 -> 29.7 mm
- net U2FS: track 64.2 -> 90.4 mm
- net RPA14: track 42.2 -> 62.2 mm, vias 2 -> 0
- net MCLEAR: track 131.9 -> 151.5 mm, vias 5 -> 3
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Other:
- board text added: "fgb@mchp vcan 1.05"
- board text removed: "fgb@mchp vcan 1.04"
