File: pic32mk.sch (EAGLE design)
At the start: 39 parts, among them IC1 PIC32MK1024MCF100-I_PT, IC2 ADM3095EBRZ, IC3 MC33931EK, IC4 MAX203ECWP, IC5 MC33931EK, IC6 TXB0101DCKR, IC7 TXB0101DCKR, IC8 TXB0101DCKR, X1 22-23-2101

Commit message: up
Parts:
- added C14, C15, C16, C17, C18, C19: 0.1, rcl:C-USC0805
- added IC9: TXB0101DCKR, TXB0101DCKR:TXB0101DCKR
- added J1: 1-1586043-4, 1-1586043-4:1-1586043-4
- added U1, U2: PMIC-MC33932VW(SOP44), PMIC-MC33932VW_SOP44_:PMIC-MC33932VW(SOP44)
- IC3, IC5: value MC33931EK -> TXB0101DCKR; device MC33931EK:MC33931EK -> TXB0101DCKR:TXB0101DCKR
Connections:
- new net +24V: C18.1, C19.1, J1.14, U1.VPWRA, U1.VPWRA@1, U1.VPWRA@2, U1.VPWRA@3, U1.VPWRA@4, U1.VPWRB, U1.VPWRB@1, U1.VPWRB@2, U1.VPWRB@3, U1.VPWRB@4, U2.VPWRA, U2.VPWRA@1, U2.VPWRA@2, U2.VPWRA@3, U2.VPWRA@4, U2.VPWRB, U2.VPWRB@1, U2.VPWRB@2, U2.VPWRB@3, U2.VPWRB@4
- new net N$15: IC9.A, X1-6.S
- new net N$5: IC3.A, X1-4.S
- new net N$8: IC5.A, X1-5.S
- net +5V: now also C15.1, C17.1, IC3.VCCB, IC5.VCCB, IC9.VCCB, J1.3, X1-7.S
- net RE8: now also IC3.OE, IC5.OE, IC9.OE
- net VDD: now also C14.1, C16.1, IC3.VCCA, IC5.VCCA, IC9.VCCA, J1.2
- net VSS: now also C14.2, C15.2, C16.2, C17.2, C18.2, C19.2, IC3.GND, IC5.GND, IC9.GND, J1.1, J1.13, U1.PGNDA, U1.PGNDA@1, U1.PGNDA@2, U1.PGNDA@3, U1.PGNDB, U1.PGNDB@1, U1.PGNDB@2, U1.PGNDB@3, U2.PGNDA, U2.PGNDA@1, U2.PGNDA@2, U2.PGNDA@3, U2.PGNDB, U2.PGNDB@1, U2.PGNDB@2, U2.PGNDB@3, X1-10.S; no longer IC3.PGND_1, IC3.PGND_2, IC3.PGND_3, IC3.PGND_4, IC5.PGND_1, IC5.PGND_2, IC5.PGND_3, IC5.PGND_4
Other:
- moved on the sheet: IC4

Commit message: up
Connections:
- new net RPB1: IC1.PGEC3/OA1OUT/AN3/C1IN4-/C4IN2-/RPB1/CTED1/RB1, IC3.B
- new net RPC1: IC1.OA3IN-/AN7/CVD7/C3IN1-/C4IN1-/RPC1/RC1, IC5.B
- new net RPC10: IC1.DAC2/AN48/CVD48/RPC10/PMPA14/PSPCS/RC10, IC9.B
Other:
- moved on the sheet: U$1
Changed lines of the file:
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@@
 <?xml version="1.0" encoding="utf-8"?>
 <!DOCTYPE eagle SYSTEM "eagle.dtd">
-<eagle version="9.6.1">
+<eagle version="9.6.2">
 <drawing>
 <settings>
@@
 <attribute name="VALUE" x="208.28" y="-38.1" size="1.778" layer="96"/>
 </instance>
-<instance part="U$1" gate="G$1" x="-66.04" y="-99.06" smashed="yes">
-<attribute name="VALUE" x="-73.67086875" y="-86.3419" size="2.54361875" layer="96"/>
-<attribute name="NAME" x="-83.869" y="-63.402" size="1.7829" layer="95"/>
+<instance part="U$1" gate="G$1" x="-58.42" y="-106.68" smashed="yes">
+<attribute name="VALUE" x="-66.05086875" y="-93.9619" size="2.54361875" layer="96"/>
+<attribute name="NAME" x="-76.249" y="-71.022" size="1.7829" layer="95"/>
 </instance>
 <instance part="U$2" gate="G$1" x="-152.4" y="66.04" smashed="yes">
@@
 <attribute name="VALUE" x="-73.025" y="85.725" size="1.778" layer="96"/>
 </instance>
-<instance part="SUPPLY2" gate="GND" x="-66.04" y="-137.16" smashed="yes">
-<attribute name="VALUE" x="-67.945" y="-140.335" size="1.778" layer="96"/>
-</instance>
-<instance part="P+4" gate="VCC" x="-66.04" y="-58.42" smashed="yes">
-<attribute name="VALUE" x="-68.58" y="-60.96" size="1.778" layer="96" rot="R90"/>
+<instance part="SUPPLY2" gate="GND" x="-58.42" y="-149.86" smashed="yes">
+<attribute name="VALUE" x="-60.325" y="-153.035" size="1.778" layer="96"/>
+</instance>
+<instance part="P+4" gate="VCC" x="-58.42" y="-68.58" smashed="yes">
+<attribute name="VALUE" x="-60.96" y="-71.12" size="1.778" layer="96" rot="R90"/>
 </instance>
 <instance part="C10" gate="G$1" x="-86.36" y="106.68" smashed="yes">
@@
 <pinref part="U$1" gate="G$1" pin="VCC"/>
 <pinref part="P+4" gate="VCC" pin="VCC"/>
-<wire x1="-66.04" y1="-63.5" x2="-66.04" y2="-60.96" width="0.1524" layer="91"/>
 </segment>
 </net>
@@
 <pinref part="U$1" gate="G$1" pin="GND"/>
 <pinref part="SUPPLY2" gate="GND" pin="GND"/>
+<wire x1="-58.42" y1="-142.24" x2="-58.42" y2="-147.32" width="0.1524" layer="91"/>
+<junction x="-58.42" y="-142.24"/>
+<junction x="-58.42" y="-147.32"/>
 </segment>
 <segment>
@@
 <label x="2.54" y="2.54" size="1.778" layer="95"/>
 <junction x="5.08" y="2.54"/>
+<junction x="12.7" y="2.54"/>
 </segment>
 </net>
@@
 <label x="2.54" y="-5.08" size="1.778" layer="95"/>
 <junction x="2.54" y="-5.08"/>
+<junction x="12.7" y="-5.08"/>
 </segment>
 </net>
@@
 <label x="185.42" y="22.86" size="1.778" layer="95"/>
 <junction x="182.88" y="22.86"/>
+<junction x="160.02" y="22.86"/>
 </segment>
 </net>
@@
 <label x="187.96" y="33.02" size="1.778" layer="95"/>
 <junction x="185.42" y="33.02"/>
+<junction x="160.02" y="33.02"/>
 </segment>
 </net>
@@
 </segment>
 </net>
+<net name="RPB1" class="0">
+<segment>
+<pinref part="IC3" gate="G$1" pin="B"/>
+<wire x1="-106.68" y1="-73.66" x2="-91.44" y2="-73.66" width="0.1524" layer="91"/>
+<junction x="-106.68" y="-73.66"/>
+<junction x="-91.44" y="-73.66"/>
+<label x="-91.44" y="-73.66" size="1.778" layer="95"/>
+</segment>
+<segment>
+<pinref part="IC1" gate="G$1" pin="PGEC3/OA1OUT/AN3/C1IN4-/C4IN2-/RPB1/CTED1/RB1"/>
+<wire x1="12.7" y1="-15.24" x2="2.54" y2="-15.24" width="0.1524" layer="91"/>
+<label x="2.54" y="-15.24" size="1.778" layer="95"/>
+<junction x="2.54" y="-15.24"/>
+<junction x="12.7" y="-15.24"/>
+</segment>
+</net>
+<net name="RPC1" class="0">
+<segment>
+<pinref part="IC5" gate="G$1" pin="B"/>
+<wire x1="-106.68" y1="-91.44" x2="-91.44" y2="-91.44" width="0.1524" layer="91"/>
+<junction x="-106.68" y="-91.44"/>
+<junction x="-91.44" y="-91.44"/>
+<label x="-91.44" y="-91.44" size="1.778" layer="95"/>
+</segment>
+<segment>
+<pinref part="IC1" gate="G$1" pin="OA3IN-/AN7/CVD7/C3IN1-/C4IN1-/RPC1/RC1"/>
+<wire x1="73.66" y1="-88.9" x2="73.66" y2="-121.92" width="0.1524" layer="91"/>
+<label x="73.66" y="-121.92" size="1.778" layer="95"/>
+<junction x="73.66" y="-88.9"/>
+<junction x="73.66" y="-121.92"/>
+</segment>
+</net>
+<net name="RPC10" class="0">
+<segment>
+<pinref part="IC9" gate="G$1" pin="B"/>
+<wire x1="-106.68" y1="-109.22" x2="-91.44" y2="-109.22" width="0.1524" layer="91"/>
+<junction x="-106.68" y="-109.22"/>
+<junction x="-91.44" y="-109.22"/>
+<label x="-91.44" y="-109.22" size="1.778" layer="95"/>
+</segment>
+<segment>
+<pinref part="IC1" gate="G$1" pin="DAC2/AN48/CVD48/RPC10/PMPA14/PSPCS/RC10"/>
+<wire x1="160.02" y1="35.56" x2="185.42" y2="35.56" width="0.1524" layer="91"/>
+<label x="185.42" y="35.56" size="1.778" layer="95"/>
+<junction x="160.02" y="35.56"/>
+<junction x="185.42" y="35.56"/>
+</segment>
+</net>

Commit message: up
Parts:
- added C20, C21: 0.1, rcl:C-USC0805
- added X3: 22-23-2101, con-molex:22-23-2101
Connections:
- new net N$17: U$1.IN2, X3-2.S
- new net N$18: U$1.IN3, X3-3.S
- new net N$19: U$1.IN4, X3-4.S
- new net N$20: U$1.IN5, X3-5.S
- new net N$21: U$1.IN6, X3-6.S
- new net N$22: U$1.IN7, X3-7.S
- new net N$23: U$1.IN8, X3-8.S
- new net N$24: U2.OUT1, U2.OUT1@1, U2.OUT1@2
- new net N$25: U2.OUT2, U2.OUT2@1, U2.OUT2@2
- new net N$26: U2.OUT4, U2.OUT4@1, U2.OUT4@2
- new net N$27: U2.OUT3, U2.OUT3@1, U2.OUT3@2
- new net N$4: U$1.IN1, X3-1.S
- new net RD8: IC1.RD8, U$1.EN_L
- new net RPB7: IC1.OA5OUT/AN25/CVD25/C5IN4-/RPB7/SCK1/INT0/RB7, U$1.CH_L
- new net U1O1: J1.12, U1.OUT1, U1.OUT1@1, U1.OUT1@2
- new net U1O2: J1.11, U1.OUT2, U1.OUT2@1, U1.OUT2@2
- new net U1O3: J1.10, U1.OUT3, U1.OUT3@1, U1.OUT3@2
- new net U1O4: J1.9, U1.OUT4, U1.OUT4@1, U1.OUT4@2
- net +24V: now also C20.1, C21.1
- net +5V: now also X3-10.S
- net VSS: now also C20.2, C21.2, X3-9.S
Other:
- moved on the sheet: C18, C19, U$1

Commit message: up
Parts:
- added R10: 1k, rcl:R-US_M0805
- added R4, R7, R8, R9: 100, rcl:R-US_R0805
Connections:
- new net N$28: R4.2, U2.FBA
- new net N$29: R7.1, U2.FBB
- new net N$30: R9.2, U1.FBA
- new net N$31: R8.1, U1.FBB
- new net N$32: R10.2, S1.+
- new net PWM1H: IC1.RPB14/PWM1H/VBUSON1/PMPD6/RB14, U1.IN1
- new net PWM1L: IC1.RPB15/PWM7H/PWM1L/PMPD7/RB15, U1.IN2
- new net PWM2H: IC1.RPB12/PWM2H/PMPD2/RB12, U1.IN3
- new net PWM2L: IC1.RPB13/PWM8H/PWM2L/CTPLS/PMPD3/RB13, U1.IN4
- new net RPG9: IC1.AN16/CVD16/RPG9/PMPA2/RG9, R10.1
- net VSS: now also R4.1, R7.2, R8.2, R9.1, S1.-, U1.EH@1, U1.EH@2, U1.EH@3, U2.EH@1, U2.EH@2, U2.EH@3

Commit message: up
Parts:
- added C22, C23, C24, C25: 0.1, rcl:C-USC0805
- added C26, C27: 22uf, rcl:C-USC0805
- added LED1: led1, led:LEDCHIPLED_1206
- added LED2: led2, led:LEDCHIPLED_1206
- added LED3: led3, led:LEDCHIPLED_1206
- added R11, R12, R13: 1k, rcl:R-US_M0805
- added TP2, TP3, TP5, TP6: TPB1,27, testpad:TPB1,27
Connections:
- new net DERE: IC1.SOSCO/RPB8(4)/RB8(4), IC2.!RE, IC2.DE
- new net IN1: IC1.AN38/CVD38/RD14, U$1.OUT1
- new net IN2: IC1.AN39/CVD39/RD15, U$1.OUT2
- new net IN3: IC1.TDI/DAC3/AN26/CVD26/RPA8/PMPA9/RA8(6), U$1.OUT3
- new net IN4: IC1.FLT15/RPB4/PMPA8/RB4(5), U$1.OUT4
- new net IN5: IC1.AN45/CVD45/RF5, U$1.OUT5
- new net N$33: IC1.TRD2/PMPA20/RG14, R11.2
- new net N$34: IC1.TRD1/RPG12/PMPA21/RG12, R12.2
- new net N$35: IC1.TRD0/PMPA22/RG13, R13.2
- new net N$36: LED1.A, R11.1
- new net N$37: LED2.A, R12.1
- new net N$38: LED3.A, R13.1
- new net N$39: IC2.B, TP5.TP
- new net N$40: IC2.A, TP6.TP
- new net N$41: IC4G$1.V-/1, IC4G$1.V-/2
- new net N$42: IC4G$1.C2-/1, IC4G$1.C2-/2
- new net N$43: IC4G$1.C2+/1, IC4G$1.C2+/2
- new net N$44: IC4G$1.T1OUT, TP2.TP
- new net N$45: IC4G$1.R1IN, TP3.TP
- new net PWM3H: IC1.RPB10/PWM3H/PMPD0/RB10, U2.IN1
- new net PWM3L: IC1.RPB11/PWM9H/PWM3L/PMPD1/RB11, U2.IN2
- new net PWM4H: IC1.TDO/PWM4H/PMPD4/RA10, U2.IN3
- new net PWM4L: IC1.TCK/RPA7/PWM10H/PWM4L/PMPD5/RA7, U2.IN4
- new net RPE0: IC1.AN40/CVD40/RPE0/RE0, U1.EN/!D2, U1.EN/!D4
- new net RPE1: IC1.AN41/CVD41/RPE1/RE1, U2.EN/!D2, U2.EN/!D4
- new net U1FS: IC1.AN12/CVD12/C2IN2-/C5IN2-/FLT5/PMPA11/RE12(6), U1.!SFA, U1.!SFB
- new net U201: J1.8, U2.OUT1, U2.OUT1@1, U2.OUT1@2
- new net U202: J1.7, U2.OUT2, U2.OUT2@1, U2.OUT2@2
- new net U203: J1.6, U2.OUT3, U2.OUT3@1, U2.OUT3@2
- new net U204: J1.5, U2.OUT4, U2.OUT4@1, U2.OUT4@2
- new net U2FS: IC1.AN13/CVD13/C3IN2-/FLT6/PMPA10/RE13(5), U2.!SFA, U2.!SFB
- new net U3RX: IC1.RPC7/PMPA17/RC7, IC4G$1.R1OUT
- new net U3TX: IC1.RPC6/USBID2/PMPA16/RC6, IC4G$1.T1IN
- new net U6RX: IC1.AN47/CVD47/RPA15/RA15, IC2.RXD
- new net U6TX: IC1.OA5IN+/DAC1/AN24/CVD24/C5IN1+/C5IN3-/RPA4/T1CK/T1G/_RA4, IC2.TXD
- net +24V: now also C22.2, C23.1, C24.2, C25.2
- net +3V3: now also C27.1, J1.2; no longer SV2.3
- net +5V: now also C26.1; no longer C15.1, C17.1, C3.1, IC2.VIO, IC3.VCCB, IC5.VCCB, IC6.VCCB, IC7.VCCB, IC8.VCCB, IC9.VCCB, X1-7.S, X1-8.S, X3-10.S
- net N$16: now also IC1.SOSCI/RPC13(4)/RC13(4); no longer IC1.SOSCO/RPB8(4)/RB8(4)
- net N$24: now also C22.1, U1.CCPB; no longer U2.OUT1, U2.OUT1@1, U2.OUT1@2
- net N$25: now also C23.2, U1.CCPA; no longer U2.OUT2, U2.OUT2@1, U2.OUT2@2
- net N$26: now also C24.1, U2.CCPB; no longer U2.OUT4, U2.OUT4@1, U2.OUT4@2
- net N$27: now also C25.1, U2.CCPA; no longer U2.OUT3, U2.OUT3@1, U2.OUT3@2
- net VCC: now also C15.1, C17.1, C3.1, IC2.VIO, IC3.VCCB, IC5.VCCB, IC6.VCCB, IC7.VCCB, IC8.VCCB, IC9.VCCB, SV2.3, X1-7.S, X1-8.S, X3-10.S
- net VDD: no longer J1.2
- net VSS: now also C26.2, C27.2, LED1.C, LED2.C, LED3.C, U1.D1, U1.D3, U2.D1, U2.D3
Other:
- moved on the sheet: C20

Commit message: up
Connections:
- net VCC: no longer U$1.VCC
- net VDD: now also U$1.VCC
Changed lines of the file:
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@@
 <part name="SUPPLY1" library="supply2" library_urn="urn:adsk.eagle:library:372" deviceset="GND" device=""/>
 <part name="SUPPLY2" library="supply2" library_urn="urn:adsk.eagle:library:372" deviceset="GND" device=""/>
-<part name="P+4" library="supply1" library_urn="urn:adsk.eagle:library:371" deviceset="VCC" device=""/>
 <part name="C10" library="rcl" library_urn="urn:adsk.eagle:library:334" deviceset="C-US" device="C0805" package3d_urn="urn:adsk.eagle:package:23617/2" value="0.1"/>
 <part name="C11" library="rcl" library_urn="urn:adsk.eagle:library:334" deviceset="C-US" device="C0805" package3d_urn="urn:adsk.eagle:package:23617/2" value="22uf"/>
@@
 <part name="C27" library="rcl" library_urn="urn:adsk.eagle:library:334" deviceset="C-US" device="C0805" package3d_urn="urn:adsk.eagle:package:23617/2" value="22uf"/>
 <part name="P+22" library="supply1" library_urn="urn:adsk.eagle:library:371" deviceset="VCC" device=""/>
+<part name="VDD19" library="supply1" library_urn="urn:adsk.eagle:library:371" deviceset="VDD" device=""/>
 </parts>
 <sheets>
@@
 </instance>
 <instance part="VDD16" gate="G$1" x="-93.98" y="106.68" smashed="yes" rot="R180">
-<attribute name="VALUE" x="-91.44" y="109.22" size="1.778" layer="96" rot="R270"/>
+<attribute name="VALUE" x="-93.98" y="101.6" size="1.778" layer="96"/>
 </instance>
 <instance part="P+2" gate="VCC" x="-76.2" y="132.08" smashed="yes" rot="R180">
-<attribute name="VALUE" x="-63.5" y="132.08" size="1.778" layer="96" rot="R270"/>
+<attribute name="VALUE" x="-73.66" y="132.08" size="1.778" layer="96"/>
 </instance>
 <instance part="+3V1" gate="G$1" x="-121.92" y="109.22" smashed="yes" rot="R90">
@@
 <instance part="SUPPLY2" gate="GND" x="-48.26" y="-185.42" smashed="yes">
 <attribute name="VALUE" x="-50.165" y="-188.595" size="1.778" layer="96"/>
-</instance>
-<instance part="P+4" gate="VCC" x="-48.26" y="-104.14" smashed="yes">
-<attribute name="VALUE" x="-50.8" y="-106.68" size="1.778" layer="96" rot="R90"/>
 </instance>
 <instance part="C10" gate="G$1" x="-86.36" y="106.68" smashed="yes">
@@
 <instance part="P+22" gate="VCC" x="-15.24" y="-83.82" smashed="yes">
 <attribute name="VALUE" x="-17.78" y="-83.82" size="1.778" layer="96" rot="R90"/>
+</instance>
+<instance part="VDD19" gate="G$1" x="-48.26" y="-104.14" smashed="yes">
+<attribute name="VALUE" x="-50.8" y="-106.68" size="1.778" layer="96" rot="R90"/>
 </instance>
 </instances>
@@
 <wire x1="-86.36" y1="109.22" x2="-93.98" y2="109.22" width="0.1524" layer="91"/>
 <wire x1="-93.98" y1="109.22" x2="-96.52" y2="109.22" width="0.1524" layer="91"/>
+<junction x="-96.52" y="109.22"/>
 </segment>
 <segment>
@@
 <pinref part="VDD14" gate="G$1" pin="VDD"/>
 <junction x="-134.62" y="-104.14"/>
+</segment>
+<segment>
+<pinref part="U$1" gate="G$1" pin="VCC"/>
+<wire x1="-48.26" y1="-109.22" x2="-48.26" y2="-106.68" width="0.1524" layer="91"/>
+<junction x="-48.26" y="-109.22"/>
+<pinref part="VDD19" gate="G$1" pin="VDD"/>
+<junction x="-48.26" y="-106.68"/>
 </segment>
 </net>
@@
 <pinref part="C10" gate="G$1" pin="2"/>
 <pinref part="VSS25" gate="G$1" pin="VSS"/>
+<junction x="-86.36" y="101.6"/>
 </segment>
 <segment>
 <pinref part="C11" gate="G$1" pin="2"/>
 <pinref part="VSS26" gate="G$1" pin="VSS"/>
+<junction x="-76.2" y="101.6"/>
 </segment>
 <segment>
@@
 <pinref part="P+3" gate="1" pin="+5V"/>
 <wire x1="-96.52" y1="134.62" x2="-99.06" y2="134.62" width="0.1524" layer="91"/>
+<junction x="-96.52" y="134.62"/>
+<junction x="-99.06" y="134.62"/>
 </segment>
 <segment>
@@
 <pinref part="F2" gate="G$1" pin="1"/>
 <pinref part="R5" gate="G$1" pin="1"/>
+<junction x="-106.68" y="109.22"/>
 </segment>
 </net>
@@
 <pinref part="F1" gate="G$1" pin="1"/>
 <pinref part="R6" gate="G$1" pin="1"/>
+<junction x="-86.36" y="134.62"/>
 </segment>
 </net>
@@
 <pinref part="R6" gate="G$1" pin="2"/>
 <pinref part="P+2" gate="VCC" pin="VCC"/>
-</segment>
-<segment>
-<pinref part="U$1" gate="G$1" pin="VCC"/>
-<pinref part="P+4" gate="VCC" pin="VCC"/>
-<wire x1="-48.26" y1="-109.22" x2="-48.26" y2="-106.68" width="0.1524" layer="91"/>
-<junction x="-48.26" y="-109.22"/>
+<junction x="-76.2" y="134.62"/>
 </segment>
 <segment>
@@
 <pinref part="+3V1" gate="G$1" pin="+3V3"/>
 <wire x1="-116.84" y1="109.22" x2="-119.38" y2="109.22" width="0.1524" layer="91"/>
-</segment>
-<segment>
+<junction x="-116.84" y="109.22"/>
+<junction x="-119.38" y="109.22"/>
+</segment>
+<segment>

Commit message: up
Parts:
- removed S3: JS202011SCQN, JS202011SCQN_fixed:JS202011SCQN
- removed U$2: IRLML2502TRPBF, IRLML2502TRPBF:IRLML2502TRPBF
- added U3: ULN2803ADW, maxim-10:ULN2803ADW
Connections:
- net GND: now also U3.GND
Changed lines of the file:
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@@
 <part name="IC4" library="maxim" library_urn="urn:adsk.eagle:library:269" deviceset="MAX203ECWP" device="" package3d_urn="urn:adsk.eagle:package:17520/2"/>
 <part name="U$1" library="MAX6818" deviceset="MAX6818" device=""/>
-<part name="U$2" library="IRLML2502TRPBF" deviceset="IRLML2502TRPBF" device=""/>
-<part name="S3" library="JS202011SCQN_fixed" deviceset="JS202011SCQN" device=""/>
 <part name="F1" library="polyfuse-smd_10" deviceset="?" device="1206L" technology="050"/>
 <part name="F2" library="polyfuse-smd_10" deviceset="?" device="1206L" technology="050"/>
@@
 <part name="P+22" library="supply1" library_urn="urn:adsk.eagle:library:371" deviceset="VCC" device=""/>
 <part name="VDD19" library="supply1" library_urn="urn:adsk.eagle:library:371" deviceset="VDD" device=""/>
+<part name="U3" library="maxim-10" deviceset="ULN2803ADW" device=""/>
+<part name="SUPPLY3" library="supply2" library_urn="urn:adsk.eagle:library:372" deviceset="GND" device=""/>
 </parts>
 <sheets>
@@
 <attribute name="NAME" x="-66.089" y="-109.122" size="1.7829" layer="95"/>
 </instance>
-<instance part="U$2" gate="G$1" x="-152.4" y="66.04" smashed="yes">
-<attribute name="VALUE" x="-163.861" y="66.04" size="1.78281875" layer="96"/>
-<attribute name="NAME" x="-163.8527" y="68.585059375" size="1.78153125" layer="95"/>
-</instance>
-<instance part="S3" gate="G$1" x="-119.38" y="68.58" smashed="yes">
-<attribute name="NAME" x="-134.6422" y="71.1237" size="1.27185" layer="95"/>
-<attribute name="VALUE" x="-134.6312" y="63.496259375" size="1.270940625" layer="96"/>
-</instance>
 <instance part="F1" gate="G$1" x="-91.44" y="134.62" smashed="yes">
 <attribute name="NAME" x="-95.25" y="137.16" size="1.778" layer="95"/>
@@
 <instance part="VDD19" gate="G$1" x="-48.26" y="-104.14" smashed="yes">
 <attribute name="VALUE" x="-50.8" y="-106.68" size="1.778" layer="96" rot="R90"/>
+</instance>
+<instance part="U3" gate="A" x="-111.76" y="40.64" smashed="yes">
+<attribute name="NAME" x="-116.94811875" y="55.7466" size="2.034559375" layer="95" ratio="5" rot="SR0"/>
+<attribute name="VALUE" x="-115.70293125" y="15.3798" size="2.035059375" layer="96" ratio="5" rot="SR0"/>
+</instance>
+<instance part="SUPPLY3" gate="GND" x="-129.54" y="22.86" smashed="yes">
+<attribute name="VALUE" x="-131.445" y="19.685" size="1.778" layer="96"/>
 </instance>
 </instances>
@@
 <junction x="-53.34" y="91.44"/>
 </segment>
+<segment>
+<pinref part="U3" gate="A" pin="GND"/>
+<pinref part="SUPPLY3" gate="GND" pin="GND"/>
+<junction x="-129.54" y="25.4"/>
+</segment>
 </net>

Commit message: up
Parts:
- added DO: 22-23-2101, con-molex:22-23-2101
- added R14: 0, rcl:R-US_M0805
- added RS485: 22-23-2051, con-molex:22-23-2051
- added TP7: TPB1,27, testpad:TPB1,27
- renumbered X3 to DIN
Connections:
- new net N$46: DO-1.S, U3.1C
- new net N$47: DO-2.S, U3.2C
- new net N$48: DO-3.S, U3.3C
- new net N$49: DO-4.S, U3.4C
- new net N$50: DO-5.S, U3.5C
- new net N$51: DO-6.S, U3.6C
- new net N$52: DO-7.S, U3.7C
- new net N$53: DO-8.S, U3.8C
- new net N$54: R14.1, U3.COM
- net +24V: now also DO-10.S, R14.2
- net GND: now also DO-9.S
- net N$39: now also RS485-2.S
- net N$40: now also RS485-3.S
- net VCC: now also RS485-5.S
- net VSS: now also RS485-1.S, RS485-4.S, TP7.TP
