File: pic32mk.sch (EAGLE design)
At the start: 85 parts, among them IC1 PIC32MK1024MCF100-I_PT, IC2 ADM3095EBRZ, IC3 TXB0101DCKR, IC4 MAX203ECWP, IC5 TXB0101DCKR, IC6 TXB0101DCKR, IC7 TXB0101DCKR, IC8 TXB0101DCKR, IC9 TXB0101DCKR, J1 1-1586043-4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

Commit message: up
Connections:
- net VCC: no longer SV2.3
- net VDD: now also SV2.2
- net VSS: now also SV2.3; no longer SV2.2
Other:
- note added: "change to VDD from VSS"
- note added: "change to VSS from orig VCC"
Changed lines of the file:
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@@
 <part name="VSS26" library="supply1" library_urn="urn:adsk.eagle:library:371" deviceset="VSS" device=""/>
 <part name="SV2" library="con-lstb" library_urn="urn:adsk.eagle:library:162" deviceset="MA06-1" device="" package3d_urn="urn:adsk.eagle:package:8340/1" value="ICSP2"/>
-<part name="VSS28" library="supply1" library_urn="urn:adsk.eagle:library:371" deviceset="VSS" device=""/>
 <part name="OS2" library="IQD-Frequency-Products" library_urn="urn:adsk.eagle:library:90" deviceset="OSC-OE" device="-IQXO-793" package3d_urn="urn:adsk.eagle:package:3371/1"/>
 <part name="C12" library="rcl" library_urn="urn:adsk.eagle:library:334" deviceset="C-US" device="C0805" package3d_urn="urn:adsk.eagle:package:23617/2" value="0.1"/>
@@
 <part name="+3V2" library="supply1" library_urn="urn:adsk.eagle:library:371" deviceset="+3V3" device=""/>
 <part name="C27" library="rcl" library_urn="urn:adsk.eagle:library:334" deviceset="C-US" device="C0805" package3d_urn="urn:adsk.eagle:package:23617/2" value="22uf"/>
-<part name="P+22" library="supply1" library_urn="urn:adsk.eagle:library:371" deviceset="VCC" device=""/>
 <part name="VDD19" library="supply1" library_urn="urn:adsk.eagle:library:371" deviceset="VDD" device=""/>
 <part name="U3" library="maxim-10" deviceset="ULN2803ADW" device=""/>
@@
 <part name="VDD20" library="supply1" library_urn="urn:adsk.eagle:library:371" deviceset="VDD" device=""/>
 <part name="P+33" library="supply1" library_urn="urn:adsk.eagle:library:371" deviceset="VCC" device=""/>
+<part name="VSS68" library="supply1" library_urn="urn:adsk.eagle:library:371" deviceset="VSS" device=""/>
+<part name="VDD25" library="supply1" library_urn="urn:adsk.eagle:library:371" deviceset="VDD" device=""/>
 </parts>
 <sheets>
 <sheet>
 <plain>
+<text x="-12.7" y="-109.22" size="1.778" layer="91">change to VDD from VSS</text>
+<text x="-12.7" y="-86.36" size="1.778" layer="91">change to VSS from orig VCC</text>
 </plain>
 <instances>
@@
 <attribute name="NAME" x="-31.75" y="-88.138" size="1.778" layer="95"/>
 </instance>
-<instance part="VSS28" gate="G$1" x="-15.24" y="-111.76" smashed="yes">
-<attribute name="VALUE" x="-17.78" y="-116.84" size="1.778" layer="96" rot="R90"/>
-</instance>
 <instance part="OS2" gate="A" x="238.76" y="45.72" smashed="yes" rot="R180">
 <attribute name="NAME" x="246.38" y="37.465" size="1.778" layer="95" rot="R180"/>
@@
 <attribute name="VALUE" x="54.229" y="-130.556" size="1.778" layer="96" rot="R270"/>
 </instance>
-<instance part="P+22" gate="VCC" x="-15.24" y="-83.82" smashed="yes">
-<attribute name="VALUE" x="-17.78" y="-83.82" size="1.778" layer="96" rot="R90"/>
-</instance>
 <instance part="VDD19" gate="G$1" x="-48.26" y="-104.14" smashed="yes">
 <attribute name="VALUE" x="-50.8" y="-106.68" size="1.778" layer="96" rot="R90"/>
@@
 <attribute name="VALUE" x="40.64" y="-132.08" size="1.778" layer="96" rot="R180"/>
 </instance>
-<instance part="P+32" gate="1" x="27.94" y="-162.56" smashed="yes">
-<attribute name="VALUE" x="25.4" y="-167.64" size="1.778" layer="96" rot="R90"/>
+<instance part="P+32" gate="1" x="33.02" y="-162.56" smashed="yes">
+<attribute name="VALUE" x="30.48" y="-167.64" size="1.778" layer="96" rot="R90"/>
 </instance>
 <instance part="C28" gate="G$1" x="17.78" y="-167.64" smashed="yes">
@@
 <instance part="P+33" gate="VCC" x="147.32" y="132.08" smashed="yes" rot="R270">
 <attribute name="VALUE" x="147.32" y="134.62" size="1.778" layer="96" rot="R90"/>
+</instance>
+<instance part="VSS68" gate="G$1" x="-15.24" y="-83.82" smashed="yes" rot="R180">
+<attribute name="VALUE" x="-12.7" y="-78.74" size="1.778" layer="96" rot="R270"/>
+</instance>
+<instance part="VDD25" gate="G$1" x="-15.24" y="-111.76" smashed="yes" rot="R180">
+<attribute name="VALUE" x="-12.7" y="-111.76" size="1.778" layer="96" rot="R270"/>
 </instance>
 </instances>
@@
 <pinref part="VDD20" gate="G$1" pin="VDD"/>
 </segment>
+<segment>
+<pinref part="SV2" gate="1" pin="2"/>
+<wire x1="-22.86" y1="-101.6" x2="-15.24" y2="-101.6" width="0.1524" layer="91"/>
+<wire x1="-15.24" y1="-101.6" x2="-15.24" y2="-109.22" width="0.1524" layer="91"/>
+<junction x="-22.86" y="-101.6"/>
+<pinref part="VDD25" gate="G$1" pin="VDD"/>
+<junction x="-15.24" y="-109.22"/>
+</segment>
 </net>
 <net name="VSS" class="0">
@@
 </segment>
 <segment>
-<pinref part="SV2" gate="1" pin="2"/>
-<wire x1="-22.86" y1="-101.6" x2="-15.24" y2="-101.6" width="0.1524" layer="91"/>
-<wire x1="-15.24" y1="-101.6" x2="-15.24" y2="-109.22" width="0.1524" layer="91"/>
-<pinref part="VSS28" gate="G$1" pin="VSS"/>
-<junction x="-15.24" y="-109.22"/>
-<junction x="-22.86" y="-101.6"/>
-</segment>
-<segment>
 <pinref part="OS2" gate="A" pin="VSS"/>
 <pinref part="VSS29" gate="G$1" pin="VSS"/>
@@
 <pinref part="VSS67" gate="G$1" pin="VSS"/>
 </segment>
+<segment>
+<pinref part="SV2" gate="1" pin="3"/>
+<wire x1="-22.86" y1="-99.06" x2="-15.24" y2="-99.06" width="0.1524" layer="91"/>
+<wire x1="-15.24" y1="-99.06" x2="-15.24" y2="-86.36" width="0.1524" layer="91"/>
+<junction x="-22.86" y="-99.06"/>
+<pinref part="VSS68" gate="G$1" pin="VSS"/>
+<junction x="-15.24" y="-86.36"/>
+</segment>
 </net>
 <net name="+5V" class="0">
@@
 <wire x1="20.32" y1="-165.1" x2="22.86" y2="-165.1" width="0.1524" layer="91"/>
 <pinref part="P+32" gate="1" pin="+5V"/>
-<junction x="27.94" y="-165.1"/>
+<junction x="33.02" y="-165.1"/>
 <pinref part="C28" gate="G$1" pin="1"/>
 <pinref part="C29" gate="G$1" pin="1"/>
-<wire x1="22.86" y1="-165.1" x2="27.94" y2="-165.1" width="0.1524" layer="91"/>
+<wire x1="22.86" y1="-165.1" x2="33.02" y2="-165.1" width="0.1524" layer="91"/>
 <junction x="22.86" y="-165.1"/>
 </segment>
@@
 </segment>
 <segment>
-<pinref part="SV2" gate="1" pin="3"/>
-<wire x1="-22.86" y1="-99.06" x2="-15.24" y2="-99.06" width="0.1524" layer="91"/>
-<wire x1="-15.24" y1="-99.06" x2="-15.24" y2="-86.36" width="0.1524" layer="91"/>
-<junction x="-22.86" y="-99.06"/>
-<pinref part="P+22" gate="VCC" pin="VCC"/>
-<junction x="-15.24" y="-86.36"/>
-</segment>
-<segment>

Commit message: up
Connections:
- net VCC: now also C14.1, C16.1, IC3.VCCA, IC5.VCCA, IC6.VCCA, IC7.VCCA, IC8.VCCA, IC9.VCCA; no longer C15.1, C17.1, IC3.VCCB, IC5.VCCB, IC6.VCCB, IC7.VCCB, IC8.VCCB, IC9.VCCB
- net VDD: now also C15.1, C17.1, IC3.VCCB, IC5.VCCB, IC6.VCCB, IC7.VCCB, IC8.VCCB, IC9.VCCB; no longer C14.1, C16.1, IC3.VCCA, IC5.VCCA, IC6.VCCA, IC7.VCCA, IC8.VCCA, IC9.VCCA

Commit message: up
Other:
- note added: "A"
- note added: "B"
- note added: "Index"
Changed lines of the file:
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@@
 <text x="-12.7" y="-109.22" size="1.778" layer="91">change to VDD from VSS</text>
 <text x="-12.7" y="-86.36" size="1.778" layer="91">change to VSS from orig VCC</text>
+<text x="-132.08" y="-40.64" size="1.778" layer="91">A</text>
+<text x="-132.08" y="-50.8" size="1.778" layer="91">B</text>
+<text x="-132.08" y="-35.56" size="1.778" layer="91">Index</text>
+<text x="-137.16" y="-33.02" size="1.778" layer="91">Index</text>
+<text x="-137.16" y="-30.48" size="1.778" layer="91">A</text>
+<text x="-137.16" y="-27.94" size="1.778" layer="91">B</text>
 </plain>
 <instances>

Commit message: up
Connections:
- net N$10: now also IC8.B; no longer IC8.A
- net N$11: now also IC6.B; no longer IC6.A
- net N$12: now also IC7.B; no longer IC7.A
- net N$15: now also IC9.B; no longer IC9.A
- net N$5: now also IC3.B; no longer IC3.A
- net N$8: now also IC5.B; no longer IC5.A
- net RPA0: now also IC8.A; no longer IC8.B
- net RPA14: now also IC6.A; no longer IC6.B
- net RPB1: now also IC3.A; no longer IC3.B
- net RPB6: now also IC7.A; no longer IC7.B
- net RPC1: now also IC5.A; no longer IC5.B
- net RPC10: now also IC9.A; no longer IC9.B
Changed lines of the file:
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@@
 <net name="RPA14" class="0">
 <segment>
-<pinref part="IC6" gate="G$1" pin="B"/>
-<wire x1="-60.96" y1="-35.56" x2="-45.72" y2="-35.56" width="0.1524" layer="91"/>
 <label x="-45.72" y="-35.56" size="1.778" layer="95"/>
-<junction x="-60.96" y="-35.56"/>
 <junction x="-45.72" y="-35.56"/>
+<wire x1="-53.34" y1="-35.56" x2="-45.72" y2="-35.56" width="0.1524" layer="91"/>
+<pinref part="IC6" gate="G$1" pin="A"/>
+<wire x1="-88.9" y1="-35.56" x2="-88.9" y2="-38.1" width="0.1524" layer="91"/>
+<wire x1="-88.9" y1="-38.1" x2="-53.34" y2="-38.1" width="0.1524" layer="91"/>
+<wire x1="-53.34" y1="-38.1" x2="-53.34" y2="-35.56" width="0.1524" layer="91"/>
+<junction x="-88.9" y="-35.56"/>
 </segment>
 <segment>
@@
 <net name="RPB6" class="0">
 <segment>
-<pinref part="IC7" gate="G$1" pin="B"/>
-<wire x1="-60.96" y1="-20.32" x2="-53.34" y2="-20.32" width="0.1524" layer="91"/>
-<wire x1="-53.34" y1="-20.32" x2="-53.34" y2="-12.7" width="0.1524" layer="91"/>
+<wire x1="-53.34" y1="-25.4" x2="-53.34" y2="-12.7" width="0.1524" layer="91"/>
 <wire x1="-53.34" y1="-12.7" x2="-35.56" y2="-12.7" width="0.1524" layer="91"/>
 <label x="-35.56" y="-12.7" size="1.778" layer="95"/>
-<junction x="-60.96" y="-20.32"/>
 <junction x="-35.56" y="-12.7"/>
+<junction x="-53.34" y="-12.7"/>
+<pinref part="IC7" gate="G$1" pin="A"/>
+<wire x1="-88.9" y1="-20.32" x2="-88.9" y2="-25.4" width="0.1524" layer="91"/>
+<wire x1="-88.9" y1="-25.4" x2="-53.34" y2="-25.4" width="0.1524" layer="91"/>
+<junction x="-88.9" y="-20.32"/>
 </segment>
 <segment>
@@
 <wire x1="-137.16" y1="-40.64" x2="-139.7" y2="-40.64" width="0.1524" layer="91"/>
 <junction x="-139.7" y="-40.64"/>
-<pinref part="IC8" gate="G$1" pin="A"/>
-<wire x1="-88.9" y1="-50.8" x2="-137.16" y2="-50.8" width="0.1524" layer="91"/>
-<junction x="-88.9" y="-50.8"/>
+<wire x1="-99.06" y1="-50.8" x2="-137.16" y2="-50.8" width="0.1524" layer="91"/>
+<pinref part="IC8" gate="G$1" pin="B"/>
+<wire x1="-60.96" y1="-50.8" x2="-60.96" y2="-58.42" width="0.1524" layer="91"/>
+<wire x1="-60.96" y1="-58.42" x2="-99.06" y2="-58.42" width="0.1524" layer="91"/>
+<wire x1="-99.06" y1="-58.42" x2="-99.06" y2="-50.8" width="0.1524" layer="91"/>
+<junction x="-60.96" y="-50.8"/>
 </segment>
 </net>
 <net name="N$11" class="0">
 <segment>
-<pinref part="IC6" gate="G$1" pin="A"/>
-<wire x1="-88.9" y1="-35.56" x2="-93.98" y2="-35.56" width="0.1524" layer="91"/>
-<wire x1="-93.98" y1="-35.56" x2="-93.98" y2="-40.64" width="0.1524" layer="91"/>
-<wire x1="-93.98" y1="-40.64" x2="-134.62" y2="-40.64" width="0.1524" layer="91"/>
 <wire x1="-134.62" y1="-40.64" x2="-134.62" y2="-38.1" width="0.1524" layer="91"/>
 <pinref part="X1" gate="-2" pin="S"/>
 <wire x1="-139.7" y1="-38.1" x2="-134.62" y2="-38.1" width="0.1524" layer="91"/>
-<junction x="-88.9" y="-35.56"/>
 <junction x="-139.7" y="-38.1"/>
+<pinref part="IC6" gate="G$1" pin="B"/>
+<wire x1="-60.96" y1="-35.56" x2="-60.96" y2="-40.64" width="0.1524" layer="91"/>
+<wire x1="-60.96" y1="-40.64" x2="-134.62" y2="-40.64" width="0.1524" layer="91"/>
+<junction x="-60.96" y="-35.56"/>
 </segment>
 </net>
 <net name="N$12" class="0">
 <segment>
-<pinref part="IC7" gate="G$1" pin="A"/>
-<wire x1="-88.9" y1="-20.32" x2="-109.22" y2="-20.32" width="0.1524" layer="91"/>
-<wire x1="-109.22" y1="-20.32" x2="-109.22" y2="-35.56" width="0.1524" layer="91"/>
 <pinref part="X1" gate="-3" pin="S"/>
+<wire x1="-109.22" y1="-22.86" x2="-109.22" y2="-35.56" width="0.1524" layer="91"/>
 <wire x1="-109.22" y1="-35.56" x2="-139.7" y2="-35.56" width="0.1524" layer="91"/>
-<junction x="-88.9" y="-20.32"/>
 <junction x="-139.7" y="-35.56"/>
+<pinref part="IC7" gate="G$1" pin="B"/>
+<wire x1="-60.96" y1="-20.32" x2="-60.96" y2="-22.86" width="0.1524" layer="91"/>
+<wire x1="-60.96" y1="-22.86" x2="-109.22" y2="-22.86" width="0.1524" layer="91"/>
+<junction x="-60.96" y="-20.32"/>
 </segment>
 </net>
 <net name="N$5" class="0">
 <segment>
-<pinref part="IC3" gate="G$1" pin="A"/>
-<wire x1="-134.62" y1="-73.66" x2="-154.94" y2="-73.66" width="0.1524" layer="91"/>
-<wire x1="-154.94" y1="-73.66" x2="-154.94" y2="-33.02" width="0.1524" layer="91"/>
+<wire x1="-154.94" y1="-76.2" x2="-154.94" y2="-33.02" width="0.1524" layer="91"/>
 <pinref part="X1" gate="-4" pin="S"/>
 <wire x1="-154.94" y1="-33.02" x2="-139.7" y2="-33.02" width="0.1524" layer="91"/>
 <junction x="-139.7" y="-33.02"/>
-<junction x="-134.62" y="-73.66"/>
+<pinref part="IC3" gate="G$1" pin="B"/>
+<wire x1="-106.68" y1="-73.66" x2="-106.68" y2="-76.2" width="0.1524" layer="91"/>
+<wire x1="-106.68" y1="-76.2" x2="-154.94" y2="-76.2" width="0.1524" layer="91"/>
+<junction x="-106.68" y="-73.66"/>
 </segment>
 </net>
 <net name="N$8" class="0">
 <segment>
-<pinref part="IC5" gate="G$1" pin="A"/>
-<wire x1="-134.62" y1="-91.44" x2="-157.48" y2="-91.44" width="0.1524" layer="91"/>
-<wire x1="-157.48" y1="-91.44" x2="-157.48" y2="-30.48" width="0.1524" layer="91"/>
+<wire x1="-157.48" y1="-96.52" x2="-157.48" y2="-30.48" width="0.1524" layer="91"/>
 <pinref part="X1" gate="-5" pin="S"/>
 <wire x1="-157.48" y1="-30.48" x2="-139.7" y2="-30.48" width="0.1524" layer="91"/>
 <junction x="-139.7" y="-30.48"/>
-<junction x="-134.62" y="-91.44"/>
+<pinref part="IC5" gate="G$1" pin="B"/>
+<wire x1="-106.68" y1="-91.44" x2="-106.68" y2="-96.52" width="0.1524" layer="91"/>
+<wire x1="-106.68" y1="-96.52" x2="-157.48" y2="-96.52" width="0.1524" layer="91"/>
+<junction x="-106.68" y="-91.44"/>
 </segment>
 </net>
 <net name="N$15" class="0">
 <segment>
-<wire x1="-160.02" y1="-109.22" x2="-160.02" y2="-27.94" width="0.1524" layer="91"/>
+<wire x1="-160.02" y1="-114.3" x2="-160.02" y2="-27.94" width="0.1524" layer="91"/>
 <pinref part="X1" gate="-6" pin="S"/>
 <wire x1="-160.02" y1="-27.94" x2="-139.7" y2="-27.94" width="0.1524" layer="91"/>
 <junction x="-139.7" y="-27.94"/>
-<pinref part="IC9" gate="G$1" pin="A"/>
-<wire x1="-134.62" y1="-109.22" x2="-160.02" y2="-109.22" width="0.1524" layer="91"/>
-<junction x="-134.62" y="-109.22"/>
+<pinref part="IC9" gate="G$1" pin="B"/>
+<wire x1="-106.68" y1="-109.22" x2="-106.68" y2="-114.3" width="0.1524" layer="91"/>
+<wire x1="-106.68" y1="-114.3" x2="-160.02" y2="-114.3" width="0.1524" layer="91"/>
+<junction x="-106.68" y="-109.22"/>
 </segment>
 </net>
@@
 <net name="RPB1" class="0">
 <segment>
-<pinref part="IC3" gate="G$1" pin="B"/>
-<wire x1="-106.68" y1="-73.66" x2="-91.44" y2="-73.66" width="0.1524" layer="91"/>
-<junction x="-106.68" y="-73.66"/>
 <junction x="-91.44" y="-73.66"/>
 <label x="-91.44" y="-73.66" size="1.778" layer="95"/>
+<wire x1="-96.52" y1="-73.66" x2="-91.44" y2="-73.66" width="0.1524" layer="91"/>
+<pinref part="IC3" gate="G$1" pin="A"/>
+<wire x1="-134.62" y1="-73.66" x2="-134.62" y2="-81.28" width="0.1524" layer="91"/>
+<wire x1="-134.62" y1="-81.28" x2="-96.52" y2="-81.28" width="0.1524" layer="91"/>
+<wire x1="-96.52" y1="-81.28" x2="-96.52" y2="-73.66" width="0.1524" layer="91"/>
+<junction x="-134.62" y="-73.66"/>
 </segment>
 <segment>
@@
 <net name="RPC1" class="0">
 <segment>
-<pinref part="IC5" gate="G$1" pin="B"/>
-<wire x1="-106.68" y1="-91.44" x2="-91.44" y2="-91.44" width="0.1524" layer="91"/>
-<junction x="-106.68" y="-91.44"/>
 <junction x="-91.44" y="-91.44"/>
 <label x="-91.44" y="-91.44" size="1.778" layer="95"/>
+<wire x1="-99.06" y1="-91.44" x2="-91.44" y2="-91.44" width="0.1524" layer="91"/>
+<pinref part="IC5" gate="G$1" pin="A"/>
+<wire x1="-134.62" y1="-91.44" x2="-134.62" y2="-93.98" width="0.1524" layer="91"/>
+<wire x1="-134.62" y1="-93.98" x2="-99.06" y2="-93.98" width="0.1524" layer="91"/>
+<wire x1="-99.06" y1="-93.98" x2="-99.06" y2="-91.44" width="0.1524" layer="91"/>
+<junction x="-134.62" y="-91.44"/>
 </segment>
 <segment>
@@
 <net name="RPC10" class="0">
 <segment>
-<pinref part="IC9" gate="G$1" pin="B"/>
-<wire x1="-106.68" y1="-109.22" x2="-91.44" y2="-109.22" width="0.1524" layer="91"/>
-<junction x="-106.68" y="-109.22"/>
 <junction x="-91.44" y="-109.22"/>
 <label x="-91.44" y="-109.22" size="1.778" layer="95"/>
+<wire x1="-96.52" y1="-109.22" x2="-91.44" y2="-109.22" width="0.1524" layer="91"/>
+<pinref part="IC9" gate="G$1" pin="A"/>
+<wire x1="-134.62" y1="-109.22" x2="-134.62" y2="-116.84" width="0.1524" layer="91"/>
+<wire x1="-134.62" y1="-116.84" x2="-96.52" y2="-116.84" width="0.1524" layer="91"/>
+<wire x1="-96.52" y1="-116.84" x2="-96.52" y2="-109.22" width="0.1524" layer="91"/>
+<junction x="-134.62" y="-109.22"/>
 </segment>
 <segment>
@@
 </segment>
 <segment>
-<pinref part="IC8" gate="G$1" pin="B"/>
-<wire x1="-60.96" y1="-50.8" x2="-48.26" y2="-50.8" width="0.1524" layer="91"/>
 <label x="-50.8" y="-50.8" size="1.778" layer="95"/>
-<junction x="-60.96" y="-50.8"/>
 <junction x="-48.26" y="-50.8"/>
-</segment>
-</net>
+<wire x1="-53.34" y1="-50.8" x2="-48.26" y2="-50.8" width="0.1524" layer="91"/>
+<wire x1="-53.34" y1="-50.8" x2="-53.34" y2="-60.96" width="0.1524" layer="91"/>
+<pinref part="IC8" gate="G$1" pin="A"/>
+<wire x1="-88.9" y1="-50.8" x2="-88.9" y2="-60.96" width="0.1524" layer="91"/>
+<wire x1="-53.34" y1="-60.96" x2="-88.9" y2="-60.96" width="0.1524" layer="91"/>
+<junction x="-88.9" y="-50.8"/>
+</segment>
+</net>

Commit message: up
Connections:
- net RC11: now also SPI-9.S
- net RC2: now also SPI-6.S
- net VDD: now also SPI-10.S
Changed lines of the file:
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@@
 <part name="P+6" library="supply1" library_urn="urn:adsk.eagle:library:371" deviceset="VCC" device=""/>
 <part name="VDD9" library="supply1" library_urn="urn:adsk.eagle:library:371" deviceset="VDD" device=""/>
+<part name="VDD24" library="supply1" library_urn="urn:adsk.eagle:library:371" deviceset="VDD" device=""/>
 </parts>
 <sheets>
@@
 <attribute name="VALUE" x="-55.88" y="-7.62" size="1.778" layer="96" rot="R90"/>
 </instance>
+<instance part="VDD24" gate="G$1" x="-104.14" y="60.96" smashed="yes" rot="R180">
+<attribute name="VALUE" x="-104.14" y="55.88" size="1.778" layer="96"/>
+</instance>
 </instances>
 <busses>
@@
 <junction x="-60.96" y="-15.24"/>
 </segment>
+<segment>
+<pinref part="SPI" gate="-10" pin="S"/>
+<pinref part="VDD24" gate="G$1" pin="VDD"/>
+<junction x="-104.14" y="63.5"/>
+</segment>
 </net>
 <net name="VSS" class="0">
@@
 <junction x="114.3" y="-162.56"/>
 </segment>
+<segment>
+<pinref part="SPI" gate="-6" pin="S"/>
+<junction x="-104.14" y="73.66"/>
+<label x="-111.76" y="73.66" size="1.778" layer="95"/>
+</segment>
 </net>
 <net name="RC11" class="0">
@@
 <junction x="114.3" y="-160.02"/>
 </segment>
+<segment>
+<pinref part="SPI" gate="-9" pin="S"/>
+<junction x="-104.14" y="66.04"/>
+<label x="-111.76" y="66.04" size="1.778" layer="95"/>
+</segment>
 </net>
