File: pic32mk.sch (EAGLE design)
At the start: 85 parts, among them IC1 PIC32MK1024MCF100-I_PT, IC2 ADM3095EBRZ, IC3 TXB0101DCKR, IC4 MAX203ECWP, IC5 TXB0101DCKR, IC6 TXB0101DCKR, IC7 TXB0101DCKR, IC8 TXB0101DCKR, IC9 TXB0101DCKR, J1 1-1586043-4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

Commit message: up
Connections:
- removed net DERE: IC1.SOSCO/RPB8(4)/RB8(4), IC2.!RE, IC2.DE
- removed net N$16: IC1.SOSCI/RPC13(4)/RC13(4), OS2.OUT
- new net N$1: IC1.SOSCO/RPB8(4)/RB8(4), OS2.OUT
- new net SOSCI: IC1.SOSCI/RPC13(4)/RC13(4)
- net RG11: now also IC2.!RE, IC2.DE
Other:
- moved on the sheet: C3
Changed lines of the file:
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@@
 <attribute name="VALUE" x="258.064" y="19.431" size="1.778" layer="96" rot="R180"/>
 </instance>
-<instance part="C3" gate="G$1" x="185.42" y="-60.96" smashed="yes">
-<attribute name="NAME" x="186.436" y="-60.325" size="1.778" layer="95"/>
-<attribute name="VALUE" x="186.436" y="-65.151" size="1.778" layer="96"/>
+<instance part="C3" gate="G$1" x="180.34" y="-60.96" smashed="yes">
+<attribute name="NAME" x="176.276" y="-60.325" size="1.778" layer="95"/>
+<attribute name="VALUE" x="181.356" y="-65.151" size="1.778" layer="96"/>
 </instance>
 <instance part="C4" gate="G$1" x="195.58" y="-53.34" smashed="yes" rot="R180">
@@
 <attribute name="VALUE" x="194.564" y="-49.149" size="1.778" layer="96" rot="R180"/>
 </instance>
-<instance part="VSS12" gate="G$1" x="185.42" y="-68.58" smashed="yes">
-<attribute name="VALUE" x="182.88" y="-73.66" size="1.778" layer="96" rot="R90"/>
+<instance part="VSS12" gate="G$1" x="180.34" y="-68.58" smashed="yes">
+<attribute name="VALUE" x="177.8" y="-73.66" size="1.778" layer="96" rot="R90"/>
 </instance>
 <instance part="VSS13" gate="G$1" x="195.58" y="-45.72" smashed="yes" rot="R180">
@@
 <pinref part="C3" gate="G$1" pin="2"/>
 <pinref part="VSS12" gate="G$1" pin="VSS"/>
-<junction x="185.42" y="-66.04"/>
+<junction x="180.34" y="-66.04"/>
 </segment>
 <segment>
@@
 <segment>
 <pinref part="IC2" gate="G$1" pin="VIO"/>
-<wire x1="203.2" y1="-58.42" x2="185.42" y2="-58.42" width="0.1524" layer="91"/>
+<wire x1="203.2" y1="-58.42" x2="180.34" y2="-58.42" width="0.1524" layer="91"/>
 <junction x="203.2" y="-58.42"/>
 <pinref part="C3" gate="G$1" pin="1"/>
-<wire x1="185.42" y1="-58.42" x2="175.26" y2="-58.42" width="0.1524" layer="91"/>
-<junction x="185.42" y="-58.42"/>
+<wire x1="180.34" y1="-58.42" x2="175.26" y2="-58.42" width="0.1524" layer="91"/>
+<junction x="180.34" y="-58.42"/>
 <pinref part="P+11" gate="VCC" pin="VCC"/>
 <junction x="175.26" y="-58.42"/>
@@
 </segment>
 </net>
-<net name="N$16" class="0">
-<segment>
-<pinref part="OS2" gate="A" pin="OUT"/>
-<wire x1="226.06" y1="43.18" x2="226.06" y2="45.72" width="0.1524" layer="91"/>
-<pinref part="IC1" gate="G$1" pin="SOSCI/RPC13(4)/RC13(4)"/>
-<wire x1="160.02" y1="40.64" x2="218.44" y2="40.64" width="0.1524" layer="91"/>
-<wire x1="218.44" y1="40.64" x2="218.44" y2="43.18" width="0.1524" layer="91"/>
-<wire x1="218.44" y1="43.18" x2="226.06" y2="43.18" width="0.1524" layer="91"/>
-<junction x="160.02" y="40.64"/>
-<junction x="226.06" y="45.72"/>
-</segment>
-</net>
 <net name="RE8" class="0">
 <segment>
@@
 </segment>
 </net>
-<net name="DERE" class="0">
-<segment>
-<pinref part="IC2" gate="G$1" pin="!RE"/>
-<pinref part="IC2" gate="G$1" pin="DE"/>
-<wire x1="203.2" y1="-66.04" x2="203.2" y2="-63.5" width="0.1524" layer="91"/>
-<wire x1="203.2" y1="-63.5" x2="195.58" y2="-63.5" width="0.1524" layer="91"/>
-<junction x="195.58" y="-63.5"/>
-<junction x="203.2" y="-63.5"/>
-<junction x="203.2" y="-66.04"/>
-<label x="190.5" y="-66.04" size="1.778" layer="95"/>
-</segment>
-<segment>
-<pinref part="IC1" gate="G$1" pin="SOSCO/RPB8(4)/RB8(4)"/>
-<wire x1="160.02" y1="43.18" x2="185.42" y2="43.18" width="0.1524" layer="91"/>
-<junction x="160.02" y="43.18"/>
-<junction x="185.42" y="43.18"/>
-<label x="187.96" y="43.18" size="1.778" layer="95"/>
-</segment>
-</net>
 <net name="IN5" class="0">
 <segment>
@@
 <label x="137.16" y="-157.48" size="1.778" layer="95"/>
 </segment>
+<segment>
+<pinref part="IC2" gate="G$1" pin="!RE"/>
+<pinref part="IC2" gate="G$1" pin="DE"/>
+<wire x1="203.2" y1="-66.04" x2="203.2" y2="-63.5" width="0.1524" layer="91"/>
+<junction x="203.2" y="-66.04"/>
+<wire x1="203.2" y1="-66.04" x2="195.58" y2="-66.04" width="0.1524" layer="91"/>
+<junction x="203.2" y="-63.5"/>
+<junction x="195.58" y="-66.04"/>
+<label x="187.96" y="-66.04" size="1.778" layer="95"/>
+</segment>
 </net>
 <net name="RF13" class="0">
@@
 </segment>
 </net>
+<net name="N$1" class="0">
+<segment>
+<pinref part="IC1" gate="G$1" pin="SOSCO/RPB8(4)/RB8(4)"/>
+<wire x1="160.02" y1="43.18" x2="220.98" y2="43.18" width="0.1524" layer="91"/>
+<pinref part="OS2" gate="A" pin="OUT"/>
+<wire x1="220.98" y1="43.18" x2="220.98" y2="45.72" width="0.1524" layer="91"/>
+<wire x1="220.98" y1="45.72" x2="226.06" y2="45.72" width="0.1524" layer="91"/>
+<junction x="160.02" y="43.18"/>
+<junction x="226.06" y="45.72"/>
+</segment>
+</net>
+<net name="SOSCI" class="0">
+<segment>
+<pinref part="IC1" gate="G$1" pin="SOSCI/RPC13(4)/RC13(4)"/>
+<wire x1="160.02" y1="40.64" x2="185.42" y2="40.64" width="0.1524" layer="91"/>
+<junction x="160.02" y="40.64"/>
+<junction x="185.42" y="40.64"/>
+<label x="185.42" y="40.64" size="1.778" layer="95"/>
+</segment>
+</net>

Commit message: up
Parts:
- removed JP1: vref-, pinhead:PINHD-1X2
- removed JP2: vref+, pinhead:PINHD-1X2
- added SPI_VOLTS: 1-2 3.3, 3-2 5.0, con-lstb:MA03-1
Connections:
- removed net N$57: IC1.VREF-/AN33/CVD33/PMPA7/RF9, JP1.1
- removed net N$58: IC1.VREF+/AN34/CVD34/PMPA6/RF10, JP2.1
- new net N$16: SPI-7.S, SPI_VOLTS.2
- net REFOUT: now also IC1.VREF+/AN34/CVD34/PMPA6/RF10; no longer JP2.2
- net RG11: no longer JP3.3
- net VCC: now also SPI_VOLTS.3; no longer SPI-7.S
- net VDD: now also SPI_VOLTS.1
- net VSS: now also IC1.VREF-/AN33/CVD33/PMPA7/RF9; no longer JP1.2

Commit message: up
Parts:
- added C32, C33, C34, C35: 0.1, rcl:C-USC0805
- added F3: 1206L050, polyfuse-smd_10:1206L050
- added IC10: 5.0VDC, linear:7805T
- added IC11: 3.3VDC, linear:7805T
Connections:
- new net N$30: C32.1, C33.1, F3.2, IC10.VI, IC11.VI
- net +24V: now also F3.1
- net +3V3: now also C34.1, IC11.VO
- net +5V: now also C35.1, IC10.VO
- net RG11: now also JP3.3
- net VSS: now also C32.2, C33.2, C34.2, C35.2, IC10.GND, IC11.GND
Changed lines of the file:
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@@
 <part name="P+27" library="supply1" library_urn="urn:adsk.eagle:library:371" deviceset="VCC" device=""/>
 <part name="VDD26" library="supply1" library_urn="urn:adsk.eagle:library:371" deviceset="VDD" device=""/>
+<part name="IC10" library="linear" library_urn="urn:adsk.eagle:library:262" deviceset="78*" device="T" package3d_urn="urn:adsk.eagle:package:16414/1" technology="05" value="5.0VDC"/>
+<part name="IC11" library="linear" library_urn="urn:adsk.eagle:library:262" deviceset="78*" device="T" package3d_urn="urn:adsk.eagle:package:16414/1" technology="05" value="3.3VDC"/>
+<part name="VSS60" library="supply1" library_urn="urn:adsk.eagle:library:371" deviceset="VSS" device=""/>
+<part name="VSS69" library="supply1" library_urn="urn:adsk.eagle:library:371" deviceset="VSS" device=""/>
+<part name="+3V3" library="supply1" library_urn="urn:adsk.eagle:library:371" deviceset="+3V3" device=""/>
+<part name="P+29" library="supply1" library_urn="urn:adsk.eagle:library:371" deviceset="+5V" device=""/>
+<part name="C32" library="rcl" library_urn="urn:adsk.eagle:library:334" deviceset="C-US" device="C0805" package3d_urn="urn:adsk.eagle:package:23617/2" value="0.1"/>
+<part name="C33" library="rcl" library_urn="urn:adsk.eagle:library:334" deviceset="C-US" device="C0805" package3d_urn="urn:adsk.eagle:package:23617/2" value="0.1"/>
+<part name="C34" library="rcl" library_urn="urn:adsk.eagle:library:334" deviceset="C-US" device="C0805" package3d_urn="urn:adsk.eagle:package:23617/2" value="0.1"/>
+<part name="C35" library="rcl" library_urn="urn:adsk.eagle:library:334" deviceset="C-US" device="C0805" package3d_urn="urn:adsk.eagle:package:23617/2" value="0.1"/>
+<part name="F3" library="polyfuse-smd_10" deviceset="?" device="1206L" technology="050"/>
+<part name="P+34" library="supply1" library_urn="urn:adsk.eagle:library:371" deviceset="+24V" device=""/>
 </parts>
 <sheets>
@@
 <attribute name="VALUE" x="-132.08" y="60.96" size="1.778" layer="96"/>
 </instance>
+<instance part="IC10" gate="A1" x="-139.7" y="134.62" smashed="yes">
+<attribute name="NAME" x="-147.32" y="140.335" size="1.778" layer="95"/>
+<attribute name="VALUE" x="-147.32" y="137.795" size="1.778" layer="96"/>
+</instance>
+<instance part="IC11" gate="A1" x="-139.7" y="109.22" smashed="yes">
+<attribute name="NAME" x="-147.32" y="114.935" size="1.778" layer="95"/>
+<attribute name="VALUE" x="-147.32" y="112.395" size="1.778" layer="96"/>
+</instance>
+<instance part="VSS60" gate="G$1" x="-139.7" y="99.06" smashed="yes">
+<attribute name="VALUE" x="-142.24" y="93.98" size="1.778" layer="96" rot="R90"/>
+</instance>
+<instance part="VSS69" gate="G$1" x="-139.7" y="124.46" smashed="yes">
+<attribute name="VALUE" x="-142.24" y="119.38" size="1.778" layer="96" rot="R90"/>
+</instance>
+<instance part="+3V3" gate="G$1" x="-124.46" y="109.22" smashed="yes" rot="R270">
+<attribute name="VALUE" x="-129.54" y="111.76" size="1.778" layer="96"/>
+</instance>
+<instance part="P+29" gate="1" x="-116.84" y="134.62" smashed="yes" rot="R270">
+<attribute name="VALUE" x="-121.92" y="137.16" size="1.778" layer="96"/>
+</instance>
+<instance part="C32" gate="G$1" x="-154.94" y="106.68" smashed="yes">
+<attribute name="NAME" x="-153.924" y="107.315" size="1.778" layer="95"/>
+<attribute name="VALUE" x="-153.924" y="102.489" size="1.778" layer="96"/>
+</instance>
+<instance part="C33" gate="G$1" x="-154.94" y="132.08" smashed="yes">
+<attribute name="NAME" x="-153.924" y="132.715" size="1.778" layer="95"/>
+<attribute name="VALUE" x="-153.924" y="127.889" size="1.778" layer="96"/>
+</instance>
+<instance part="C34" gate="G$1" x="-129.54" y="106.68" smashed="yes">
+<attribute name="NAME" x="-128.524" y="107.315" size="1.778" layer="95"/>
+<attribute name="VALUE" x="-128.524" y="102.489" size="1.778" layer="96"/>
+</instance>
+<instance part="C35" gate="G$1" x="-129.54" y="132.08" smashed="yes">
+<attribute name="NAME" x="-128.524" y="132.715" size="1.778" layer="95"/>
+<attribute name="VALUE" x="-128.524" y="127.889" size="1.778" layer="96"/>
+</instance>
+<instance part="F3" gate="G$1" x="-157.48" y="93.98" smashed="yes" rot="R270">
+<attribute name="NAME" x="-154.94" y="97.79" size="1.778" layer="95" rot="R270"/>
+<attribute name="VALUE" x="-161.29" y="97.79" size="1.778" layer="96" rot="R270"/>
+</instance>
+<instance part="P+34" gate="1" x="-160.02" y="88.9" smashed="yes" rot="R90">
+<attribute name="VALUE" x="-154.94" y="86.36" size="1.778" layer="96" rot="R180"/>
+</instance>
 </instances>
 <busses>
@@
 <junction x="20.32" y="-104.14"/>
 </segment>
+<segment>
+<pinref part="IC11" gate="A1" pin="GND"/>
+<pinref part="VSS60" gate="G$1" pin="VSS"/>
+<pinref part="C32" gate="G$1" pin="2"/>
+<pinref part="C34" gate="G$1" pin="2"/>
+<wire x1="-154.94" y1="101.6" x2="-139.7" y2="101.6" width="0.1524" layer="91"/>
+<junction x="-139.7" y="101.6"/>
+<wire x1="-139.7" y1="101.6" x2="-129.54" y2="101.6" width="0.1524" layer="91"/>
+<junction x="-129.54" y="101.6"/>
+<junction x="-154.94" y="101.6"/>
+</segment>
+<segment>
+<pinref part="IC10" gate="A1" pin="GND"/>
+<pinref part="VSS69" gate="G$1" pin="VSS"/>
+<pinref part="C33" gate="G$1" pin="2"/>
+<pinref part="C35" gate="G$1" pin="2"/>
+<wire x1="-154.94" y1="127" x2="-139.7" y2="127" width="0.1524" layer="91"/>
+<junction x="-154.94" y="127"/>
+<junction x="-139.7" y="127"/>
+<wire x1="-139.7" y1="127" x2="-129.54" y2="127" width="0.1524" layer="91"/>
+<junction x="-129.54" y="127"/>
+</segment>
 </net>
-<net name="+5V" class="2">
+<net name="+5V" class="1">
 <segment>
 <pinref part="F1" gate="G$1" pin="2"/>
@@
 <junction x="22.86" y="-165.1"/>
 </segment>
+<segment>
+<pinref part="IC10" gate="A1" pin="VO"/>
+<pinref part="P+29" gate="1" pin="+5V"/>
+<wire x1="-119.38" y1="134.62" x2="-129.54" y2="134.62" width="0.1524" layer="91"/>
+<pinref part="C35" gate="G$1" pin="1"/>
+<junction x="-129.54" y="134.62"/>
+<junction x="-119.38" y="134.62"/>
+</segment>
 </net>
 <net name="N$6" class="0">
@@
 </segment>
 </net>
-<net name="VCC" class="0">
+<net name="VCC" class="1">
 <segment>
 <pinref part="R6" gate="G$1" pin="2"/>
@@
 </segment>
 </net>
-<net name="+3V3" class="2">
+<net name="+3V3" class="1">
 <segment>
 <pinref part="F2" gate="G$1" pin="2"/>
@@
 <junction x="71.12" y="-137.16"/>
 </segment>
+<segment>
+<pinref part="IC11" gate="A1" pin="VO"/>
+<pinref part="+3V3" gate="G$1" pin="+3V3"/>
+<wire x1="-127" y1="109.22" x2="-129.54" y2="109.22" width="0.1524" layer="91"/>
+<pinref part="C34" gate="G$1" pin="1"/>
+<junction x="-129.54" y="109.22"/>
+<junction x="-127" y="109.22"/>
+</segment>
 </net>
 <net name="GND" class="1">
@@
 <junction x="-83.82" y="25.4"/>
 </segment>
+<segment>
+<pinref part="F3" gate="G$1" pin="1"/>
+<pinref part="P+34" gate="1" pin="+24V"/>
+<junction x="-157.48" y="88.9"/>
+</segment>
 </net>
 <net name="RPB1" class="0">
@@
 <label x="187.96" y="-66.04" size="1.778" layer="95"/>
 </segment>
+<segment>
+<pinref part="JP3" gate="A" pin="3"/>
+<wire x1="114.3" y1="-157.48" x2="132.08" y2="-157.48" width="0.1524" layer="91"/>
+<junction x="114.3" y="-157.48"/>
+<junction x="132.08" y="-157.48"/>
+<label x="137.16" y="-157.48" size="1.778" layer="95"/>
+</segment>
 </net>
 <net name="RF13" class="0">
@@
 </segment>
 </net>
+<net name="N$30" class="2">
+<segment>
+<pinref part="IC10" gate="A1" pin="VI"/>
+<pinref part="C33" gate="G$1" pin="1"/>
+<wire x1="-154.94" y1="134.62" x2="-149.86" y2="134.62" width="0.1524" layer="91"/>
+<junction x="-154.94" y="134.62"/>
+<pinref part="F3" gate="G$1" pin="2"/>
+<wire x1="-157.48" y1="99.06" x2="-160.02" y2="99.06" width="0.1524" layer="91"/>
+<wire x1="-160.02" y1="99.06" x2="-160.02" y2="109.22" width="0.1524" layer="91"/>
+<wire x1="-160.02" y1="109.22" x2="-160.02" y2="134.62" width="0.1524" layer="91"/>
+<wire x1="-160.02" y1="134.62" x2="-154.94" y2="134.62" width="0.1524" layer="91"/>
+<junction x="-157.48" y="99.06"/>
+<pinref part="IC11" gate="A1" pin="VI"/>
+<wire x1="-160.02" y1="109.22" x2="-154.94" y2="109.22" width="0.1524" layer="91"/>
+<pinref part="C32" gate="G$1" pin="1"/>
+<wire x1="-154.94" y1="109.22" x2="-149.86" y2="109.22" width="0.1524" layer="91"/>
+<junction x="-154.94" y="109.22"/>
+<junction x="-160.02" y="109.22"/>
+</segment>
+</net>
