File: pic32mk.sch (EAGLE design)
At the start: 91 parts, among them IC1 PIC32MK1024MCF100-I_PT, IC10 5.0VDC, IC11 3.3VDC, IC2 ADM3095EBRZ, IC3 TXB0101DCKR, IC4 MAX203ECWP, IC5 TXB0101DCKR, IC6 TXB0101DCKR, IC7 TXB0101DCKR, IC8 TXB0101DCKR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

Commit message: up
Other:
- note added: "FLT15"
- note added: "FLT5"
- note added: "FLT6"
Changed lines of the file:
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@@
 <text x="-137.16" y="-30.48" size="1.778" layer="91">A</text>
 <text x="-137.16" y="-27.94" size="1.778" layer="91">B</text>
+<text x="182.88" y="-149.86" size="1.778" layer="91">FLT6</text>
+<text x="200.66" y="73.66" size="1.778" layer="91">FLT5</text>
+<text x="5.08" y="-149.86" size="1.778" layer="91">FLT15</text>
 </plain>
 <instances>
@@
 <instance part="C13" gate="G$1" x="96.52" y="-99.06" smashed="yes" rot="R270">
 <attribute name="NAME" x="97.155" y="-100.076" size="1.778" layer="95" rot="R270"/>
-<attribute name="VALUE" x="92.329" y="-100.076" size="1.778" layer="96" rot="R270"/>
+<attribute name="VALUE" x="94.869" y="-102.616" size="1.778" layer="96" rot="R270"/>
 </instance>
 <instance part="IC6" gate="G$1" x="-88.9" y="-30.48" smashed="yes">
@@
 </instance>
 <instance part="VSS19" gate="G$1" x="182.88" y="-121.92" smashed="yes">
-<attribute name="VALUE" x="180.34" y="-127" size="1.778" layer="96" rot="R90"/>
+<attribute name="VALUE" x="180.34" y="-121.92" size="1.778" layer="96" rot="R180"/>
 </instance>
 <instance part="VSS22" gate="G$1" x="243.84" y="-121.92" smashed="yes">
@@
 </instance>
 <instance part="VSS23" gate="G$1" x="200.66" y="101.6" smashed="yes">
-<attribute name="VALUE" x="198.12" y="96.52" size="1.778" layer="96" rot="R90"/>
+<attribute name="VALUE" x="198.12" y="101.6" size="1.778" layer="96" rot="R180"/>
 </instance>
 <instance part="VSS27" gate="G$1" x="256.54" y="101.6" smashed="yes">
-<attribute name="VALUE" x="254" y="96.52" size="1.778" layer="96" rot="R90"/>
+<attribute name="VALUE" x="264.16" y="104.14" size="1.778" layer="96" rot="R180"/>
 </instance>
 <instance part="IC3" gate="G$1" x="-134.62" y="-68.58" smashed="yes">
@@
 </instance>
 <instance part="VSS40" gate="G$1" x="162.56" y="-109.22" smashed="yes">
-<attribute name="VALUE" x="160.02" y="-114.3" size="1.778" layer="96" rot="R90"/>
+<attribute name="VALUE" x="160.02" y="-109.22" size="1.778" layer="96" rot="R180"/>
 </instance>
-<instance part="VSS41" gate="G$1" x="259.08" y="-109.22" smashed="yes">
-<attribute name="VALUE" x="256.54" y="-114.3" size="1.778" layer="96" rot="R90"/>
+<instance part="VSS41" gate="G$1" x="261.62" y="-109.22" smashed="yes">
+<attribute name="VALUE" x="261.62" y="-111.76" size="1.778" layer="96"/>
 </instance>
 <instance part="DIN" gate="-1" x="-109.22" y="-137.16" smashed="yes">
@@
 </instance>
 <instance part="P+23" gate="1" x="175.26" y="81.28" smashed="yes" rot="R180">
-<attribute name="VALUE" x="177.8" y="86.36" size="1.778" layer="96" rot="R270"/>
+<attribute name="VALUE" x="167.64" y="83.82" size="1.778" layer="96"/>
 </instance>
 <instance part="P+24" gate="1" x="274.32" y="119.38" smashed="yes" rot="R180">
@@
 <pinref part="C18" gate="G$1" pin="2"/>
 <pinref part="VSS41" gate="G$1" pin="VSS"/>
-<wire x1="259.08" y1="-106.68" x2="256.54" y2="-106.68" width="0.1524" layer="91"/>
+<wire x1="261.62" y1="-106.68" x2="256.54" y2="-106.68" width="0.1524" layer="91"/>
 <pinref part="C21" gate="G$1" pin="2"/>
 <wire x1="256.54" y1="-114.3" x2="256.54" y2="-106.68" width="0.1524" layer="91"/>
 <junction x="256.54" y="-114.3"/>
 <junction x="256.54" y="-106.68"/>
-<junction x="259.08" y="-106.68"/>
+<junction x="261.62" y="-106.68"/>
 </segment>
 <segment>
@@
 <junction x="93.98" y="-88.9"/>
 <junction x="93.98" y="-93.98"/>
-<label x="93.98" y="-96.52" size="1.778" layer="95"/>
+<label x="93.98" y="-96.52" size="1.778" layer="95" rot="R180"/>
 </segment>
 <segment>
@@
 <junction x="96.52" y="-88.9"/>
 <junction x="96.52" y="-93.98"/>
-<label x="96.52" y="-93.98" size="1.778" layer="95"/>
+<label x="96.52" y="-96.52" size="1.778" layer="95"/>
 </segment>
 <segment>
@@
 <junction x="71.12" y="-88.9"/>
 <junction x="71.12" y="-101.6"/>
-<label x="71.12" y="-101.6" size="1.778" layer="95"/>
+<label x="71.12" y="-101.6" size="1.778" layer="95" rot="R270"/>
 </segment>
 <segment>
@@
 <wire x1="76.2" y1="-88.9" x2="76.2" y2="-96.52" width="0.1524" layer="91"/>
 <junction x="76.2" y="-96.52"/>
-<label x="76.2" y="-96.52" size="1.778" layer="95"/>
+<label x="76.2" y="-96.52" size="1.778" layer="95" rot="R270"/>
 <junction x="76.2" y="-88.9"/>
 </segment>
@@
 <wire x1="78.74" y1="-88.9" x2="78.74" y2="-96.52" width="0.1524" layer="91"/>
 <junction x="78.74" y="-96.52"/>
-<label x="78.74" y="-96.52" size="1.778" layer="95"/>
+<label x="78.74" y="-96.52" size="1.778" layer="95" rot="R270"/>
 <junction x="78.74" y="-88.9"/>
 </segment>
@@
 <wire x1="86.36" y1="-88.9" x2="86.36" y2="-96.52" width="0.1524" layer="91"/>
 <junction x="86.36" y="-96.52"/>
-<label x="86.36" y="-96.52" size="1.778" layer="95"/>
+<label x="86.36" y="-99.06" size="1.778" layer="95" rot="R270"/>
 <junction x="86.36" y="-88.9"/>
 </segment>
@@
 <wire x1="88.9" y1="-88.9" x2="88.9" y2="-93.98" width="0.1524" layer="91"/>
 <junction x="88.9" y="-93.98"/>
-<label x="88.9" y="-93.98" size="1.778" layer="95"/>
+<label x="88.9" y="-99.06" size="1.778" layer="95" rot="R270"/>
 <junction x="88.9" y="-88.9"/>
 </segment>
@@
 <wire x1="91.44" y1="-88.9" x2="91.44" y2="-93.98" width="0.1524" layer="91"/>
 <junction x="91.44" y="-93.98"/>
-<label x="91.44" y="-93.98" size="1.778" layer="95"/>
+<label x="91.44" y="-99.06" size="1.778" layer="95" rot="R270"/>
 <junction x="91.44" y="-88.9"/>
 </segment>

Commit message: up
Parts:
- added X3: 53261-10, con-molex:53261-10
Connections:
- new net D1+: IC1.D1+, X3-4.S
- new net D1-: IC1.D1-, X3-3.S
- new net D2+: IC1.D2+, X3-7.S
- new net D2-: IC1.D2-, X3-6.S
- new net USBID1: IC1.PGED2/RPB5/USBID1/RB5(6), X3-1.S
- new net VBUS: IC1.VBUS, X3-2.S
- new net VBUS2: IC1.VBUS2, X3-5.S
- net IN7: now also IC1.TMS/OA5IN-/AN27/CVD27/C5IN1-/RPB9/RB9; no longer IC1.PGED2/RPB5/USBID1/RB5(6)
- net SOSCI: now also SPI-10.S
- net VCC: now also X3-10.S
- net VDD: now also X3-9.S; no longer SPI-10.S
- net VSS: now also X3-8.S
Changed lines of the file:
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@@
 <part name="P+6" library="supply1" library_urn="urn:adsk.eagle:library:371" deviceset="VCC" device=""/>
 <part name="VDD9" library="supply1" library_urn="urn:adsk.eagle:library:371" deviceset="VDD" device=""/>
-<part name="VDD24" library="supply1" library_urn="urn:adsk.eagle:library:371" deviceset="VDD" device=""/>
 <part name="VSS28" library="supply1" library_urn="urn:adsk.eagle:library:371" deviceset="VSS" device=""/>
 <part name="SPI_VOLTS" library="con-lstb" library_urn="urn:adsk.eagle:library:162" deviceset="MA03-1" device="" package3d_urn="urn:adsk.eagle:package:8339/1" value="1-2 3.3, 3-2 5.0"/>
@@
 <part name="F3" library="polyfuse-smd_10" deviceset="?" device="1206L" technology="050"/>
 <part name="P+34" library="supply1" library_urn="urn:adsk.eagle:library:371" deviceset="+24V" device=""/>
+<part name="X3" library="con-molex" library_urn="urn:adsk.eagle:library:165" deviceset="53?-10" device="261" package3d_urn="urn:adsk.eagle:package:8078504/1"/>
+<part name="VSS70" library="supply1" library_urn="urn:adsk.eagle:library:371" deviceset="VSS" device=""/>
+<part name="VDD24" library="supply1" library_urn="urn:adsk.eagle:library:371" deviceset="VDD" device=""/>
+<part name="P+35" library="supply1" library_urn="urn:adsk.eagle:library:371" deviceset="VCC" device=""/>
 </parts>
 <sheets>
@@
 <attribute name="VALUE" x="-55.88" y="-7.62" size="1.778" layer="96" rot="R90"/>
 </instance>
-<instance part="VDD24" gate="G$1" x="-104.14" y="60.96" smashed="yes" rot="R180">
-<attribute name="VALUE" x="-104.14" y="55.88" size="1.778" layer="96"/>
-</instance>
 <instance part="VSS28" gate="G$1" x="17.78" y="-104.14" smashed="yes" rot="R270">
 <attribute name="VALUE" x="12.7" y="-101.6" size="1.778" layer="96"/>
@@
 <attribute name="VALUE" x="-154.94" y="86.36" size="1.778" layer="96" rot="R180"/>
 </instance>
+<instance part="X3" gate="-1" x="205.74" y="68.58" smashed="yes">
+<attribute name="NAME" x="208.28" y="67.818" size="1.524" layer="95"/>
+<attribute name="VALUE" x="204.978" y="69.977" size="1.778" layer="96"/>
+</instance>
+<instance part="X3" gate="-2" x="205.74" y="66.04" smashed="yes">
+<attribute name="NAME" x="208.28" y="65.278" size="1.524" layer="95"/>
+</instance>
+<instance part="X3" gate="-3" x="205.74" y="63.5" smashed="yes">
+<attribute name="NAME" x="208.28" y="62.738" size="1.524" layer="95"/>
+</instance>
+<instance part="X3" gate="-4" x="205.74" y="60.96" smashed="yes">
+<attribute name="NAME" x="208.28" y="60.198" size="1.524" layer="95"/>
+</instance>
+<instance part="X3" gate="-5" x="205.74" y="58.42" smashed="yes">
+<attribute name="NAME" x="208.28" y="57.658" size="1.524" layer="95"/>
+</instance>
+<instance part="X3" gate="-6" x="205.74" y="55.88" smashed="yes">
+<attribute name="NAME" x="208.28" y="55.118" size="1.524" layer="95"/>
+</instance>
+<instance part="X3" gate="-7" x="205.74" y="53.34" smashed="yes">
+<attribute name="NAME" x="208.28" y="52.578" size="1.524" layer="95"/>
+</instance>
+<instance part="X3" gate="-8" x="205.74" y="50.8" smashed="yes">
+<attribute name="NAME" x="208.28" y="50.038" size="1.524" layer="95"/>
+</instance>
+<instance part="X3" gate="-9" x="205.74" y="48.26" smashed="yes">
+<attribute name="NAME" x="208.28" y="47.498" size="1.524" layer="95"/>
+</instance>
+<instance part="X3" gate="-10" x="205.74" y="45.72" smashed="yes">
+<attribute name="NAME" x="208.28" y="44.958" size="1.524" layer="95"/>
+</instance>
+<instance part="VSS70" gate="G$1" x="200.66" y="50.8" smashed="yes" rot="R270">
+<attribute name="VALUE" x="195.58" y="53.34" size="1.778" layer="96"/>
+</instance>
+<instance part="VDD24" gate="G$1" x="200.66" y="48.26" smashed="yes" rot="R90">
+<attribute name="VALUE" x="203.2" y="45.72" size="1.778" layer="96" rot="R180"/>
+</instance>
+<instance part="P+35" gate="VCC" x="200.66" y="45.72" smashed="yes" rot="R90">
+<attribute name="VALUE" x="200.66" y="43.18" size="1.778" layer="96" rot="R180"/>
+</instance>
 </instances>
 <busses>
@@
 </segment>
 <segment>
-<pinref part="SPI" gate="-10" pin="S"/>
-<pinref part="VDD24" gate="G$1" pin="VDD"/>
-<junction x="-104.14" y="63.5"/>
-</segment>
-<segment>
 <pinref part="SPI_VOLTS" gate="G$1" pin="1"/>
 <pinref part="VDD26" gate="G$1" pin="VDD"/>
 <junction x="-132.08" y="68.58"/>
 </segment>
+<segment>
+<pinref part="X3" gate="-9" pin="S"/>
+<junction x="203.2" y="48.26"/>
+<pinref part="VDD24" gate="G$1" pin="VDD"/>
+</segment>
 </net>
 <net name="VSS" class="1">
@@
 <junction x="-129.54" y="127"/>
 </segment>
+<segment>
+<pinref part="X3" gate="-8" pin="S"/>
+<junction x="203.2" y="50.8"/>
+<pinref part="VSS70" gate="G$1" pin="VSS"/>
+</segment>
 </net>
 <net name="+5V" class="1">
@@
 <junction x="-132.08" y="73.66"/>
 </segment>
+<segment>
+<pinref part="X3" gate="-10" pin="S"/>
+<junction x="203.2" y="45.72"/>
+<pinref part="P+35" gate="VCC" pin="VCC"/>
+</segment>
 </net>
 <net name="+3V3" class="1">
@@
 <net name="IN7" class="0">
 <segment>
-<pinref part="IC1" gate="G$1" pin="PGED2/RPB5/USBID1/RB5(6)"/>
-<wire x1="160.02" y1="30.48" x2="185.42" y2="30.48" width="0.1524" layer="91"/>
-<junction x="160.02" y="30.48"/>
-<junction x="185.42" y="30.48"/>
-<label x="185.42" y="30.48" size="1.778" layer="95"/>
-</segment>
-<segment>
 <pinref part="U$1" gate="G$1" pin="OUT7"/>
 <wire x1="-25.4" y1="-165.1" x2="-5.08" y2="-165.1" width="0.1524" layer="91"/>
@@
 <label x="0" y="-165.1" size="1.778" layer="95"/>
 </segment>
+<segment>
+<pinref part="IC1" gate="G$1" pin="TMS/OA5IN-/AN27/CVD27/C5IN1-/RPB9/RB9"/>
+<wire x1="116.84" y1="104.14" x2="116.84" y2="111.76" width="0.1524" layer="91"/>
+<junction x="116.84" y="104.14"/>
+<junction x="116.84" y="111.76"/>
+<label x="119.38" y="111.76" size="1.778" layer="95"/>
+</segment>
 </net>
 <net name="IN6" class="0">
@@
 <label x="185.42" y="40.64" size="1.778" layer="95"/>
 </segment>
+<segment>
+<pinref part="SPI" gate="-10" pin="S"/>
+<wire x1="-104.14" y1="63.5" x2="-104.14" y2="58.42" width="0.1524" layer="91"/>
+<junction x="-104.14" y="63.5"/>
+<junction x="-104.14" y="58.42"/>
+<label x="-99.06" y="58.42" size="1.778" layer="95"/>
+</segment>
 </net>
 <net name="N$16" class="0">
@@
 </segment>
 </net>
+<net name="USBID1" class="0">
+<segment>
+<pinref part="IC1" gate="G$1" pin="PGED2/RPB5/USBID1/RB5(6)"/>
+<wire x1="160.02" y1="30.48" x2="185.42" y2="30.48" width="0.1524" layer="91"/>
+<junction x="160.02" y="30.48"/>
+<junction x="185.42" y="30.48"/>
+<label x="185.42" y="30.48" size="1.778" layer="95"/>
+</segment>
+<segment>
+<pinref part="X3" gate="-1" pin="S"/>
+<junction x="203.2" y="68.58"/>
+<label x="187.96" y="68.58" size="1.778" layer="95"/>
+</segment>
+</net>
+<net name="VBUS" class="0">
+<segment>
+<pinref part="IC1" gate="G$1" pin="VBUS"/>
+<junction x="160.02" y="-7.62"/>
+<label x="160.02" y="-7.62" size="1.778" layer="95"/>
+</segment>
+<segment>
+<pinref part="X3" gate="-2" pin="S"/>
+<junction x="203.2" y="66.04"/>
+<label x="187.96" y="66.04" size="1.778" layer="95"/>
+</segment>
+</net>
+<net name="D1-" class="0">
+<segment>
+<pinref part="IC1" gate="G$1" pin="D1-"/>
+<junction x="160.02" y="-2.54"/>
+<label x="160.02" y="-2.54" size="1.778" layer="95"/>
+</segment>
+<segment>
+<pinref part="X3" gate="-3" pin="S"/>
+<junction x="203.2" y="63.5"/>
+<label x="187.96" y="63.5" size="1.778" layer="95"/>
+</segment>
+</net>
+<net name="D1+" class="0">
+<segment>
+<pinref part="IC1" gate="G$1" pin="D1+"/>
+<junction x="160.02" y="0"/>
+<label x="160.02" y="0" size="1.778" layer="95"/>
+</segment>
+<segment>
+<pinref part="X3" gate="-4" pin="S"/>
+<junction x="203.2" y="60.96"/>
+<label x="187.96" y="60.96" size="1.778" layer="95"/>
+</segment>
+</net>
+<net name="VBUS2" class="0">
+<segment>
+<pinref part="IC1" gate="G$1" pin="VBUS2"/>
+<junction x="160.02" y="2.54"/>
+<label x="160.02" y="2.54" size="1.778" layer="95"/>
+</segment>
+<segment>
+<pinref part="X3" gate="-5" pin="S"/>
+<junction x="203.2" y="58.42"/>
+<label x="187.96" y="58.42" size="1.778" layer="95"/>
+</segment>
+</net>
+<net name="D2-" class="0">
+<segment>
+<pinref part="IC1" gate="G$1" pin="D2-"/>
+<junction x="160.02" y="5.08"/>
+<label x="160.02" y="5.08" size="1.778" layer="95"/>
+</segment>
+<segment>
+<pinref part="X3" gate="-6" pin="S"/>
+<junction x="203.2" y="55.88"/>
+<label x="187.96" y="55.88" size="1.778" layer="95"/>
+</segment>
+</net>
+<net name="D2+" class="0">
+<segment>
+<pinref part="IC1" gate="G$1" pin="D2+"/>
+<junction x="160.02" y="7.62"/>
+<label x="160.02" y="7.62" size="1.778" layer="95"/>
+</segment>
+<segment>
+<pinref part="X3" gate="-7" pin="S"/>
+<junction x="203.2" y="53.34"/>
+<label x="187.96" y="53.34" size="1.778" layer="95"/>
+</segment>
+</net>

Commit message: up
Parts:
- renumbered S1 to RESET, X1 to QEI, X3 to USB-BO

Commit message: up
Parts:
- added QEI3: 22-23-2041, con-molex:22-23-2041
Connections:
- net RG6: now also QEI3-2.S
- net RG7: now also QEI3-1.S
- net VDD: now also QEI3-3.S
- net VSS: now also QEI3-4.S
Changed lines of the file:
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@@
 <part name="VDD24" library="supply1" library_urn="urn:adsk.eagle:library:371" deviceset="VDD" device=""/>
 <part name="P+35" library="supply1" library_urn="urn:adsk.eagle:library:371" deviceset="VCC" device=""/>
+<part name="QEI3" library="con-molex" library_urn="urn:adsk.eagle:library:165" deviceset="22-23-2041" device="" package3d_urn="urn:adsk.eagle:package:8078635/1"/>
+<part name="VSS71" library="supply1" library_urn="urn:adsk.eagle:library:371" deviceset="VSS" device=""/>
+<part name="VDD27" library="supply1" library_urn="urn:adsk.eagle:library:371" deviceset="VDD" device=""/>
 </parts>
 <sheets>
@@
 <attribute name="VALUE" x="200.66" y="43.18" size="1.778" layer="96" rot="R180"/>
 </instance>
+<instance part="QEI3" gate="-1" x="-142.24" y="-2.54" smashed="yes" rot="R180">
+<attribute name="NAME" x="-144.78" y="-1.778" size="1.524" layer="95" rot="R180"/>
+<attribute name="VALUE" x="-141.478" y="-3.937" size="1.778" layer="96" rot="R180"/>
+</instance>
+<instance part="QEI3" gate="-2" x="-142.24" y="0" smashed="yes" rot="R180">
+<attribute name="NAME" x="-144.78" y="0.762" size="1.524" layer="95" rot="R180"/>
+</instance>
+<instance part="QEI3" gate="-3" x="-142.24" y="2.54" smashed="yes" rot="R180">
+<attribute name="NAME" x="-144.78" y="3.302" size="1.524" layer="95" rot="R180"/>
+</instance>
+<instance part="QEI3" gate="-4" x="-142.24" y="5.08" smashed="yes" rot="R180">
+<attribute name="NAME" x="-144.78" y="5.842" size="1.524" layer="95" rot="R180"/>
+</instance>
+<instance part="VSS71" gate="G$1" x="-129.54" y="7.62" smashed="yes" rot="R180">
+<attribute name="VALUE" x="-127" y="12.7" size="1.778" layer="96" rot="R270"/>
+</instance>
+<instance part="VDD27" gate="G$1" x="-124.46" y="5.08" smashed="yes">
+<attribute name="VALUE" x="-127" y="2.54" size="1.778" layer="96" rot="R90"/>
+</instance>
 </instances>
 <busses>
@@
 <pinref part="VDD24" gate="G$1" pin="VDD"/>
 </segment>
+<segment>
+<pinref part="QEI3" gate="-3" pin="S"/>
+<wire x1="-139.7" y1="2.54" x2="-124.46" y2="2.54" width="0.1524" layer="91"/>
+<junction x="-139.7" y="2.54"/>
+<pinref part="VDD27" gate="G$1" pin="VDD"/>
+</segment>
 </net>
 <net name="VSS" class="1">
@@
 <pinref part="VSS70" gate="G$1" pin="VSS"/>
 </segment>
+<segment>
+<pinref part="QEI3" gate="-4" pin="S"/>
+<wire x1="-139.7" y1="5.08" x2="-129.54" y2="5.08" width="0.1524" layer="91"/>
+<junction x="-139.7" y="5.08"/>
+<pinref part="VSS71" gate="G$1" pin="VSS"/>
+</segment>
 </net>
 <net name="+5V" class="1">
@@
 </segment>
 <segment>
+<pinref part="JP3" gate="A" pin="3"/>
+<wire x1="114.3" y1="-157.48" x2="132.08" y2="-157.48" width="0.1524" layer="91"/>
+<junction x="114.3" y="-157.48"/>
+<junction x="132.08" y="-157.48"/>
+<label x="137.16" y="-157.48" size="1.778" layer="95"/>
+<wire x1="132.08" y1="-157.48" x2="276.86" y2="-157.48" width="0.1524" layer="91"/>
+<wire x1="276.86" y1="-157.48" x2="276.86" y2="-78.74" width="0.1524" layer="91"/>
+<wire x1="276.86" y1="-78.74" x2="187.96" y2="-78.74" width="0.1524" layer="91"/>
+<wire x1="187.96" y1="-78.74" x2="187.96" y2="-66.04" width="0.1524" layer="91"/>
 <pinref part="IC2" gate="G$1" pin="!RE"/>
 <pinref part="IC2" gate="G$1" pin="DE"/>
@@
 <junction x="195.58" y="-66.04"/>
 <label x="187.96" y="-66.04" size="1.778" layer="95"/>
-</segment>
-<segment>
-<pinref part="JP3" gate="A" pin="3"/>
-<wire x1="114.3" y1="-157.48" x2="132.08" y2="-157.48" width="0.1524" layer="91"/>
-<junction x="114.3" y="-157.48"/>
-<junction x="132.08" y="-157.48"/>
-<label x="137.16" y="-157.48" size="1.778" layer="95"/>
+<wire x1="187.96" y1="-66.04" x2="195.58" y2="-66.04" width="0.1524" layer="91"/>
 </segment>
 </net>
@@
 <label x="137.16" y="-142.24" size="1.778" layer="95"/>
 </segment>
+<segment>
+<pinref part="QEI3" gate="-2" pin="S"/>
+<wire x1="-139.7" y1="0" x2="-134.62" y2="0" width="0.1524" layer="91"/>
+<junction x="-139.7" y="0"/>
+<junction x="-134.62" y="0"/>
+<label x="-129.54" y="0" size="1.778" layer="95"/>
+</segment>
 </net>
 <net name="RG7" class="0">
@@
 <label x="137.16" y="-139.7" size="1.778" layer="95"/>
 </segment>
+<segment>
+<pinref part="QEI3" gate="-1" pin="S"/>
+<wire x1="-139.7" y1="-2.54" x2="-134.62" y2="-2.54" width="0.1524" layer="91"/>
+<junction x="-139.7" y="-2.54"/>
+<junction x="-134.62" y="-2.54"/>
+<label x="-129.54" y="-2.54" size="1.778" layer="95"/>
+</segment>
 </net>
