File: lcd240.brd (EAGLE design)
At the start: 119.4 x 100 mm, 27 parts, among them IC1 CAT4238TD-GT3

Commit message: up
Parts:
- added LED1: power, led:SML0805
- added R7: 1000, rcl:R0805
- added SJ1: LCD_blank, jumper:SJ_2
- added SJ2: PLED_ON, jumper:SJ
Connections:
- new net N$27: IC1.4, SJ1.2
- new net N$28: R7.1, SJ2.2
- new net N$29: LED1.A, R7.2
- net GND: now also LED1.C
- net N$17: now also SJ1.3
- net N$4: now also SJ1.1; no longer IC1.4
- net VDD: now also SJ2.1
Routing:
- net N$17: track 0.00 -> 88.3 mm
- net N$27: track 0.00 -> 54.5 mm
- net VDD: track 168.2 -> 211.4 mm, vias 1 -> 3
- net N$4: track 164.0 -> 139.6 mm, vias 0 -> 1
- net N$24: track 56.4 -> 74.8 mm, vias 0 -> 1
- net GND: track 55.1 -> 40.2 mm
- net N$29: track 0.00 -> 6.96 mm
- net N$28: track 0.00 -> 3.90 mm
- net N$26: track 41.9 -> 45.1 mm
- net N$15: track 33.8 -> 35.1 mm, vias 2 -> 0
- net N$25: track 41.9 -> 41.8 mm, vias 1 -> 0

Commit message: up
Parts:
- added L2: 47uh, rcl:L2012C
Connections:
- net N$23: now also L2.1
- net VDD: now also L2.2
Routing:
- net N$23: track 17.8 -> 23.5 mm
- net VDD: track 211.4 -> 217.2 mm
Other:
- board text added: "EA DOGXL240-7 W BL 1.1 FGB"
Changed lines of the file:
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@@
 <wire x1="119.36" y1="100" x2="0" y2="100" width="0" layer="20"/>
 <wire x1="0" y1="100" x2="0" y2="0" width="0" layer="20"/>
-<hole x="3.81" y="96.52" drill="0.35"/>
-<hole x="115.57" y="96.52" drill="0.35"/>
-<hole x="115.57" y="3.81" drill="0.35"/>
-<hole x="3.81" y="3.81" drill="0.35"/>
-<hole x="96.52" y="85.09" drill="0.35"/>
+<hole x="6.35" y="93.98" drill="1.524"/>
+<hole x="113.03" y="93.98" drill="1.524"/>
+<hole x="113.03" y="6.35" drill="1.524"/>
+<hole x="6.35" y="6.35" drill="1.524"/>
+<hole x="93.98" y="85.09" drill="1.524"/>
+<text x="113.03" y="15.24" size="2.54" layer="1" font="vector" ratio="16" rot="R90">EA DOGXL240-7 W BL 1.1 FGB</text>
 </plain>
 <attributes>
@@
 <param name="RoutingGrid" value="3mil"/>
 <param name="AutoGrid" value="1"/>
-<param name="Efforts" value="0"/>
+<param name="Efforts" value="2"/>
 <param name="TopRouterVariant" value="1"/>
 <param name="tpViaShape" value="round"/>
@@
 <attribute name="VALUE" x="109.76" y="86.59" size="1.27" layer="27" rot="R270"/>
 </element>
+<element name="L2" library="rcl" library_urn="urn:adsk.eagle:library:334" package="L2012C" package3d_urn="urn:adsk.eagle:package:23475/2" value="47uh" x="12.7" y="7.62" smashed="yes" rot="R90">
+<attribute name="NAME" x="11.43" y="5.715" size="1.27" layer="25" rot="R90"/>
+<attribute name="POPULARITY" value="6" x="12.7" y="7.62" size="1.778" layer="27" rot="R90" display="off"/>
+<attribute name="SPICEPREFIX" value="L" x="12.7" y="7.62" size="1.778" layer="27" rot="R90" display="off"/>
+<attribute name="VALUE" x="15.24" y="5.715" size="1.27" layer="27" rot="R90"/>
+</element>
 </elements>
 <signals>
@@
 <wire x1="111.7092" y1="72.5424" x2="112.4712" y2="73.3044" width="0.3048" layer="1"/>
 <wire x1="110.2614" y1="72.5424" x2="111.7092" y2="72.5424" width="0.3048" layer="1"/>
-<wire x1="97.917" y1="84.8868" x2="110.2614" y2="72.5424" width="0.3048" layer="1"/>
-<wire x1="97.917" y1="87.4776" x2="97.917" y2="84.8868" width="0.3048" layer="1"/>
-<wire x1="92.7354" y1="92.6592" x2="97.917" y2="87.4776" width="0.3048" layer="1"/>
 <wire x1="112.4712" y1="73.6092" x2="112.522" y2="73.66" width="0.3048" layer="1"/>
-<wire x1="92.7354" y1="92.6592" x2="92.71" y2="92.71" width="0.3048" layer="1"/>
 <wire x1="63.0936" y1="87.0204" x2="63.0936" y2="81.0768" width="0.3048" layer="1"/>
 <wire x1="70.6374" y1="94.5642" x2="63.0936" y2="87.0204" width="0.3048" layer="1"/>
@@
 <via x="38.862" y="5.1054" extent="1-16" drill="0.35"/>
 <via x="34.671" y="6.858" extent="1-16" drill="0.35"/>
+<contactref element="L2" pad="2"/>
+<wire x1="16.3068" y1="8.6868" x2="12.7254" y2="8.6868" width="0.3048" layer="1"/>
+<wire x1="17.78" y1="10.16" x2="16.3068" y2="8.6868" width="0.3048" layer="1"/>
+<wire x1="12.7254" y1="8.6868" x2="12.7" y2="8.62" width="0.3048" layer="1"/>
+<wire x1="98.4504" y1="84.3534" x2="110.2614" y2="72.5424" width="0.3048" layer="1"/>
+<wire x1="98.4504" y1="86.7918" x2="98.4504" y2="84.3534" width="0.3048" layer="1"/>
+<wire x1="92.7354" y1="92.5068" x2="98.4504" y2="86.7918" width="0.3048" layer="1"/>
+<wire x1="92.7354" y1="92.5068" x2="92.71" y2="92.71" width="0.3048" layer="1"/>
 </signal>
 <signal name="GND" class="1">
@@
 <wire x1="17.8308" y1="5.1054" x2="17.78" y2="5.08" width="0.1524" layer="1"/>
 <wire x1="23.4696" y1="5.1054" x2="23.5" y2="5.08" width="0.1524" layer="1"/>
+<contactref element="L2" pad="1"/>
+<wire x1="16.3068" y1="6.5532" x2="12.7254" y2="6.5532" width="0.1524" layer="1"/>
+<wire x1="17.78" y1="5.08" x2="16.3068" y2="6.5532" width="0.1524" layer="1"/>
+<wire x1="12.7254" y1="6.5532" x2="12.7" y2="6.62" width="0.1524" layer="1"/>
 </signal>
 <signal name="N$24" class="2">

Commit message: up
Parts:
- R1: value 25 -> 21.5
Changed lines of the file:
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@@
 <attribute name="VALUE" x="24.13" y="7.62" size="1.27" layer="27"/>
 </element>
-<element name="R1" library="rcl" library_urn="urn:adsk.eagle:library:334" package="R0805" package3d_urn="urn:adsk.eagle:package:23553/2" value="25" x="53.34" y="5.08" smashed="yes">
+<element name="R1" library="rcl" library_urn="urn:adsk.eagle:library:334" package="R0805" package3d_urn="urn:adsk.eagle:package:23553/2" value="21.5" x="53.34" y="5.08" smashed="yes">
 <attribute name="NAME" x="52.705" y="6.35" size="1.27" layer="25"/>
 <attribute name="POPULARITY" value="85" x="53.34" y="5.08" size="1.778" layer="27" display="off"/>
