File: tic12400.brd (EAGLE design)
At the start: 100 x 80 mm, 12 parts, among them X1 22-23-2031

Commit message: up
Parts:
- added C6: 10uf, rcl:C0805
- added C7: 0.1, rcl:C0805
- moved R4 2.84 mm to (52.1, 12.7)
- moved R1 2.84 mm to (55.9, 12.7)
- moved R3 2.54 mm to (47.0, 12.7)
Connections:
- net GND: now also C6.2, C7.2
- net VDD: now also C6.1, C7.1
Routing:
- net GND: track 32.5 -> 8.48 mm, vias 1 -> 14
- net N$2: track 31.4 -> 21.9 mm
- net N$4: track 24.2 -> 32.9 mm
- net N$3: track 30.1 -> 38.4 mm
- net N$6: track 29.5 -> 24.2 mm, vias 0 -> 1
- net N$7: track 30.7 -> 35.9 mm, vias 1 -> 0
- net N$5: track 34.8 -> 38.8 mm
- net VDD: track 26.2 -> 29.9 mm
- net +24V: track 19.0 -> 19.6 mm
- added copper zone on layer 1, net GND

Commit message: up
Parts:
- added SV2: DEBUG_H, con-lsta:FE10
- added X2, X3, X4: (no value), con-molex:KK-156-10
- moved R1 1.27 mm to (55.9, 14.0)
- moved R3 1.27 mm to (47.0, 14.0)
- moved R4 1.27 mm to (52.1, 14.0)
Connections:
- removed net VDD: C6.1, C7.1, IC1.19, R3.2, R4.1, SV1.7
- new net CS_JP3P11: IC1.15, R3.1, SV1.5, SV2.5
- new net EXT2_JP3P8: IC1.26, R4.2, SV1.9, SV2.9
- new net GND_JP4P8: C1.2, C2.2, C3.2, C4.2, C5.2, C6.2, C7.2, IC1.30, R1.1, X1.1
- new net MISO_JP4P1: IC1.18, SV1.1, SV2.1
- new net MOSI_JP4P2: IC1.16, SV1.3, SV2.3
- new net N$1: IC1.13, X2.1
- new net N$11: IC1.6, X4.3
- new net N$12: IC1.5, X4.2
- new net N$13: IC1.4, X4.1
- new net N$14: IC1.3, X3.8
- new net N$15: IC1.2, X3.7
- new net N$16: IC1.1, X3.6
- new net N$17: IC1.27, X2.3
- new net N$18: IC1.28, X2.4
- new net N$19: IC1.29, X2.5
- new net N$20: IC1.31, X2.6
- new net N$21: IC1.32, X2.7
- new net N$22: IC1.33, X2.8
- new net N$23: IC1.34, X3.1
- new net N$24: IC1.35, X3.2
- new net N$25: IC1.36, X3.3
- new net N$26: IC1.37, X3.4
- new net N$27: IC1.38, X3.5
- new net N$28: IC1.12, X4.8
- new net SCK_JP4P3: IC1.17, SV1.2, SV2.2
- new net VDD_JP4P5: C6.1, C7.1, IC1.19, R3.2, R4.1, SV1.7, SV2.7
- net +24V: now also X2.9, X3.9, X4.9
- net GND: now also SV2.8, X2.10, X3.10, X4.10; no longer C1.2, C2.2, C3.2, C4.2, C5.2, C6.2, C7.2, IC1.30, R1.1, X1.1
- net N$2: now also IC1.14, X2.2; no longer IC1.18, SV1.1
- net N$3: now also IC1.10, X4.6; no longer IC1.16, SV1.3
- net N$4: now also IC1.11, X4.7; no longer IC1.17, SV1.2
- net N$5: now also IC1.8, X4.5; no longer IC1.15, R3.1, SV1.5
- net N$6: now also SV2.6
- net N$7: now also IC1.7, X4.4; no longer IC1.26, R4.2, SV1.9
Routing:
- net +24V: track 19.6 -> 194.8 mm
- net GND_JP4P8: track 0.00 -> 149.0 mm, vias 0 -> 2
- net N$14: track 0.00 -> 71.6 mm, vias 0 -> 1
- net N$16: track 0.00 -> 58.4 mm
- net N$15: track 0.00 -> 57.7 mm
- net N$28: track 0.00 -> 56.9 mm, vias 0 -> 1
- net N$12: track 0.00 -> 56.5 mm, vias 0 -> 1
- net N$11: track 0.00 -> 55.0 mm, vias 0 -> 1
- net N$13: track 0.00 -> 54.1 mm, vias 0 -> 1
- net N$22: track 0.00 -> 52.9 mm, vias 0 -> 1
- net N$20: track 0.00 -> 47.6 mm, vias 0 -> 2
- net EXT2_JP3P8: track 0.00 -> 45.1 mm
- net N$18: track 0.00 -> 43.6 mm, vias 0 -> 2
- net N$21: track 0.00 -> 41.6 mm, vias 0 -> 1
- net N$26: track 0.00 -> 40.5 mm
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
Commit message: up
Parts:
- added C10, C8, C9: 0.1, rcl:C0805
- moved X3 6.35 mm to (73.7, 40.6)
- moved X4 3.81 mm to (88.9, 40.6)
Connections:
- removed net GND_JP4P8: C1.2, C2.2, C3.2, C4.2, C5.2, C6.2, C7.2, IC1.30, R1.1, X1.1
- net +24V: now also C10.1, C8.1, C9.1, IC2.37, IC2.38
- net GND: now also C1.2, C10.2, C2.2, C3.2, C4.2, C5.2, C6.2, C7.2, C8.2, C9.2, IC1.30, R1.1, X1.1
- net N$15: now also IC2.2
- net N$16: now also IC2.1
- net N$8: now also IC2.20
- net VDD_JP4P5: now also IC2.19
Routing:
- net GND_JP4P8: track 149.0 -> 0.00 mm, vias 2 -> 0
- net N$11: track 55.0 -> 93.7 mm, vias 1 -> 0
- net N$12: track 56.5 -> 85.9 mm, vias 1 -> 0
- net N$8: track 5.60 -> 34.3 mm
- net +24V: track 194.8 -> 168.2 mm, vias 0 -> 1
- net N$14: track 71.6 -> 47.5 mm, vias 1 -> 2
- net GND: track 0.00 -> 22.9 mm
- net VDD_JP4P5: track 38.9 -> 61.5 mm, vias 0 -> 3
- net N$13: track 54.1 -> 74.3 mm, vias 1 -> 0
- net N$5: track 69.2 -> 52.6 mm, vias 3 -> 2
- net N$17: track 40.3 -> 53.6 mm
- net N$4: track 64.1 -> 52.1 mm, vias 2 -> 0
- net N$23: track 33.5 -> 24.3 mm
- net N$6: track 33.6 -> 24.5 mm
- net N$25: track 34.9 -> 26.2 mm
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
Commit message: up
Parts:
- removed IC2: (no value), allegro2:TSSOP38
- added U1: TIC12400DCPR, TIC12400DCPR:SOP50P640X120-38N
Connections:
- net +24V: no longer IC2.37, IC2.38
- net CS_JP3P11: now also U1.15
- net EXT2_JP3P8: now also U1.24
- net GND: now also U1.28, U1.39, U1.40, U1.41, U1.42, U1.43, U1.44, U1.45, U1.46, U1.47, U1.48, U1.49, U1.50, U1.51, U1.52, U1.53, U1.54, U1.55, U1.56, U1.57, U1.58, U1.59, U1.60, U1.61, U1.62, U1.63, U1.9
- net MISO_JP4P1: now also U1.18
- net MOSI_JP4P2: now also U1.16
- net N$1: now also U1.13
- net N$10: now also U1.23
- net N$11: now also U1.6
- net N$12: now also U1.5
- net N$13: now also U1.4
- net N$14: now also U1.3
- net N$15: now also U1.2; no longer IC2.2
- net N$16: now also U1.1; no longer IC2.1
- net N$17: now also U1.25
- net N$18: now also U1.26
- net N$19: now also U1.27
- net N$2: now also U1.14
- net N$20: now also U1.29
- net N$21: now also U1.30
- net N$22: now also U1.31
- net N$23: now also U1.32
- net N$24: now also U1.33
- net N$25: now also U1.34
- net N$26: now also U1.35
- net N$27: now also U1.36, U1.37, U1.38
- net N$28: now also U1.12
- net N$3: now also U1.10
- net N$4: now also U1.11
- net N$5: now also U1.8
- net N$6: now also U1.21
- net N$7: now also U1.7
- net N$8: now also U1.20; no longer IC2.20
- net N$9: now also U1.22
- net SCK_JP4P3: now also U1.17
- net VDD_JP4P5: now also U1.19; no longer IC2.19
Routing:
- net +24V: track 168.2 -> 0.00 mm, vias 1 -> 0
- net N$11: track 93.7 -> 0.00 mm
- net N$12: track 85.9 -> 0.00 mm
- net N$13: track 74.3 -> 0.00 mm
- net VDD_JP4P5: track 61.5 -> 0.00 mm, vias 3 -> 0
- net N$15: track 55.4 -> 0.00 mm, vias 3 -> 0
- net N$16: track 54.7 -> 0.00 mm, vias 2 -> 0
- net N$17: track 53.6 -> 0.00 mm, vias 1 -> 0
- net N$28: track 53.4 -> 0.00 mm, vias 2 -> 0
- net N$5: track 52.6 -> 0.00 mm, vias 2 -> 0
- net N$4: track 52.1 -> 0.00 mm
- net N$7: track 51.4 -> 0.00 mm, vias 2 -> 0
- net N$3: track 50.7 -> 0.00 mm
- net N$14: track 47.5 -> 0.00 mm, vias 2 -> 0
- net EXT2_JP3P8: track 46.8 -> 0.00 mm
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
Commit message: up
Parts:
- moved X1 20.4 mm to (68.6, 73.7)
- moved IC1 10.2 mm to (48.3, 53.3)
- moved U1 8.89 mm to (48.3, 19.1)
- moved R1 8.03 mm to (63.5, 16.5), turned to 270 degrees
- moved R3 6.48 mm to (40.6, 12.7), turned to 180 degrees
- moved R4 4.02 mm to (55.9, 12.7), turned to 0 degrees
- moved C2 3.59 mm to (59.7, 24.1)
- moved C3 3.59 mm to (59.7, 26.7)
- moved C1 2.54 mm to (59.7, 21.6)
- moved C6 2.54 mm to (36.8, 16.5)
- moved C7 2.54 mm to (36.8, 19.1)
- moved X3 1.27 mm to (73.7, 41.9)
- moved X4 1.27 mm to (88.9, 41.9)
Routing:
- net +24V: track 0.00 -> 175.4 mm, vias 0 -> 1
- net N$11: track 0.00 -> 146.6 mm, vias 0 -> 2
- net N$7: track 0.00 -> 145.7 mm, vias 0 -> 2
- net N$12: track 0.00 -> 137.2 mm, vias 0 -> 2
- net N$13: track 0.00 -> 122.5 mm, vias 0 -> 2
- net GND: track 0.00 -> 121.1 mm, vias 0 -> 12
- net N$16: track 0.00 -> 115.4 mm
- net N$24: track 0.00 -> 110.6 mm, vias 0 -> 1
- net N$15: track 0.00 -> 104.0 mm, vias 0 -> 4
- net N$17: track 0.00 -> 101.3 mm, vias 0 -> 1
- net N$5: track 0.00 -> 99.5 mm
- net N$3: track 0.00 -> 97.8 mm, vias 0 -> 3
- net N$27: track 0.00 -> 94.9 mm
- net N$14: track 0.00 -> 93.9 mm, vias 0 -> 2
- net N$23: track 0.00 -> 89.6 mm, vias 0 -> 2
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
Commit message: up
Parts:
- removed IC1: (no value), ic-package:DIL40
- added D1: ES2D, diode:SMB
- X2: value (none) -> INPUT1
- X3: value (none) -> INPUT2
- X4: value (none) -> INPUT3
- moved X1 65.9 mm to (90.2, 11.4), turned to 270 degrees
- moved C5 37.0 mm to (64.8, 30.5), turned to 270 degrees
- moved C4 34.3 mm to (62.2, 30.5), turned to 270 degrees
- moved X2 18.9 mm to (35.6, 55.9)
- moved C9 15.5 mm to (78.7, 39.4)
- moved C10 15.5 mm to (94.0, 39.4)
- moved C8 15.3 mm to (29.2, 40.6)
- moved X3 14.0 mm to (72.4, 55.9)
- moved X4 14.0 mm to (87.6, 55.9)
- moved R3 6.48 mm to (47.0, 14.0), turned to 90 degrees
- moved U1 5.08 mm to (48.3, 24.1)
- moved R4 1.27 mm to (54.6, 12.7)
Connections:
- removed net MOSI_JP4P2: IC1.16, SV1.3, SV2.3, U1.16
- removed net SCK_JP4P3: IC1.17, SV1.2, SV2.2, U1.17
- new net MOSI_JP4P3: SV1.2, SV2.2, U1.17
- new net N$29: D1.A, X1.2, X1.3
- new net SCK_JP4P2: SV1.3, SV2.3, U1.16
- net +24V: now also D1.C, U1.37, U1.38; no longer IC1.39, IC1.40, X1.2, X1.3
- net CS_JP3P11: no longer IC1.15
- net EXT2_JP3P8: no longer IC1.26
- net GND: no longer IC1.30, IC1.9
- net MISO_JP4P1: no longer IC1.18
- net N$1: no longer IC1.13
- net N$10: no longer IC1.25
- net N$11: no longer IC1.6
- net N$12: no longer IC1.5
- net N$13: no longer IC1.4
- net N$14: no longer IC1.3
- net N$15: no longer IC1.2
- net N$16: no longer IC1.1
- net N$17: no longer IC1.27
- net N$18: no longer IC1.28
- net N$19: no longer IC1.29
- net N$2: no longer IC1.14
- net N$20: no longer IC1.31
- net N$21: no longer IC1.32
- net N$22: no longer IC1.33
- net N$23: no longer IC1.34
- net N$24: no longer IC1.35
- net N$25: no longer IC1.36
- net N$26: no longer IC1.37
- net N$27: no longer IC1.38, U1.37, U1.38
- net N$28: no longer IC1.12
- net N$3: no longer IC1.10
- net N$4: no longer IC1.11
- net N$5: no longer IC1.8
- net N$6: no longer IC1.23
- net N$7: no longer IC1.7
- net N$8: no longer IC1.22
- net N$9: no longer IC1.24
- net VDD_JP4P5: no longer IC1.19
Routing:
- net GND: track 121.1 -> 21.3 mm, vias 12 -> 16
- net N$16: track 115.4 -> 37.5 mm, vias 0 -> 1
- net N$7: track 145.7 -> 69.3 mm
- net N$12: track 137.2 -> 69.1 mm
- net N$15: track 104.0 -> 38.4 mm, vias 4 -> 1
- net N$11: track 146.6 -> 82.9 mm, vias 2 -> 1
- net N$24: track 110.6 -> 53.3 mm
- net N$14: track 93.9 -> 38.1 mm
- net N$27: track 94.9 -> 39.5 mm, vias 0 -> 1
- net +24V: track 175.4 -> 121.8 mm, vias 1 -> 3
- net MOSI_JP4P2: track 42.5 -> 0.00 mm, vias 2 -> 0
- net N$13: track 122.5 -> 80.6 mm, vias 2 -> 1
- net SCK_JP4P3: track 40.7 -> 0.00 mm, vias 1 -> 0
- net N$20: track 87.9 -> 47.9 mm, vias 3 -> 1
- net EXT2_JP3P8: track 64.0 -> 25.9 mm, vias 2 -> 1
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Other:
- board text added: "SPI 4MHz MAX"
- board text added: "TIC12400 input board V1.0"

Commit message: up
Parts:
- added U2: MCZ33996EK, MCZ33996EK:SOP65P1030X265-33N
- moved C8 34.3 mm to (63.5, 39.4)
- moved X2 21.6 mm to (57.1, 55.9)
Connections:
- net +24V: now also U2.6
- net GND: now also U2.10, U2.23, U2.24, U2.25, U2.26, U2.33, U2.7, U2.8, U2.9
- net MISO_JP4P1: now also U2.22
- net MOSI_JP4P3: now also U2.19
- net N$6: now also U2.27
- net SCK_JP4P2: now also U2.11
- net VDD_JP4P5: now also U2.3
Routing:
- net GND: track 21.3 -> 114.9 mm, vias 16 -> 2
- net +24V: track 121.8 -> 168.2 mm, vias 3 -> 2
- net N$6: track 39.2 -> 78.8 mm, vias 0 -> 1
- net SCK_JP4P2: track 19.2 -> 50.1 mm, vias 0 -> 1
- net N$23: track 62.4 -> 89.4 mm
- net VDD_JP4P5: track 58.4 -> 80.5 mm
- net MISO_JP4P1: track 20.9 -> 42.0 mm, vias 1 -> 2
- net N$7: track 69.3 -> 90.0 mm, vias 2 -> 1
- net N$12: track 69.1 -> 86.9 mm, vias 2 -> 1
- net N$22: track 42.4 -> 25.4 mm, vias 0 -> 3
- net N$18: track 61.7 -> 45.0 mm, vias 1 -> 3
- net MOSI_JP4P3: track 20.0 -> 36.2 mm, vias 1 -> 2
- net N$17: track 67.2 -> 79.9 mm, vias 1 -> 0
- net N$27: track 39.5 -> 51.7 mm
- net N$19: track 53.4 -> 41.3 mm
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
Commit message: up
Parts:
- added C11, C13, C14: 0.1, rcl:C0805
- added C12: 10uf, rcl:C0805
- added D2: ES2D, diode:SMB
- added X5: 22-23-2031, con-molex:22-23-2031
- added X6: OUTPUT1, con-molex:KK-156-10
- added X7: OUTPUT2, con-molex:KK-156-10
Connections:
- new net N$30: D2.A, X5.2, X5.3
- new net N$32: C11.1, C12.1, C13.1, D2.C, U2.6, X6.9, X7.9
- new net N$33: SV1.4, SV2.4, U2.14
- new net N$34: SV1.10, SV2.10, U2.30
- new net N$35: U2.1, X6.1
- new net N$36: U2.2, X6.2
- new net N$37: U2.4, X6.3
- new net N$38: U2.5, X6.4
- new net N$39: U2.12, X6.5
- new net N$40: U2.13, X6.6
- new net N$41: U2.15, X6.7
- new net N$42: U2.16, X6.8
- new net N$43: U2.17, X7.1
- new net N$44: U2.18, X7.2
- new net N$45: U2.20, X7.3
- new net N$46: U2.21, X7.4
- new net N$47: U2.28, X7.5
- new net N$48: U2.29, X7.6
- new net N$49: U2.31, X7.7
- new net N$50: U2.32, X7.8
- net +24V: no longer U2.6
- net GND: now also C11.2, C12.2, C13.2, C14.2, X5.1, X6.10, X7.10
- net VDD_JP4P5: now also C14.1
Routing:
- net N$32: track 0.00 -> 71.4 mm, vias 0 -> 2
- net +24V: track 168.2 -> 104.3 mm, vias 2 -> 0
- net N$43: track 0.00 -> 60.4 mm
- net N$44: track 0.00 -> 56.8 mm, vias 0 -> 1
- net N$34: track 0.00 -> 55.4 mm
- net N$36: track 0.00 -> 50.2 mm
- net N$45: track 0.00 -> 49.9 mm
- net N$35: track 0.00 -> 48.1 mm, vias 0 -> 1
- net N$37: track 0.00 -> 47.9 mm
- net N$38: track 0.00 -> 47.9 mm, vias 0 -> 1
- net N$46: track 0.00 -> 47.4 mm, vias 0 -> 1
- net N$39: track 0.00 -> 41.3 mm
- net N$41: track 0.00 -> 40.8 mm
- net N$40: track 0.00 -> 39.3 mm, vias 0 -> 1
- net N$33: track 0.00 -> 37.1 mm
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