File: tic12400.brd (EAGLE design)
At the start: 100 x 80 mm, 30 parts, among them U1 TIC12400DCPR, U2 MCZ33996EK, X1 22-23-2031, X2 INPUT1, X3 INPUT2, X4 INPUT3, X5 22-23-2031, X6 OUTPUT1, X7 OUTPUT2

Commit message: up
Routing:
- net GND: track 117.4 -> 93.1 mm, vias 4 -> 17
- net N$18: track 46.1 -> 67.8 mm, vias 1 -> 0
- net N$5: track 81.1 -> 97.0 mm, vias 0 -> 1
- net N$14: track 40.6 -> 54.6 mm
- net N$4: track 82.1 -> 94.7 mm, vias 1 -> 0
- net N$27: track 59.0 -> 47.6 mm
- net N$15: track 57.8 -> 48.0 mm
- net N$16: track 54.8 -> 45.4 mm
- net N$39: track 41.3 -> 50.2 mm
- net N$35: track 48.1 -> 55.6 mm, vias 1 -> 0
- net VDD_JP4P5: track 74.2 -> 81.4 mm, vias 4 -> 3
- net N$38: track 47.9 -> 40.7 mm
- net SCK_JP4P2: track 59.8 -> 52.8 mm
- net N$1: track 66.2 -> 60.0 mm
- net +24V: track 104.3 -> 110.4 mm, vias 0 -> 2
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Other:
- board text added: "TIC12400 MC33996 I/O board V1.1"
- board text removed: "TIC12400 input board V1.0"

Commit message: up
Parts:
- added F1, F2: 1206L020, polyfuse-smd_10:1206L
- added R2, R5: 100, rcl:R0805
- moved X5 5.08 mm to (7.62, 22.9)
- moved D2 2.54 mm to (11.4, 10.2)
- moved R3 1.27 mm to (48.3, 14.0)
Connections:
- new net MOSI_SIG: R5.1, U1.17, U2.19
- new net N$31: D2.A, F1.2
- new net N$51: D1.A, F2.2
- new net SCK_SIG: R2.1, U1.16, U2.11
- net MOSI_JP4P3: now also R5.2; no longer U1.17, U2.19
- net N$29: now also F2.1; no longer D1.A
- net N$30: now also C11.1, C12.1, C13.1, D2.C, U2.6; no longer D2.A, X5.2, X5.3
- net N$32: now also F1.1, X5.2, X5.3; no longer C11.1, C12.1, C13.1, D2.C, U2.6
- net SCK_JP4P2: now also R2.2; no longer U1.16, U2.11
Routing:
- net SCK_JP4P2: track 52.8 -> 9.02 mm, vias 2 -> 0
- net N$30: track 8.00 -> 51.7 mm, vias 0 -> 3
- net SCK_SIG: track 0.00 -> 42.6 mm, vias 0 -> 2
- net N$4: track 94.7 -> 60.8 mm, vias 0 -> 1
- net MOSI_JP4P3: track 41.1 -> 9.06 mm, vias 2 -> 0
- net MOSI_SIG: track 0.00 -> 28.2 mm, vias 0 -> 2
- net N$28: track 58.8 -> 83.8 mm, vias 1 -> 0
- net N$32: track 71.2 -> 48.5 mm, vias 2 -> 0
- net N$18: track 67.8 -> 45.6 mm, vias 0 -> 1
- net N$5: track 97.0 -> 75.4 mm, vias 1 -> 2
- net N$15: track 48.0 -> 66.7 mm, vias 1 -> 0
- net VDD_JP4P5: track 81.4 -> 96.4 mm
- net N$3: track 88.2 -> 73.5 mm
- net N$25: track 62.4 -> 48.8 mm, vias 2 -> 1
- net +24V: track 110.4 -> 97.2 mm, vias 2 -> 3
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
Commit message: up
Parts:
- added C15: 1uf, rcl:C0805
- added C16: 0.1, rcl:C0805
- added LED1: SPI ACT, led:CHIP-LED0805
- added LED2: POWER, led:CHIP-LED0805
- added Q1: CSTCR6M00G53Z, murata-filter:CSTCR6M
- added R6, R7, R8: 390, rcl:R0805
- added SV3: MCP2210_GPIO, con-lsta:FE10
- added U3: MCP2210-I/SO, MCP2210-I_SO:SOP65P780X200-20N
- added X8: MINI-USB-32005-201, con-cypressindustries:32005-201
- moved D1 21.7 mm to (72.4, 29.2)
- moved X1 17.8 mm to (88.9, 29.2)
- moved F2 15.3 mm to (80.0, 29.2)
Connections:
- removed net VDD_JP4P5: C14.1, C6.1, C7.1, R3.2, R4.1, SV1.7, SV2.7, U1.19, U2.3
- new net N$52: C15.1, U3.17
- new net N$53: Q1.1, U3.3
- new net N$54: R6.1, U3.4
- new net N$55: U3.19, X8.3
- new net N$56: U3.18, X8.2
- new net N$57: Q1.3, U3.2
- new net N$58: LED2.A, R7.2
- new net N$59: LED1.A, R8.2
- new net N$60: R8.1, SV3.4, U3.8
- new net N$61: SV3.1, U3.5
- new net N$62: SV3.2, U3.6
- new net N$63: SV3.3, U3.7
- new net N$64: SV3.5, U3.10
- new net N$65: SV3.8, U3.15
- new net VDD: C14.1, C16.1, C6.1, C7.1, R3.2, R4.1, R6.2, R7.1, SV1.7, SV2.7, U1.19, U2.3, U3.1, X8.1
- net CS_JP3P11: now also SV3.6, U3.12
- net EXT2_JP3P8: now also SV3.7, U3.14
- net GND: now also C15.2, C16.2, LED1.C, LED2.C, Q1.2, SV3.10, U3.20, X8.5
- net MISO_JP4P1: now also U3.13
- net MOSI_SIG: now also U3.9
- net N$33: now also SV3.9, U3.16
- net SCK_SIG: now also U3.11
Routing:
- net VDD: track 0.00 -> 151.5 mm, vias 0 -> 6
- net VDD_JP4P5: track 96.4 -> 0.00 mm, vias 3 -> 0
- net N$33: track 41.2 -> 136.4 mm, vias 0 -> 2
- net CS_JP3P11: track 24.1 -> 91.9 mm, vias 0 -> 4
- net GND: track 86.9 -> 151.6 mm, vias 12 -> 19
- net MOSI_SIG: track 28.2 -> 84.9 mm, vias 2 -> 5
- net SCK_SIG: track 42.6 -> 97.0 mm, vias 2 -> 5
- net MISO_JP4P1: track 37.3 -> 87.8 mm, vias 2 -> 3
- net EXT2_JP3P8: track 26.3 -> 76.6 mm, vias 1 -> 2
- net N$60: track 0.00 -> 48.9 mm
- net N$62: track 0.00 -> 34.7 mm, vias 0 -> 1
- net N$58: track 0.00 -> 28.3 mm
- net N$63: track 0.00 -> 24.4 mm, vias 0 -> 1
- net N$61: track 0.00 -> 24.1 mm, vias 0 -> 1
- net N$15: track 66.7 -> 43.0 mm, vias 0 -> 2
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Other:
- board text added: "TIC12400 MC33996 I/O board V1.3"
- board text removed: "TIC12400 MC33996 I/O board V1.1"

Commit message: up
Parts:
- added R9: 100, rcl:R0805
- added TP1, TP2, TP3: PTR1B1,27, testpad:B1,27
Connections:
- new net N$66: R9.1, U3.13
- net GND: now also TP3.TP
- net MISO_JP4P1: now also R9.2; no longer U3.13
- net N$53: now also TP2.TP
- net N$54: now also TP1.TP
Routing:
- net N$66: track 0.00 -> 19.7 mm, vias 0 -> 2
- net MISO_JP4P1: track 87.8 -> 78.1 mm, vias 3 -> 5
- net N$53: track 6.91 -> 13.6 mm
- net GND: track 151.6 -> 156.0 mm
- net N$54: track 11.2 -> 13.8 mm

Commit message: up
Connections:
- net N$30: now also X6.9, X7.9
- net N$32: no longer X6.9, X7.9
Routing:
- net N$32: track 47.1 -> 8.22 mm
- net N$30: track 59.2 -> 81.6 mm, vias 3 -> 4
Other:
- board text added: "TIC12400 MC33996 I/O board V1.4"
- board text removed: "TIC12400 MC33996 I/O board V1.3"
Changed lines of the file:
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@@
 <wire x1="100" y1="80" x2="0" y2="80" width="0" layer="20"/>
 <wire x1="0" y1="80" x2="0" y2="0" width="0" layer="20"/>
-<text x="5.08" y="36.83" size="1.27" layer="1" font="vector" ratio="20" rot="R90">TIC12400 MC33996  I/O board V1.3</text>
+<text x="5.08" y="36.83" size="1.27" layer="1" font="vector" ratio="20" rot="R90">TIC12400 MC33996  I/O board V1.4</text>
 <text x="29.21" y="6.35" size="1.778" layer="1" font="vector" ratio="20" rot="R180">SPI 4MHz MAX</text>
 <hole x="5.08" y="74.93" drill="2.54"/>
@@
 <attribute name="MF" value="NXP USA" x="21.59" y="22.86" size="1.778" layer="27" display="off"/>
 <attribute name="MP" value="MCZ33996EK" x="21.59" y="22.86" size="1.778" layer="27" display="off"/>
+<attribute name="NAME" x="18.185309375" y="29.168690625" size="1.27175" layer="25"/>
 <attribute name="NAME" x="18.189590625" y="29.16075" size="1.27015" layer="25"/>
-<attribute name="NAME" x="18.185309375" y="29.168690625" size="1.27175" layer="25"/>
 <attribute name="PACKAGE" value="SOIC-32 NXP Semiconductors" x="21.59" y="22.86" size="1.778" layer="27" display="off"/>
 <attribute name="PRICE" value="None" x="21.59" y="22.86" size="1.778" layer="27" display="off"/>
@@
 </signal>
 <signal name="N$32" class="1">
-<contactref element="X6" pad="9"/>
-<contactref element="X7" pad="9"/>
 <contactref element="X5" pad="2"/>
 <contactref element="X5" pad="3"/>
@@
 <wire x1="7.62" y1="20.2692" x2="7.62" y2="20.32" width="0.3048" layer="1"/>
 <wire x1="7.62" y1="20.32" x2="7.62" y2="22.86" width="0.3048" layer="1"/>
-<wire x1="31.6992" y1="42.0624" x2="15.24" y2="42.0624" width="0.3048" layer="16"/>
-<wire x1="15.24" y1="42.0624" x2="15.24" y2="42.02" width="0.3048" layer="16"/>
-<wire x1="31.6992" y1="42.0624" x2="31.75" y2="42.02" width="0.3048" layer="16"/>
-<wire x1="7.62" y1="23.0886" x2="7.62" y2="22.86" width="0.3048" layer="16"/>
-<wire x1="12.3444" y1="27.813" x2="7.62" y2="23.0886" width="0.3048" layer="16"/>
-<wire x1="12.3444" y1="39.0906" x2="12.3444" y2="27.813" width="0.3048" layer="16"/>
-<wire x1="15.1638" y1="41.91" x2="12.3444" y2="39.0906" width="0.3048" layer="16"/>
-<wire x1="15.1638" y1="41.91" x2="15.24" y2="42.02" width="0.3048" layer="16"/>
 </signal>
 <signal name="N$33">
@@
 <wire x1="16.002" y1="20.6502" x2="16.764" y2="20.6502" width="0.3048" layer="1"/>
 <wire x1="12.3444" y1="24.3078" x2="16.002" y2="20.6502" width="0.3048" layer="1"/>
-<wire x1="12.3444" y1="47.0916" x2="12.3444" y2="24.3078" width="0.3048" layer="1"/>
 <wire x1="12.3444" y1="54.9402" x2="12.3444" y2="47.0916" width="0.3048" layer="16"/>
 <wire x1="15.24" y1="57.8358" x2="12.3444" y2="54.9402" width="0.3048" layer="16"/>
@@
 <wire x1="15.24" y1="57.8358" x2="15.24" y2="57.86" width="0.3048" layer="16"/>
 <via x="12.3444" y="47.0916" extent="1-16" drill="0.35"/>
+<wire x1="12.3444" y1="47.0916" x2="12.3444" y2="24.3078" width="0.3048" layer="1"/>
 </signal>
 <signal name="N$40" class="1">
@@
 <wire x1="37.5666" y1="40.3098" x2="38.1" y2="40.3098" width="0.3048" layer="1"/>
 <wire x1="36.3474" y1="39.0906" x2="37.5666" y2="40.3098" width="0.3048" layer="1"/>
-<wire x1="22.098" y1="24.8412" x2="36.3474" y2="39.0906" width="0.3048" layer="16"/>
+<wire x1="22.098" y1="24.8412" x2="35.5092" y2="38.2524" width="0.3048" layer="16"/>
+<wire x1="35.5092" y1="38.2524" x2="36.3474" y2="39.0906" width="0.3048" layer="16"/>
 <wire x1="18.288" y1="24.8412" x2="22.098" y2="24.8412" width="0.3048" layer="16"/>
 <wire x1="17.9832" y1="24.8412" x2="18.288" y2="24.8412" width="0.3048" layer="1"/>
@@
 <via x="18.288" y="24.8412" extent="1-16" drill="0.35"/>
 <via x="14.7828" y="16.6116" extent="1-16" drill="0.35"/>
+<contactref element="X6" pad="9"/>
+<contactref element="X7" pad="9"/>
+<wire x1="17.4498" y1="39.7764" x2="15.24" y2="41.9862" width="0.3048" layer="1"/>
+<wire x1="17.4498" y1="39.3954" x2="17.4498" y2="39.7764" width="0.3048" layer="16"/>
+<wire x1="18.1356" y1="38.7096" x2="17.4498" y2="39.3954" width="0.3048" layer="16"/>
+<wire x1="18.1356" y1="29.1084" x2="18.1356" y2="38.7096" width="0.3048" layer="16"/>
+<wire x1="16.0782" y1="27.051" x2="18.1356" y2="29.1084" width="0.3048" layer="16"/>
+<wire x1="15.24" y1="41.9862" x2="15.24" y2="42.02" width="0.3048" layer="1"/>
+<wire x1="35.5092" y1="38.2524" x2="31.7754" y2="41.9862" width="0.3048" layer="16"/>
+<wire x1="31.7754" y1="41.9862" x2="31.75" y2="42.02" width="0.3048" layer="16"/>
+<via x="17.4498" y="39.7764" extent="1-16" drill="0.35"/>
 </signal>
 <signal name="N$31" class="1">

Commit message: up
Parts:
- added OS1: OSC-OE-CFPS-73, IQD-Frequency-Products:7.2X5.2-4-PAD
- moved D1 5.08 mm to (72.4, 34.3)
- turned C15 to 90 degrees
Connections:
- removed net N$52: C15.1, U3.17
- net GND: now also OS1.2
- net N$57: now also OS1.3
- net VDD: now also C15.1, OS1.1, OS1.4, U3.17
Routing:
- net VDD: track 151.4 -> 171.9 mm, vias 6 -> 8
- net N$33: track 136.4 -> 146.7 mm
- net N$57: track 7.39 -> 12.8 mm, vias 0 -> 2
- net GND: track 156.0 -> 151.9 mm
- net N$52: track 3.82 -> 0.00 mm
- net N$51: track 4.08 -> 6.77 mm
- net N$65: track 15.5 -> 17.5 mm

Commit message: up
Parts:
- added TP4: PTR1B1,27, testpad:B1,27
- moved TP1 5.39 mm to (73.7, 17.8)
Connections:
- new net N$52: C15.1, U3.17
- net N$57: now also TP4.TP
- net VDD: no longer C15.1, U3.17
Routing:
- net VDD: track 171.9 -> 157.6 mm, vias 8 -> 6
- net N$52: track 0.00 -> 4.42 mm
- net N$57: track 12.8 -> 15.4 mm
- net N$54: track 13.8 -> 12.5 mm
Other:
- board text added: "TIC12400 MC33996 I/O board V1.5"
- board text removed: "TIC12400 MC33996 I/O board V1.4"
Changed lines of the file:
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@@
 <wire x1="100" y1="80" x2="0" y2="80" width="0" layer="20"/>
 <wire x1="0" y1="80" x2="0" y2="0" width="0" layer="20"/>
-<text x="5.08" y="36.83" size="1.27" layer="1" font="vector" ratio="20" rot="R90">TIC12400 MC33996  I/O board V1.4</text>
+<text x="5.08" y="36.83" size="1.27" layer="1" font="vector" ratio="20" rot="R90">TIC12400 MC33996  I/O board V1.5</text>
 <text x="29.21" y="6.35" size="1.778" layer="1" font="vector" ratio="20" rot="R180">SPI 4MHz MAX</text>
 <hole x="5.08" y="74.93" drill="2.54"/>
@@
 <attribute name="MF" value="NXP USA" x="21.59" y="22.86" size="1.778" layer="27" display="off"/>
 <attribute name="MP" value="MCZ33996EK" x="21.59" y="22.86" size="1.778" layer="27" display="off"/>
+<attribute name="NAME" x="18.189590625" y="29.16075" size="1.27015" layer="25"/>
 <attribute name="NAME" x="18.185309375" y="29.168690625" size="1.27175" layer="25"/>
-<attribute name="NAME" x="18.189590625" y="29.16075" size="1.27015" layer="25"/>
 <attribute name="PACKAGE" value="SOIC-32 NXP Semiconductors" x="21.59" y="22.86" size="1.778" layer="27" display="off"/>
 <attribute name="PRICE" value="None" x="21.59" y="22.86" size="1.778" layer="27" display="off"/>
@@
 <attribute name="VALUE" x="76.835" y="16.51" size="1.27" layer="27" rot="R180"/>
 </element>
-<element name="TP1" library="testpad" library_urn="urn:adsk.eagle:library:385" package="B1,27" package3d_urn="urn:adsk.eagle:package:27944/2" value="PTR1B1,27" x="69.85" y="21.59" smashed="yes">
-<attribute name="NAME" x="69.215" y="22.606" size="1.27" layer="25" ratio="10"/>
-<attribute name="POPULARITY" value="2" x="69.85" y="21.59" size="1.778" layer="27" display="off"/>
-<attribute name="TP_SIGNAL_NAME" value="" x="69.85" y="21.59" size="1.778" layer="27" display="off"/>
-<attribute name="VALUE" x="69.215" y="20.828" size="0.0254" layer="27"/>
+<element name="TP1" library="testpad" library_urn="urn:adsk.eagle:library:385" package="B1,27" package3d_urn="urn:adsk.eagle:package:27944/2" value="PTR1B1,27" x="73.66" y="17.78" smashed="yes">
+<attribute name="NAME" x="73.025" y="18.796" size="1.27" layer="25" ratio="10"/>
+<attribute name="POPULARITY" value="2" x="73.66" y="17.78" size="1.778" layer="27" display="off"/>
+<attribute name="TP_SIGNAL_NAME" value="" x="73.66" y="17.78" size="1.778" layer="27" display="off"/>
+<attribute name="VALUE" x="73.025" y="17.018" size="0.0254" layer="27"/>
 </element>
 <element name="TP2" library="testpad" library_urn="urn:adsk.eagle:library:385" package="B1,27" package3d_urn="urn:adsk.eagle:package:27944/2" value="PTR1B1,27" x="83.82" y="25.4" smashed="yes">
@@
 <attribute name="POPULARITY" value="0" x="72.39" y="27.94" size="1.778" layer="27" rot="R180" display="off"/>
 <attribute name="VALUE" x="76.5092" y="33.433" size="1.27" layer="27" rot="R180"/>
+</element>
+<element name="TP4" library="testpad" library_urn="urn:adsk.eagle:library:385" package="B1,27" package3d_urn="urn:adsk.eagle:package:27944/2" value="PTR1B1,27" x="69.85" y="21.59" smashed="yes">
+<attribute name="NAME" x="69.215" y="22.606" size="1.27" layer="25" ratio="10"/>
+<attribute name="POPULARITY" value="2" x="69.85" y="21.59" size="1.778" layer="27" display="off"/>
+<attribute name="TP_SIGNAL_NAME" value="" x="69.85" y="21.59" size="1.778" layer="27" display="off"/>
+<attribute name="VALUE" x="69.215" y="20.828" size="0.0254" layer="27"/>
 </element>
 </elements>
@@
 <contactref element="U3" pad="4"/>
 <contactref element="R6" pad="1"/>
-<wire x1="77.8002" y1="19.05" x2="69.8754" y2="19.05" width="0.1524" layer="1"/>
+<wire x1="77.8002" y1="19.05" x2="73.6854" y2="19.05" width="0.1524" layer="1"/>
+<wire x1="73.6854" y1="19.05" x2="69.53" y2="19.05" width="0.1524" layer="1"/>
 <wire x1="78.7146" y1="19.9644" x2="77.8002" y2="19.05" width="0.1524" layer="1"/>
 <wire x1="80.3148" y1="19.9644" x2="78.7146" y2="19.9644" width="0.1524" layer="1"/>
 <wire x1="80.3148" y1="19.9644" x2="80.315" y2="20.025" width="0.1524" layer="1"/>
 <contactref element="TP1" pad="TP"/>
-<wire x1="69.8754" y1="19.05" x2="69.8754" y2="21.5646" width="0.1524" layer="1"/>
-<wire x1="69.8754" y1="21.5646" x2="69.85" y2="21.59" width="0.1524" layer="1"/>
-<wire x1="69.8754" y1="19.05" x2="69.53" y2="19.05" width="0.1524" layer="1"/>
+<wire x1="73.6854" y1="19.05" x2="73.6854" y2="17.8308" width="0.1524" layer="1"/>
+<wire x1="73.6854" y1="17.8308" x2="73.66" y2="17.78" width="0.1524" layer="1"/>
 </signal>
 <signal name="VDD" class="1">
@@
 <wire x1="67.63" y1="19.05" x2="67.63" y2="23.815" width="0.3048" layer="1"/>
 <wire x1="67.63" y1="23.815" x2="67.6656" y2="23.8506" width="0.3048" layer="1"/>
-<contactref element="U3" pad="17"/>
-<contactref element="C15" pad="1"/>
-<wire x1="81.8388" y1="22.2504" x2="84.1248" y2="19.9644" width="0.3048" layer="16"/>
-<wire x1="80.5434" y1="22.2504" x2="81.8388" y2="22.2504" width="0.3048" layer="1"/>
-<wire x1="80.391" y1="22.098" x2="80.5434" y2="22.2504" width="0.3048" layer="1"/>
-<wire x1="80.391" y1="22.098" x2="80.315" y2="21.975" width="0.3048" layer="1"/>
-<via x="81.8388" y="22.2504" extent="1-16" drill="0.35"/>
-<wire x1="88.5444" y1="19.9644" x2="88.6968" y2="19.812" width="0.3048" layer="1"/>
-<wire x1="87.3252" y1="19.9644" x2="88.5444" y2="19.9644" width="0.3048" layer="1"/>
-<wire x1="87.3252" y1="19.9644" x2="87.325" y2="20.025" width="0.3048" layer="1"/>
-<wire x1="84.1248" y1="19.9644" x2="88.8492" y2="19.9644" width="0.3048" layer="16"/>
-<wire x1="88.8492" y1="19.9644" x2="88.6968" y2="19.812" width="0.3048" layer="1"/>
-<via x="88.8492" y="19.9644" extent="1-16" drill="0.35"/>
-<wire x1="89.4588" y1="20.574" x2="91.44" y2="20.574" width="0.3048" layer="1"/>
-<wire x1="88.8492" y1="19.9644" x2="89.4588" y2="20.574" width="0.3048" layer="1"/>
-<wire x1="91.44" y1="20.574" x2="91.44" y2="20.64" width="0.3048" layer="1"/>
 <contactref element="OS1" pad="4"/>
 <contactref element="OS1" pad="1"/>
@@
 <via x="71.1708" y="24.5364" extent="1-16" drill="0.35"/>
 <via x="71.7804" y="23.1648" extent="1-16" drill="0.35"/>
+<contactref element="TP4" pad="TP"/>
+<wire x1="70.2564" y1="21.6408" x2="69.8754" y2="21.6408" width="0.1524" layer="1"/>
+<wire x1="71.7804" y1="23.1648" x2="70.2564" y2="21.6408" width="0.1524" layer="1"/>
+<wire x1="69.8754" y1="21.6408" x2="69.85" y2="21.59" width="0.1524" layer="1"/>
 </signal>
 <signal name="N$58">
@@
 <via x="81.8388" y="11.5062" extent="1-16" drill="0.35"/>
 </signal>
+<signal name="N$52" class="1">
+<contactref element="U3" pad="17"/>
+<contactref element="C15" pad="1"/>
+<wire x1="88.8492" y1="20.574" x2="91.44" y2="20.574" width="0.3048" layer="1"/>
+<wire x1="88.3158" y1="20.0406" x2="88.8492" y2="20.574" width="0.3048" layer="1"/>
+<wire x1="87.3252" y1="20.0406" x2="88.3158" y2="20.0406" width="0.3048" layer="1"/>
+<wire x1="91.44" y1="20.574" x2="91.44" y2="20.64" width="0.3048" layer="1"/>
+<wire x1="87.3252" y1="20.0406" x2="87.325" y2="20.025" width="0.3048" layer="1"/>
+</signal>
 </signals>

Commit message: up
Parts:
- renumbered LED1 to LED3
Connections:
- net GND: no longer LED3.C
- net N$33: no longer SV1.4, SV2.4, U2.14
- net N$59: now also LED3.C; no longer LED3.A
- net N$65: now also SV1.4, SV2.4, U2.14
- net VDD: now also LED3.A
Routing:
- net N$33: track 146.7 -> 27.1 mm, vias 2 -> 1
- net N$65: track 17.5 -> 122.5 mm, vias 0 -> 1
- net N$59: track 19.3 -> 36.1 mm
- net VDD: track 157.6 -> 164.3 mm
- net GND: track 151.9 -> 156.7 mm, vias 19 -> 18
