File: tic12400.brd (EAGLE design)
At the start: 100 x 80 mm, 57 parts, among them Q1 CSTCR6M00G53Z, U1 TIC12400DCPR, U2 MCZ33996EK, U3 MCP2210-I/SO, U4 BMX160, X1 22-23-2031, X2 INPUT1, X3 INPUT2, X4 INPUT3, X5 22-23-2031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

Commit message: up
Parts:
- added IC1: 7805TV, linear:TO220V
Connections:
- new net N$69: IC1.1, X8.1
- net GND: now also IC1.2
- net N$52: no longer C15.1, C17.1, U3.17
- net VDD: now also C15.1, C17.1, IC1.3, U3.17; no longer X8.1
Routing:
- net N$69: track 0.00 -> 83.1 mm, vias 0 -> 8
- net VDD: track 162.0 -> 212.0 mm, vias 6 -> 15
- net N$52: track 97.9 -> 91.8 mm, vias 4 -> 3

Commit message: up
Connections:
- removed net N$52: C18.1, OS1.1, OS1.4, U4.5, U4.8
- net VDD: now also C18.1, OS1.1, OS1.4, U4.5, U4.8
Routing:
- net N$52: track 91.8 -> 0.00 mm, vias 3 -> 0
- net VDD: track 212.0 -> 236.3 mm, vias 15 -> 16
- net GND: track 174.1 -> 175.9 mm, vias 19 -> 21
- net MISO_JP4P1: track 108.0 -> 108.3 mm, vias 6 -> 7
- net N$65: track 122.4 -> 122.7 mm, vias 1 -> 2

Commit message: up
Parts:
- added F3: 1206L020, polyfuse-smd_10:1206L
- added TP6: PTR1B1,27, testpad:B1,27
Connections:
- new net N$52: F3.2, IC1.1
- new net N$70: TP6.TP, U4.4
- net N$69: now also F3.1; no longer IC1.1
Routing:
- net N$70: track 0.00 -> 34.4 mm
- net N$52: track 0.00 -> 13.6 mm
- net N$69: track 83.1 -> 69.5 mm
Changed lines of the file:
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@@
 <attribute name="MF" value="NXP USA" x="21.59" y="22.86" size="1.778" layer="27" display="off"/>
 <attribute name="MP" value="MCZ33996EK" x="21.59" y="22.86" size="1.778" layer="27" display="off"/>
+<attribute name="NAME" x="18.185309375" y="29.168690625" size="1.27175" layer="25"/>
 <attribute name="NAME" x="18.189590625" y="29.16075" size="1.27015" layer="25"/>
-<attribute name="NAME" x="18.185309375" y="29.168690625" size="1.27175" layer="25"/>
 <attribute name="PACKAGE" value="SOIC-32 NXP Semiconductors" x="21.59" y="22.86" size="1.778" layer="27" display="off"/>
 <attribute name="PRICE" value="None" x="21.59" y="22.86" size="1.778" layer="27" display="off"/>
@@
 <attribute name="POPULARITY" value="57" x="19.05" y="6.35" size="1.778" layer="27" display="off"/>
 <attribute name="VALUE" x="13.97" y="-1.27" size="1.27" layer="27" ratio="10"/>
+</element>
+<element name="F3" library="polyfuse-smd_10" package="1206L" value="1206L020" x="29.21" y="5.08" smashed="yes" rot="R180">
+<attribute name="MF" value="Littelfuse" x="29.21" y="5.08" size="1.778" layer="27" rot="R180" display="off"/>
+<attribute name="MPN" value="1206L020" x="29.21" y="5.08" size="1.778" layer="27" rot="R180" display="off"/>
+<attribute name="NAME" x="30.76" y="3.78" size="1.27" layer="25" rot="R180"/>
+<attribute name="OC_FARNELL" value="2072173" x="29.21" y="5.08" size="1.778" layer="27" rot="R180" display="off"/>
+<attribute name="OC_NEWARK" value="05M2300" x="29.21" y="5.08" size="1.778" layer="27" rot="R180" display="off"/>
+<attribute name="VALUE" x="30.76" y="7.68" size="1.27" layer="27" rot="R180"/>
+</element>
+<element name="TP6" library="testpad" library_urn="urn:adsk.eagle:library:385" package="B1,27" package3d_urn="urn:adsk.eagle:package:27944/2" value="PTR1B1,27" x="31.75" y="2.54" smashed="yes">
+<attribute name="NAME" x="31.115" y="3.556" size="1.27" layer="25" ratio="10"/>
+<attribute name="POPULARITY" value="2" x="31.75" y="2.54" size="1.778" layer="27" display="off"/>
+<attribute name="TP_SIGNAL_NAME" value="" x="31.75" y="2.54" size="1.778" layer="27" display="off"/>
+<attribute name="VALUE" x="31.115" y="1.778" size="0.0254" layer="27"/>
 </element>
 </elements>
@@
 <wire x1="92.0496" y1="7.1628" x2="91.821" y2="7.3914" width="0.1524" layer="1"/>
 <wire x1="92.0496" y1="5.4864" x2="92.0496" y2="7.1628" width="0.1524" layer="1"/>
-<wire x1="88.0872" y1="1.524" x2="92.0496" y2="5.4864" width="0.1524" layer="1"/>
+<wire x1="92.0496" y1="5.4864" x2="88.0872" y2="1.524" width="0.1524" layer="1"/>
 <via x="15.4686" y="19.2786" extent="1-16" drill="0.35"/>
 <wire x1="96.4692" y1="28.575" x2="96.4692" y2="29.1846" width="0.1524" layer="1"/>
@@
 <wire x1="90.2208" y1="18.7452" x2="92.583" y2="18.7452" width="0.1524" layer="1"/>
 <wire x1="96.4692" y1="29.1846" x2="96.52" y2="29.21" width="0.1524" layer="1"/>
-<wire x1="63.4746" y1="1.524" x2="88.0872" y2="1.524" width="0.1524" layer="1"/>
-<wire x1="63.0174" y1="1.9812" x2="63.4746" y2="1.524" width="0.1524" layer="1"/>
-<wire x1="62.5602" y1="1.9812" x2="63.0174" y2="1.9812" width="0.1524" layer="16"/>
-<wire x1="62.103" y1="1.524" x2="62.5602" y2="1.9812" width="0.1524" layer="16"/>
-<wire x1="46.7868" y1="1.524" x2="62.103" y2="1.524" width="0.1524" layer="16"/>
 <wire x1="44.5008" y1="3.81" x2="46.7868" y2="1.524" width="0.1524" layer="16"/>
 <wire x1="44.5008" y1="3.81" x2="44.45" y2="3.81" width="0.1524" layer="16"/>
-<via x="63.0174" y="1.9812" extent="1-16" drill="0.35"/>
+<wire x1="88.0872" y1="1.524" x2="74.676" y2="1.524" width="0.1524" layer="1"/>
+<wire x1="73.6092" y1="1.524" x2="46.7868" y2="1.524" width="0.1524" layer="16"/>
+<wire x1="74.0664" y1="1.9812" x2="73.6092" y2="1.524" width="0.1524" layer="16"/>
+<wire x1="74.2188" y1="1.9812" x2="74.0664" y2="1.9812" width="0.1524" layer="1"/>
+<wire x1="74.676" y1="1.524" x2="74.2188" y2="1.9812" width="0.1524" layer="1"/>
+<via x="74.0664" y="1.9812" extent="1-16" drill="0.35"/>
 </signal>
 <signal name="N$66">
@@
 <signal name="N$69">
 <contactref element="X8" pad="1"/>
-<contactref element="IC1" pad="1"/>
-<wire x1="16.8402" y1="3.81" x2="16.51" y2="3.81" width="0.1524" layer="1"/>
-<wire x1="18.5928" y1="2.0574" x2="16.8402" y2="3.81" width="0.1524" layer="1"/>
-<wire x1="42.3672" y1="2.0574" x2="18.5928" y2="2.0574" width="0.1524" layer="1"/>
 <wire x1="43.434" y1="3.1242" x2="42.3672" y2="2.0574" width="0.1524" layer="1"/>
 <wire x1="43.434" y1="5.0292" x2="43.434" y2="3.1242" width="0.1524" layer="1"/>
@@
 <via x="68.6562" y="15.3162" extent="1-16" drill="0.35"/>
 <via x="75.6666" y="15.3162" extent="1-16" drill="0.35"/>
+<contactref element="F3" pad="1"/>
+<wire x1="42.3672" y1="2.0574" x2="36.3474" y2="2.0574" width="0.1524" layer="1"/>
+<wire x1="33.3756" y1="5.0292" x2="30.6324" y2="5.0292" width="0.1524" layer="1"/>
+<wire x1="36.3474" y1="2.0574" x2="33.3756" y2="5.0292" width="0.1524" layer="1"/>
+<wire x1="30.6324" y1="5.0292" x2="30.61" y2="5.08" width="0.1524" layer="1"/>
+</signal>
+<signal name="N$52">
+<contactref element="IC1" pad="1"/>
+<contactref element="F3" pad="2"/>
+<wire x1="18.288" y1="2.0574" x2="25.2984" y2="2.0574" width="0.1524" layer="1"/>
+<wire x1="16.5354" y1="3.81" x2="18.288" y2="2.0574" width="0.1524" layer="1"/>
+<wire x1="16.5354" y1="3.81" x2="16.51" y2="3.81" width="0.1524" layer="1"/>
+<wire x1="27.7368" y1="4.4958" x2="27.7368" y2="5.0292" width="0.1524" layer="1"/>
+<wire x1="25.2984" y1="2.0574" x2="27.7368" y2="4.4958" width="0.1524" layer="1"/>
+<wire x1="27.7368" y1="5.0292" x2="27.81" y2="5.08" width="0.1524" layer="1"/>
+</signal>
+<signal name="N$70">
+<contactref element="U4" pad="4"/>
+<contactref element="TP6" pad="TP"/>
+<wire x1="31.75" y1="2.54" x2="33.02" y2="1.27" width="0.1524" layer="1"/>
+<wire x1="33.02" y1="1.27" x2="62.23" y2="1.27" width="0.1524" layer="1"/>
+<wire x1="64.02" y1="3.06" x2="64.88" y2="3.06" width="0.1524" layer="1"/>
+<wire x1="62.23" y1="1.27" x2="64.02" y2="3.06" width="0.1524" layer="1"/>
 </signal>
 </signals>

Commit message: up
Parts:
- removed TP6: PTR1B1,27, testpad:B1,27
- added PAD1, PAD2: WIREPAD1,6/0,8, wirepad:1,6/0,8
Connections:
- new net N$71: PAD1.1, U4.9
- net N$70: now also PAD2.1; no longer TP6.TP
Routing:
- net N$71: track 0.00 -> 11.5 mm, vias 0 -> 3
Changed lines of the file:
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@@
 <attribute name="MF" value="NXP USA" x="21.59" y="22.86" size="1.778" layer="27" display="off"/>
 <attribute name="MP" value="MCZ33996EK" x="21.59" y="22.86" size="1.778" layer="27" display="off"/>
+<attribute name="NAME" x="18.189590625" y="29.16075" size="1.27015" layer="25"/>
 <attribute name="NAME" x="18.185309375" y="29.168690625" size="1.27175" layer="25"/>
-<attribute name="NAME" x="18.189590625" y="29.16075" size="1.27015" layer="25"/>
 <attribute name="PACKAGE" value="SOIC-32 NXP Semiconductors" x="21.59" y="22.86" size="1.778" layer="27" display="off"/>
 <attribute name="PRICE" value="None" x="21.59" y="22.86" size="1.778" layer="27" display="off"/>
@@
 <attribute name="VALUE" x="30.76" y="7.68" size="1.27" layer="27" rot="R180"/>
 </element>
-<element name="TP6" library="testpad" library_urn="urn:adsk.eagle:library:385" package="B1,27" package3d_urn="urn:adsk.eagle:package:27944/2" value="PTR1B1,27" x="31.75" y="2.54" smashed="yes">
-<attribute name="NAME" x="31.115" y="3.556" size="1.27" layer="25" ratio="10"/>
-<attribute name="POPULARITY" value="2" x="31.75" y="2.54" size="1.778" layer="27" display="off"/>
-<attribute name="TP_SIGNAL_NAME" value="" x="31.75" y="2.54" size="1.778" layer="27" display="off"/>
-<attribute name="VALUE" x="31.115" y="1.778" size="0.0254" layer="27"/>
+<element name="PAD1" library="wirepad" library_urn="urn:adsk.eagle:library:412" package="1,6/0,8" package3d_urn="urn:adsk.eagle:package:30830/1" value="WIREPAD1,6/0,8" x="74.93" y="6.35" smashed="yes">
+<attribute name="NAME" x="74.168" y="7.366" size="1.27" layer="25" ratio="10"/>
+<attribute name="POPULARITY" value="1" x="74.93" y="6.35" size="1.778" layer="27" display="off"/>
+<attribute name="VALUE" x="74.93" y="6.95" size="0.0254" layer="27"/>
+</element>
+<element name="PAD2" library="wirepad" library_urn="urn:adsk.eagle:library:412" package="1,6/0,8" package3d_urn="urn:adsk.eagle:package:30830/1" value="WIREPAD1,6/0,8" x="31.75" y="2.54" smashed="yes">
+<attribute name="NAME" x="30.988" y="3.556" size="1.27" layer="25" ratio="10"/>
+<attribute name="POPULARITY" value="1" x="31.75" y="2.54" size="1.778" layer="27" display="off"/>
+<attribute name="VALUE" x="31.75" y="3.14" size="0.0254" layer="27"/>
 </element>
 </elements>
@@
 <wire x1="27.7368" y1="5.0292" x2="27.81" y2="5.08" width="0.1524" layer="1"/>
 </signal>
+<signal name="N$71">
+<contactref element="U4" pad="9"/>
+<contactref element="PAD1" pad="1"/>
+<wire x1="67.5894" y1="3.5814" x2="67.2084" y2="3.5814" width="0.1524" layer="1"/>
+<wire x1="67.9704" y1="3.9624" x2="67.5894" y2="3.5814" width="0.1524" layer="1"/>
+<wire x1="68.5038" y1="3.9624" x2="67.9704" y2="3.9624" width="0.1524" layer="1"/>
+<wire x1="70.7136" y1="3.9624" x2="68.5038" y2="3.9624" width="0.1524" layer="16"/>
+<wire x1="71.1708" y1="4.4196" x2="70.7136" y2="3.9624" width="0.1524" layer="16"/>
+<wire x1="71.1708" y1="5.1816" x2="71.1708" y2="4.4196" width="0.1524" layer="1"/>
+<wire x1="70.4088" y1="5.9436" x2="71.1708" y2="5.1816" width="0.1524" layer="1"/>
+<wire x1="70.104" y1="5.9436" x2="70.4088" y2="5.9436" width="0.1524" layer="1"/>
+<wire x1="74.5236" y1="5.9436" x2="70.104" y2="5.9436" width="0.1524" layer="16"/>
+<wire x1="74.93" y1="6.35" x2="74.5236" y2="5.9436" width="0.1524" layer="16"/>
+<wire x1="67.2084" y1="3.5814" x2="67.2" y2="3.56" width="0.1524" layer="1"/>
+<via x="68.5038" y="3.9624" extent="1-16" drill="0.35"/>
+<via x="71.1708" y="4.4196" extent="1-16" drill="0.35"/>
+<via x="70.104" y="5.9436" extent="1-16" drill="0.35"/>
+</signal>
 <signal name="N$70">
 <contactref element="U4" pad="4"/>
-<contactref element="TP6" pad="TP"/>
-<wire x1="31.75" y1="2.54" x2="33.02" y2="1.27" width="0.1524" layer="1"/>
-<wire x1="33.02" y1="1.27" x2="62.23" y2="1.27" width="0.1524" layer="1"/>
-<wire x1="64.02" y1="3.06" x2="64.88" y2="3.06" width="0.1524" layer="1"/>
-<wire x1="62.23" y1="1.27" x2="64.02" y2="3.06" width="0.1524" layer="1"/>
+<contactref element="PAD2" pad="1"/>
+<wire x1="63.627" y1="3.048" x2="64.8462" y2="3.048" width="0.1524" layer="1"/>
+<wire x1="61.9506" y1="1.3716" x2="63.627" y2="3.048" width="0.1524" layer="1"/>
+<wire x1="32.9184" y1="1.3716" x2="61.9506" y2="1.3716" width="0.1524" layer="1"/>
+<wire x1="31.75" y1="2.54" x2="32.9184" y2="1.3716" width="0.1524" layer="1"/>
+<wire x1="64.8462" y1="3.048" x2="64.88" y2="3.06" width="0.1524" layer="1"/>
 </signal>
 </signals>
