File: tic12400.sch (EAGLE design)
At the start: 12 parts, among them X1 22-23-2031

Commit message: up
Parts:
- added C6: 10uf, rcl:C-USC0805
- added C7: 0.1, rcl:C-USC0805
Connections:
- net GND: now also C6.2, C7.2
- net VDD: now also C6.1, C7.1
Changed lines of the file:
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@@
 <part name="P+4" library="supply1" library_urn="urn:adsk.eagle:library:371" deviceset="+24V" device=""/>
 <part name="GND9" library="supply1" library_urn="urn:adsk.eagle:library:371" deviceset="GND" device=""/>
+<part name="C7" library="rcl" library_urn="urn:adsk.eagle:library:334" deviceset="C-US" device="C0805" package3d_urn="urn:adsk.eagle:package:23617/2" value="0.1"/>
+<part name="C6" library="rcl" library_urn="urn:adsk.eagle:library:334" deviceset="C-US" device="C0805" package3d_urn="urn:adsk.eagle:package:23617/2" value="10uf"/>
+<part name="GND10" library="supply1" library_urn="urn:adsk.eagle:library:371" deviceset="GND" device=""/>
+<part name="GND11" library="supply1" library_urn="urn:adsk.eagle:library:371" deviceset="GND" device=""/>
+<part name="VDD4" library="supply1" library_urn="urn:adsk.eagle:library:371" deviceset="VDD" device=""/>
+<part name="VDD5" library="supply1" library_urn="urn:adsk.eagle:library:371" deviceset="VDD" device=""/>
 </parts>
 <sheets>
@@
 <attribute name="VALUE" x="58.42" y="160.02" size="1.778" layer="96" rot="R270"/>
 </instance>
+<instance part="C7" gate="G$1" x="-2.54" y="55.88" smashed="yes">
+<attribute name="NAME" x="-1.524" y="56.515" size="1.778" layer="95"/>
+<attribute name="VALUE" x="-1.524" y="51.689" size="1.778" layer="96"/>
+</instance>
+<instance part="C6" gate="G$1" x="10.16" y="55.88" smashed="yes">
+<attribute name="NAME" x="11.176" y="56.515" size="1.778" layer="95"/>
+<attribute name="VALUE" x="11.176" y="51.689" size="1.778" layer="96"/>
+</instance>
+<instance part="GND10" gate="1" x="-2.54" y="48.26" smashed="yes">
+<attribute name="VALUE" x="-5.08" y="45.72" size="1.778" layer="96"/>
+</instance>
+<instance part="GND11" gate="1" x="10.16" y="48.26" smashed="yes">
+<attribute name="VALUE" x="7.62" y="45.72" size="1.778" layer="96"/>
+</instance>
+<instance part="VDD4" gate="G$1" x="-2.54" y="60.96" smashed="yes">
+<attribute name="VALUE" x="-5.08" y="58.42" size="1.778" layer="96" rot="R90"/>
+</instance>
+<instance part="VDD5" gate="G$1" x="10.16" y="60.96" smashed="yes">
+<attribute name="VALUE" x="7.62" y="58.42" size="1.778" layer="96" rot="R90"/>
+</instance>
 </instances>
 <busses>
@@
 <pinref part="VDD3" gate="G$1" pin="VDD"/>
 </segment>
+<segment>
+<pinref part="C7" gate="G$1" pin="1"/>
+<pinref part="VDD4" gate="G$1" pin="VDD"/>
+</segment>
+<segment>
+<pinref part="C6" gate="G$1" pin="1"/>
+<pinref part="VDD5" gate="G$1" pin="VDD"/>
+</segment>
 </net>
 <net name="GND" class="1">
@@
 <pinref part="GND9" gate="1" pin="GND"/>
 </segment>
+<segment>
+<pinref part="C7" gate="G$1" pin="2"/>
+<pinref part="GND10" gate="1" pin="GND"/>
+</segment>
+<segment>
+<pinref part="C6" gate="G$1" pin="2"/>
+<pinref part="GND11" gate="1" pin="GND"/>
+</segment>
 </net>

Commit message: up
Parts:
- added SV2: DEBUG_H, con-lsta:FE10-1
- added X2, X3, X4: (no value), con-molex:KK-156-10
Connections:
- removed net VDD: C6.1, C7.1, IC1.19, R3.2, R4.1, SV1.7
- new net CS_JP3P11: IC1.15, R3.1, SV1.5, SV2.5
- new net EXT2_JP3P8: IC1.26, R4.2, SV1.9, SV2.9
- new net GND_JP4P8: C1.2, C2.2, C3.2, C4.2, C5.2, C6.2, C7.2, IC1.30, R1.1, X1-1.S
- new net MISO_JP4P1: IC1.18, SV1.1, SV2.1
- new net MOSI_JP4P2: IC1.16, SV1.3, SV2.3
- new net N$1: IC1.13, X2-1.S
- new net N$11: IC1.6, X4-3.S
- new net N$12: IC1.5, X4-2.S
- new net N$13: IC1.4, X4-1.S
- new net N$14: IC1.3, X3-8.S
- new net N$15: IC1.2, X3-7.S
- new net N$16: IC1.1, X3-6.S
- new net N$17: IC1.27, X2-3.S
- new net N$18: IC1.28, X2-4.S
- new net N$19: IC1.29, X2-5.S
- new net N$20: IC1.31, X2-6.S
- new net N$21: IC1.32, X2-7.S
- new net N$22: IC1.33, X2-8.S
- new net N$23: IC1.34, X3-1.S
- new net N$24: IC1.35, X3-2.S
- new net N$25: IC1.36, X3-3.S
- new net N$26: IC1.37, X3-4.S
- new net N$27: IC1.38, X3-5.S
- new net N$28: IC1.12, X4-8.S
- new net SCK_JP4P3: IC1.17, SV1.2, SV2.2
- new net VDD_JP4P5: C6.1, C7.1, IC1.19, R3.2, R4.1, SV1.7, SV2.7
- net +24V: now also X2-9.S, X3-9.S, X4-9.S
- net GND: now also SV2.8, X2-10.S, X3-10.S, X4-10.S; no longer C1.2, C2.2, C3.2, C4.2, C5.2, C6.2, C7.2, IC1.30, R1.1, X1-1.S
- net N$2: now also IC1.14, X2-2.S; no longer IC1.18, SV1.1
- net N$3: now also IC1.10, X4-6.S; no longer IC1.16, SV1.3
- net N$4: now also IC1.11, X4-7.S; no longer IC1.17, SV1.2
- net N$5: now also IC1.8, X4-5.S; no longer IC1.15, R3.1, SV1.5
- net N$6: now also SV2.6
- net N$7: now also IC1.7, X4-4.S; no longer IC1.26, R4.2, SV1.9
Other:
- moved on the sheet: IC2, R3, SV1

Commit message: up
Parts:
- added C10, C8, C9: 0.1, rcl:C-USC0805
Connections:
- removed net GND_JP4P8: C1.2, C2.2, C3.2, C4.2, C5.2, C6.2, C7.2, IC1.30, R1.1, X1-1.S
- net +24V: now also C10.1, C8.1, C9.1, IC2.C2B, IC2.GH2B
- net GND: now also C1.2, C10.2, C2.2, C3.2, C4.2, C5.2, C6.2, C7.2, C8.2, C9.2, IC1.30, R1.1, X1-1.S
- net N$15: now also IC2.GH2A
- net N$16: now also IC2.C2A
- net N$8: now also IC2.GND
- net VDD_JP4P5: now also IC2.ENABLE
Other:
- moved on the sheet: IC2
Changed lines of the file:
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@@
 <part name="P+6" library="supply1" library_urn="urn:adsk.eagle:library:371" deviceset="+24V" device=""/>
 <part name="P+7" library="supply1" library_urn="urn:adsk.eagle:library:371" deviceset="+24V" device=""/>
+<part name="C8" library="rcl" library_urn="urn:adsk.eagle:library:334" deviceset="C-US" device="C0805" package3d_urn="urn:adsk.eagle:package:23617/2" value="0.1"/>
+<part name="C9" library="rcl" library_urn="urn:adsk.eagle:library:334" deviceset="C-US" device="C0805" package3d_urn="urn:adsk.eagle:package:23617/2" value="0.1"/>
+<part name="C10" library="rcl" library_urn="urn:adsk.eagle:library:334" deviceset="C-US" device="C0805" package3d_urn="urn:adsk.eagle:package:23617/2" value="0.1"/>
+<part name="GND15" library="supply1" library_urn="urn:adsk.eagle:library:371" deviceset="GND" device=""/>
+<part name="GND16" library="supply1" library_urn="urn:adsk.eagle:library:371" deviceset="GND" device=""/>
+<part name="GND17" library="supply1" library_urn="urn:adsk.eagle:library:371" deviceset="GND" device=""/>
 </parts>
 <sheets>
@@
 <attribute name="VALUE" x="56.515" y="82.55" size="1.778" layer="96"/>
 </instance>
-<instance part="IC2" gate="G$1" x="223.52" y="111.76" smashed="yes">
-<attribute name="NAME" x="218.44" y="134.62" size="1.778" layer="95"/>
-<attribute name="VALUE" x="210.82" y="83.82" size="1.778" layer="96"/>
+<instance part="IC2" gate="G$1" x="195.58" y="127" smashed="yes">
+<attribute name="NAME" x="190.5" y="149.86" size="1.778" layer="95"/>
+<attribute name="VALUE" x="182.88" y="99.06" size="1.778" layer="96"/>
 </instance>
 <instance part="SV1" gate="1" x="60.96" y="12.7" smashed="yes" rot="R90">
@@
 <instance part="P+7" gate="1" x="109.22" y="88.9" smashed="yes" rot="R180">
 <attribute name="VALUE" x="111.76" y="93.98" size="1.778" layer="96" rot="R270"/>
+</instance>
+<instance part="C8" gate="G$1" x="104.14" y="157.48" smashed="yes">
+<attribute name="NAME" x="105.156" y="158.115" size="1.778" layer="95"/>
+<attribute name="VALUE" x="105.156" y="153.289" size="1.778" layer="96"/>
+</instance>
+<instance part="C9" gate="G$1" x="106.68" y="124.46" smashed="yes">
+<attribute name="NAME" x="107.696" y="125.095" size="1.778" layer="95"/>
+<attribute name="VALUE" x="107.696" y="120.269" size="1.778" layer="96"/>
+</instance>
+<instance part="C10" gate="G$1" x="111.76" y="88.9" smashed="yes">
+<attribute name="NAME" x="112.776" y="89.535" size="1.778" layer="95"/>
+<attribute name="VALUE" x="112.776" y="84.709" size="1.778" layer="96"/>
+</instance>
+<instance part="GND15" gate="1" x="111.76" y="81.28" smashed="yes">
+<attribute name="VALUE" x="109.22" y="78.74" size="1.778" layer="96"/>
+</instance>
+<instance part="GND16" gate="1" x="106.68" y="116.84" smashed="yes">
+<attribute name="VALUE" x="104.14" y="114.3" size="1.778" layer="96"/>
+</instance>
+<instance part="GND17" gate="1" x="104.14" y="149.86" smashed="yes">
+<attribute name="VALUE" x="101.6" y="147.32" size="1.778" layer="96"/>
 </instance>
 </instances>
@@
 <pinref part="VDD5" gate="G$1" pin="VDD"/>
 </segment>
-</net>
-<net name="GND_JP4P8" class="1">
-<segment>
-<pinref part="IC1" gate="G$1" pin="30"/>
-<wire x1="68.58" y1="109.22" x2="96.52" y2="109.22" width="0.1524" layer="91"/>
-<pinref part="GND1" gate="1" pin="GND"/>
-<wire x1="96.52" y1="109.22" x2="96.52" y2="106.68" width="0.1524" layer="91"/>
-</segment>
-<segment>
-<pinref part="C1" gate="G$1" pin="2"/>
-<pinref part="GND3" gate="1" pin="GND"/>
-</segment>
-<segment>
-<pinref part="C2" gate="G$1" pin="2"/>
-<pinref part="GND4" gate="1" pin="GND"/>
-</segment>
-<segment>
-<pinref part="C3" gate="G$1" pin="2"/>
-<pinref part="GND5" gate="1" pin="GND"/>
-</segment>
-<segment>
-<pinref part="C4" gate="G$1" pin="2"/>
-<pinref part="GND6" gate="1" pin="GND"/>
-</segment>
-<segment>
-<pinref part="C5" gate="G$1" pin="2"/>
-<pinref part="GND7" gate="1" pin="GND"/>
-</segment>
-<segment>
-<pinref part="R1" gate="G$1" pin="1"/>
-<pinref part="GND8" gate="1" pin="GND"/>
-</segment>
-<segment>
-<pinref part="X1" gate="-1" pin="S"/>
-<pinref part="GND9" gate="1" pin="GND"/>
-</segment>
-<segment>
-<pinref part="C7" gate="G$1" pin="2"/>
-<pinref part="GND10" gate="1" pin="GND"/>
-</segment>
-<segment>
-<pinref part="C6" gate="G$1" pin="2"/>
-<pinref part="GND11" gate="1" pin="GND"/>
+<segment>
+<wire x1="175.26" y1="124.46" x2="154.94" y2="124.46" width="0.1524" layer="91"/>
+<pinref part="IC2" gate="G$1" pin="ENABLE"/>
 </segment>
 </net>
@@
 <pinref part="X2" gate="-9" pin="S"/>
 <pinref part="P+5" gate="1" pin="+24V"/>
-<wire x1="96.52" y1="160.02" x2="116.84" y2="160.02" width="0.1524" layer="91"/>
+<wire x1="96.52" y1="160.02" x2="104.14" y2="160.02" width="0.1524" layer="91"/>
 <junction x="116.84" y="160.02"/>
+<pinref part="C8" gate="G$1" pin="1"/>
+<wire x1="104.14" y1="160.02" x2="116.84" y2="160.02" width="0.1524" layer="91"/>
+<junction x="104.14" y="160.02"/>
 </segment>
 <segment>
 <pinref part="X3" gate="-9" pin="S"/>
 <pinref part="P+6" gate="1" pin="+24V"/>
-<wire x1="99.06" y1="127" x2="116.84" y2="127" width="0.1524" layer="91"/>
+<wire x1="99.06" y1="127" x2="106.68" y2="127" width="0.1524" layer="91"/>
 <junction x="116.84" y="127"/>
+<pinref part="C9" gate="G$1" pin="1"/>
+<wire x1="106.68" y1="127" x2="116.84" y2="127" width="0.1524" layer="91"/>
+<junction x="106.68" y="127"/>
 </segment>
 <segment>
 <pinref part="X4" gate="-9" pin="S"/>
 <pinref part="P+7" gate="1" pin="+24V"/>
-<wire x1="109.22" y1="91.44" x2="116.84" y2="91.44" width="0.1524" layer="91"/>
+<wire x1="109.22" y1="91.44" x2="111.76" y2="91.44" width="0.1524" layer="91"/>
 <junction x="116.84" y="91.44"/>
+<pinref part="C10" gate="G$1" pin="1"/>
+<wire x1="111.76" y1="91.44" x2="116.84" y2="91.44" width="0.1524" layer="91"/>
+<junction x="111.76" y="91.44"/>
+</segment>
+<segment>
+<wire x1="215.9" y1="93.98" x2="223.52" y2="93.98" width="0.1524" layer="91"/>
+<pinref part="IC2" gate="G$1" pin="GH2B"/>
+</segment>
+<segment>
+<wire x1="215.9" y1="88.9" x2="223.52" y2="88.9" width="0.1524" layer="91"/>
+<pinref part="IC2" gate="G$1" pin="C2B"/>
 </segment>
 </net>
@@
 <pinref part="C1" gate="G$1" pin="1"/>
 <wire x1="68.58" y1="88.9" x2="88.9" y2="88.9" width="0.1524" layer="91"/>
+</segment>
+<segment>
+<wire x1="195.58" y1="63.5" x2="195.58" y2="83.82" width="0.1524" layer="91"/>
+<pinref part="IC2" gate="G$1" pin="GND"/>
 </segment>
 </net>
@@
 <junction x="53.34" y="43.18"/>
 </segment>
+<segment>
+<pinref part="IC1" gate="G$1" pin="30"/>
+<wire x1="68.58" y1="109.22" x2="96.52" y2="109.22" width="0.1524" layer="91"/>
+<pinref part="GND1" gate="1" pin="GND"/>
+<wire x1="96.52" y1="109.22" x2="96.52" y2="106.68" width="0.1524" layer="91"/>
+<label x="96.52" y="111.76" size="1.778" layer="95"/>
+</segment>
+<segment>
+<pinref part="C1" gate="G$1" pin="2"/>
+<pinref part="GND3" gate="1" pin="GND"/>
+</segment>
+<segment>
+<pinref part="C2" gate="G$1" pin="2"/>
+<pinref part="GND4" gate="1" pin="GND"/>
+</segment>
+<segment>
+<pinref part="C3" gate="G$1" pin="2"/>
+<pinref part="GND5" gate="1" pin="GND"/>
+</segment>
+<segment>
+<pinref part="C4" gate="G$1" pin="2"/>
+<pinref part="GND6" gate="1" pin="GND"/>
+</segment>
+<segment>
+<pinref part="C5" gate="G$1" pin="2"/>
+<pinref part="GND7" gate="1" pin="GND"/>
+</segment>
+<segment>
+<pinref part="R1" gate="G$1" pin="1"/>
+<pinref part="GND8" gate="1" pin="GND"/>
+</segment>
+<segment>
+<pinref part="X1" gate="-1" pin="S"/>
+<pinref part="GND9" gate="1" pin="GND"/>
+</segment>
+<segment>
+<pinref part="C7" gate="G$1" pin="2"/>
+<pinref part="GND10" gate="1" pin="GND"/>
+</segment>
+<segment>
+<pinref part="C6" gate="G$1" pin="2"/>
+<pinref part="GND11" gate="1" pin="GND"/>
+</segment>
+<segment>
+<pinref part="C10" gate="G$1" pin="2"/>
+<pinref part="GND15" gate="1" pin="GND"/>
+</segment>
+<segment>
+<pinref part="C9" gate="G$1" pin="2"/>
+<pinref part="GND16" gate="1" pin="GND"/>
+</segment>
+<segment>
+<pinref part="C8" gate="G$1" pin="2"/>
+<pinref part="GND17" gate="1" pin="GND"/>
+</segment>
 </net>
 <net name="N$2" class="0">
@@
 <junction x="116.84" y="132.08"/>
 </segment>
+<segment>
+<wire x1="243.84" y1="119.38" x2="215.9" y2="119.38" width="0.1524" layer="91"/>
+<pinref part="IC2" gate="G$1" pin="GH2A"/>
+</segment>
 </net>
 <net name="N$16" class="0">
@@
 <junction x="116.84" y="134.62"/>
 </segment>
-</net>
+<segment>
+<wire x1="246.38" y1="124.46" x2="215.9" y2="124.46" width="0.1524" layer="91"/>
+<pinref part="IC2" gate="G$1" pin="C2A"/>
+</segment>
+</net>

Commit message: up
Parts:
- removed IC2: (no value), allegro2:A3986
- added U1: TIC12400DCPR, TIC12400DCPR:TIC12400DCPR
Connections:
- net +24V: no longer IC2.C2B, IC2.GH2B
- net CS_JP3P11: now also U1.!CS
- net EXT2_JP3P8: now also U1.!INT
- net GND: now also U1.AGND, U1.DGND, U1.EP
- net MISO_JP4P1: now also U1.SO
- net MOSI_JP4P2: now also U1.SCLK
- net N$1: now also U1.IN0
- net N$10: now also U1.CAP_D
- net N$11: now also U1.IN18
- net N$12: now also U1.IN17
- net N$13: now also U1.IN16
- net N$14: now also U1.IN15
- net N$15: now also U1.IN14; no longer IC2.GH2A
- net N$16: now also U1.IN13; no longer IC2.C2A
- net N$17: now also U1.IN2
- net N$18: now also U1.IN3
- net N$19: now also U1.IN4
- net N$2: now also U1.IN1
- net N$20: now also U1.IN5
- net N$21: now also U1.IN6
- net N$22: now also U1.IN7
- net N$23: now also U1.IN8
- net N$24: now also U1.IN9
- net N$25: now also U1.IN10
- net N$26: now also U1.IN11
- net N$27: now also U1.IN12, U1.VS
- net N$28: now also U1.IN23
- net N$3: now also U1.IN21
- net N$4: now also U1.IN22
- net N$5: now also U1.IN20
- net N$6: now also U1.RESET
- net N$7: now also U1.IN19
- net N$8: now also U1.CAP_A; no longer IC2.GND
- net N$9: now also U1.CAP_PRE
- net SCK_JP4P3: now also U1.SI
- net VDD_JP4P5: now also U1.VDD; no longer IC2.ENABLE

Commit message: up
Parts:
- removed IC1: (no value), ic-package:DIL40
- added D1: ES2D, diode:ES2D
- X2: value (none) -> INPUT1
- X3: value (none) -> INPUT2
- X4: value (none) -> INPUT3
Connections:
- removed net MOSI_JP4P2: IC1.16, SV1.3, SV2.3, U1.SCLK
- removed net SCK_JP4P3: IC1.17, SV1.2, SV2.2, U1.SI
- new net MOSI_JP4P3: SV1.2, SV2.2, U1.SI
- new net N$29: D1.A, X1-2.S, X1-3.S
- new net SCK_JP4P2: SV1.3, SV2.3, U1.SCLK
- net +24V: now also D1.C, U1.VS; no longer IC1.39, IC1.40, X1-2.S, X1-3.S
- net CS_JP3P11: no longer IC1.15
- net EXT2_JP3P8: no longer IC1.26
- net GND: no longer IC1.30, IC1.9
- net MISO_JP4P1: no longer IC1.18
- net N$1: no longer IC1.13
- net N$10: no longer IC1.25
- net N$11: no longer IC1.6
- net N$12: no longer IC1.5
- net N$13: no longer IC1.4
- net N$14: no longer IC1.3
- net N$15: no longer IC1.2
- net N$16: no longer IC1.1
- net N$17: no longer IC1.27
- net N$18: no longer IC1.28
- net N$19: no longer IC1.29
- net N$2: no longer IC1.14
- net N$20: no longer IC1.31
- net N$21: no longer IC1.32
- net N$22: no longer IC1.33
- net N$23: no longer IC1.34
- net N$24: no longer IC1.35
- net N$25: no longer IC1.36
- net N$26: no longer IC1.37
- net N$27: no longer IC1.38, U1.VS
- net N$28: no longer IC1.12
- net N$3: no longer IC1.10
- net N$4: no longer IC1.11
- net N$5: no longer IC1.8
- net N$6: no longer IC1.23
- net N$7: no longer IC1.7
- net N$8: no longer IC1.22
- net N$9: no longer IC1.24
- net VDD_JP4P5: no longer IC1.19

Commit message: up
Parts:
- added U2: MCZ33996EK, MCZ33996EK:MCZ33996EK
Connections:
- net +24V: now also U2.VPWR
- net GND: now also U2.EP, U2.GND@1, U2.GND@2, U2.GND@3, U2.GND@4, U2.GND@5, U2.GND@6, U2.GND@7, U2.GND@8
- net MISO_JP4P1: now also U2.SO
- net MOSI_JP4P3: now also U2.SI
- net N$6: now also U2.!RST
- net SCK_JP4P2: now also U2.SCLK
- net VDD_JP4P5: now also U2.SOPWR
Changed lines of the file:
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@@
 <part name="P+8" library="supply1" library_urn="urn:adsk.eagle:library:371" deviceset="+24V" device=""/>
 <part name="D1" library="diode" library_urn="urn:adsk.eagle:library:210" deviceset="ES2D" device="" package3d_urn="urn:adsk.eagle:package:43404/2"/>
+<part name="U2" library="MCZ33996EK" deviceset="MCZ33996EK" device=""/>
+<part name="P+1" library="supply1" library_urn="urn:adsk.eagle:library:371" deviceset="+24V" device=""/>
+<part name="GND19" library="supply1" library_urn="urn:adsk.eagle:library:371" deviceset="GND" device=""/>
 </parts>
 <sheets>
@@
 <attribute name="VALUE" x="63.7286" y="149.86" size="1.778" layer="96" rot="R270"/>
 </instance>
+<instance part="U2" gate="G$1" x="205.74" y="149.86" smashed="yes">
+<attribute name="NAME" x="193.0382" y="176.5337" size="1.77825" layer="95"/>
+<attribute name="VALUE" x="193.0329" y="121.2691" size="1.778990625" layer="96"/>
+</instance>
+<instance part="P+1" gate="1" x="185.42" y="170.18" smashed="yes" rot="R90">
+<attribute name="VALUE" x="190.5" y="167.64" size="1.778" layer="96" rot="R180"/>
+</instance>
+<instance part="GND19" gate="1" x="187.96" y="124.46" smashed="yes">
+<attribute name="VALUE" x="185.42" y="121.92" size="1.778" layer="96"/>
+</instance>
 </instances>
 <busses>
@@
 <pinref part="U1" gate="G$1" pin="VDD"/>
 </segment>
+<segment>
+<wire x1="167.64" y1="172.72" x2="187.96" y2="172.72" width="0.1524" layer="91"/>
+<pinref part="U2" gate="G$1" pin="SOPWR"/>
+</segment>
 </net>
 <net name="CS_JP3P11" class="0">
@@
 <pinref part="U1" gate="G$1" pin="RESET"/>
 </segment>
+<segment>
+<wire x1="187.96" y1="162.56" x2="172.72" y2="162.56" width="0.1524" layer="91"/>
+<pinref part="U2" gate="G$1" pin="!RST"/>
+</segment>
 </net>
 <net name="EXT2_JP3P8" class="0">
@@
 <pinref part="P+8" gate="1" pin="+24V"/>
 </segment>
+<segment>
+<pinref part="U2" gate="G$1" pin="VPWR"/>
+<pinref part="P+1" gate="1" pin="+24V"/>
+</segment>
 </net>
 <net name="N$8" class="0">
@@
 <wire x1="203.2" y1="35.56" x2="198.12" y2="33.02" width="0.1524" layer="91"/>
 </segment>
+<segment>
+<pinref part="U2" gate="G$1" pin="GND@1"/>
+<pinref part="U2" gate="G$1" pin="GND@2"/>
+<wire x1="187.96" y1="147.32" x2="187.96" y2="144.78" width="0.1524" layer="91"/>
+<pinref part="U2" gate="G$1" pin="GND@3"/>
+<wire x1="187.96" y1="142.24" x2="187.96" y2="144.78" width="0.1524" layer="91"/>
+<junction x="187.96" y="144.78"/>
+<pinref part="U2" gate="G$1" pin="GND@4"/>
+<wire x1="187.96" y1="139.7" x2="187.96" y2="142.24" width="0.1524" layer="91"/>
+<junction x="187.96" y="142.24"/>
+<pinref part="U2" gate="G$1" pin="GND@5"/>
+<wire x1="187.96" y1="137.16" x2="187.96" y2="139.7" width="0.1524" layer="91"/>
+<junction x="187.96" y="139.7"/>
+<pinref part="U2" gate="G$1" pin="GND@6"/>
+<wire x1="187.96" y1="134.62" x2="187.96" y2="137.16" width="0.1524" layer="91"/>
+<junction x="187.96" y="137.16"/>
+<pinref part="U2" gate="G$1" pin="GND@7"/>
+<wire x1="187.96" y1="132.08" x2="187.96" y2="134.62" width="0.1524" layer="91"/>
+<junction x="187.96" y="134.62"/>
+<pinref part="U2" gate="G$1" pin="GND@8"/>
+<wire x1="187.96" y1="129.54" x2="187.96" y2="132.08" width="0.1524" layer="91"/>
+<junction x="187.96" y="132.08"/>
+<pinref part="U2" gate="G$1" pin="EP"/>
+<wire x1="187.96" y1="127" x2="187.96" y2="129.54" width="0.1524" layer="91"/>
+<junction x="187.96" y="129.54"/>
+<pinref part="GND19" gate="1" pin="GND"/>
+<junction x="187.96" y="127"/>
+<junction x="187.96" y="147.32"/>
+</segment>
 </net>
 <net name="N$2" class="0">
@@
 <pinref part="U1" gate="G$1" pin="SI"/>
 </segment>
+<segment>
+<wire x1="187.96" y1="154.94" x2="182.88" y2="154.94" width="0.1524" layer="91"/>
+<pinref part="U2" gate="G$1" pin="SI"/>
+</segment>
 </net>
 <net name="SCK_JP4P2" class="0">
@@
 <pinref part="U1" gate="G$1" pin="SCLK"/>
 </segment>
+<segment>
+<wire x1="187.96" y1="157.48" x2="182.88" y2="157.48" width="0.1524" layer="91"/>
+<pinref part="U2" gate="G$1" pin="SCLK"/>
+</segment>
 </net>
 <net name="MISO_JP4P1" class="0">
@@
 <pinref part="U1" gate="G$1" pin="SO"/>
 </segment>
-</net>
+<segment>
+<wire x1="187.96" y1="152.4" x2="182.88" y2="152.4" width="0.1524" layer="91"/>
+<pinref part="U2" gate="G$1" pin="SO"/>
+</segment>
+</net>

Commit message: up
Parts:
- added C11, C13, C14: 0.1, rcl:C-USC0805
- added C12: 10uf, rcl:C-USC0805
- added D2: ES2D, diode:ES2D
- added X5: 22-23-2031, con-molex:22-23-2031
- added X6: OUTPUT1, con-molex:KK-156-10
- added X7: OUTPUT2, con-molex:KK-156-10
Connections:
- new net N$30: D2.A, X5-2.S, X5-3.S
- new net N$32: C11.1, C12.1, C13.1, D2.C, U2.VPWR, X6-9.S, X7-9.S
- new net N$33: SV1.4, SV2.4, U2.!CS
- new net N$34: SV1.10, SV2.10, U2.PWM
- new net N$35: U2.OUT0, X6-1.S
- new net N$36: U2.OUT1, X6-2.S
- new net N$37: U2.OUT2, X6-3.S
- new net N$38: U2.OUT3, X6-4.S
- new net N$39: U2.OUT4, X6-5.S
- new net N$40: U2.OUT5, X6-6.S
- new net N$41: U2.OUT6, X6-7.S
- new net N$42: U2.OUT7, X6-8.S
- new net N$43: U2.OUT8, X7-1.S
- new net N$44: U2.OUT9, X7-2.S
- new net N$45: U2.OUT10, X7-3.S
- new net N$46: U2.OUT11, X7-4.S
- new net N$47: U2.OUT12, X7-5.S
- new net N$48: U2.OUT13, X7-6.S
- new net N$49: U2.OUT14, X7-7.S
- new net N$50: U2.OUT15, X7-8.S
- net +24V: no longer U2.VPWR
- net GND: now also C11.2, C12.2, C13.2, C14.2, X5-1.S, X6-10.S, X7-10.S
- net VDD_JP4P5: now also C14.1
