File: tic12400.sch (EAGLE design)
At the start: 30 parts, among them U1 TIC12400DCPR, U2 MCZ33996EK, X1 22-23-2031, X2 INPUT1, X3 INPUT2, X4 INPUT3, X5 22-23-2031, X6 OUTPUT1, X7 OUTPUT2

Commit message: up
Parts:
- added F1, F2: 1206L020, polyfuse-smd_10:1206L020
- added R2, R5: 100, rcl:R-US_R0805
Connections:
- new net MOSI_SIG: R5.1, U1.SI, U2.SI
- new net N$31: D2.A, F1.2
- new net N$51: D1.A, F2.2
- new net SCK_SIG: R2.1, U1.SCLK, U2.SCLK
- net MOSI_JP4P3: now also R5.2; no longer U1.SI, U2.SI
- net N$29: now also F2.1; no longer D1.A
- net N$30: now also C11.1, C12.1, C13.1, D2.C, U2.VPWR; no longer D2.A, X5-2.S, X5-3.S
- net N$32: now also F1.1, X5-2.S, X5-3.S; no longer C11.1, C12.1, C13.1, D2.C, U2.VPWR
- net SCK_JP4P2: now also R2.2; no longer U1.SCLK, U2.SCLK
Other:
- moved on the sheet: D1, D2

Commit message: up
Parts:
- added C15: 1uf, rcl:C-USC0805
- added C16: 0.1, rcl:C-USC0805
- added LED1: SPI ACT, led:LEDCHIP-LED0805
- added LED2: POWER, led:LEDCHIP-LED0805
- added Q1: CSTCR6M00G53Z, murata-filter:CSTCR6M00G53Z
- added R6, R7, R8: 390, rcl:R-US_R0805
- added SV3: MCP2210_GPIO, con-lsta:FE10-1
- added U3: MCP2210-I/SO, MCP2210-I_SO:MCP2210-I/SO
- added X8: MINI-USB-32005-201, con-cypressindustries:MINI-USB-32005-201
Connections:
- removed net VDD_JP4P5: C14.1, C6.1, C7.1, R3.2, R4.1, SV1.7, SV2.7, U1.VDD, U2.SOPWR
- new net N$52: C15.1, U3.VUSB
- new net N$53: Q1.1, U3.OSC2
- new net N$54: R6.1, U3.!RST
- new net N$55: U3.D+, X8.3
- new net N$56: U3.D-, X8.2
- new net N$57: Q1.3, U3.OSC1
- new net N$58: LED2.A, R7.2
- new net N$59: LED1.A, R8.2
- new net N$60: R8.1, SV3.4, U3.GP3
- new net N$61: SV3.1, U3.GP0
- new net N$62: SV3.2, U3.GP1
- new net N$63: SV3.3, U3.GP2
- new net N$64: SV3.5, U3.GP4
- new net N$65: SV3.8, U3.GP7
- new net VDD: C14.1, C16.1, C6.1, C7.1, R3.2, R4.1, R6.2, R7.1, SV1.7, SV2.7, U1.VDD, U2.SOPWR, U3.VDD, X8.1
- net CS_JP3P11: now also SV3.6, U3.GP5
- net EXT2_JP3P8: now also SV3.7, U3.GP6
- net GND: now also C15.2, C16.2, LED1.C, LED2.C, Q1.2, SV3.10, U3.VSS, X8.5
- net MISO_JP4P1: now also U3.MISO
- net MOSI_SIG: now also U3.MOSI
- net N$33: now also SV3.9, U3.GP8
- net SCK_SIG: now also U3.SCK
Other:
- moved on the sheet: R3

Commit message: up
Parts:
- added R9: 100, rcl:R-US_R0805
- added TP1, TP2, TP3: PTR1B1,27, testpad:PTR1B1,27
Connections:
- new net N$66: R9.1, U3.MISO
- net GND: now also TP3.TP
- net MISO_JP4P1: now also R9.2; no longer U3.MISO
- net N$53: now also TP2.TP
- net N$54: now also TP1.TP
Changed lines of the file:
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@@
 <part name="VDD11" library="supply1" library_urn="urn:adsk.eagle:library:371" deviceset="VDD" device=""/>
 <part name="VDD12" library="supply1" library_urn="urn:adsk.eagle:library:371" deviceset="VDD" device=""/>
+<part name="R9" library="rcl" library_urn="urn:adsk.eagle:library:334" deviceset="R-US_" device="R0805" package3d_urn="urn:adsk.eagle:package:23553/2" value="100"/>
+<part name="TP1" library="testpad" library_urn="urn:adsk.eagle:library:385" deviceset="PTR1" device="B1,27" package3d_urn="urn:adsk.eagle:package:27944/2"/>
+<part name="TP2" library="testpad" library_urn="urn:adsk.eagle:library:385" deviceset="PTR1" device="B1,27" package3d_urn="urn:adsk.eagle:package:27944/2"/>
+<part name="TP3" library="testpad" library_urn="urn:adsk.eagle:library:385" deviceset="PTR1" device="B1,27" package3d_urn="urn:adsk.eagle:package:27944/2"/>
+<part name="GND35" library="supply1" library_urn="urn:adsk.eagle:library:371" deviceset="GND" device=""/>
 </parts>
 <sheets>
@@
 <instance part="VDD12" gate="G$1" x="172.72" y="190.5" smashed="yes">
 <attribute name="VALUE" x="170.18" y="187.96" size="1.778" layer="96" rot="R90"/>
+</instance>
+<instance part="R9" gate="G$1" x="-12.7" y="165.1" smashed="yes" rot="R180">
+<attribute name="NAME" x="-8.89" y="163.6014" size="1.778" layer="95" rot="R180"/>
+<attribute name="VALUE" x="-8.89" y="168.402" size="1.778" layer="96" rot="R180"/>
+</instance>
+<instance part="TP1" gate="G$1" x="-15.24" y="177.8" smashed="yes" rot="R180">
+<attribute name="NAME" x="-14.224" y="184.15" size="1.778" layer="95" rot="R270"/>
+<attribute name="TP_SIGNAL_NAME" x="-16.51" y="180.34" size="1.778" layer="97" rot="R180"/>
+</instance>
+<instance part="TP2" gate="G$1" x="20.32" y="157.48" smashed="yes" rot="R180">
+<attribute name="NAME" x="21.336" y="163.83" size="1.778" layer="95" rot="R270"/>
+<attribute name="TP_SIGNAL_NAME" x="19.05" y="160.02" size="1.778" layer="97" rot="R180"/>
+</instance>
+<instance part="TP3" gate="G$1" x="76.2" y="172.72" smashed="yes" rot="R180">
+<attribute name="NAME" x="77.216" y="179.07" size="1.778" layer="95" rot="R270"/>
+<attribute name="TP_SIGNAL_NAME" x="74.93" y="175.26" size="1.778" layer="97" rot="R180"/>
+</instance>
+<instance part="GND35" gate="1" x="76.2" y="167.64" smashed="yes">
+<attribute name="VALUE" x="73.66" y="165.1" size="1.778" layer="96"/>
 </instance>
 </instances>
@@
 <junction x="45.72" y="109.22"/>
 </segment>
+<segment>
+<pinref part="TP3" gate="G$1" pin="TP"/>
+<pinref part="GND35" gate="1" pin="GND"/>
+<junction x="76.2" y="170.18"/>
+</segment>
 </net>
 <net name="N$2" class="0">
@@
 </segment>
 <segment>
-<wire x1="-7.62" y1="165.1" x2="-12.7" y2="165.1" width="0.1524" layer="91"/>
-<pinref part="U3" gate="G$1" pin="MISO"/>
-<junction x="-7.62" y="165.1"/>
+<wire x1="-17.78" y1="165.1" x2="-17.78" y2="170.18" width="0.1524" layer="91"/>
+<pinref part="R9" gate="G$1" pin="2"/>
+<junction x="-17.78" y="165.1"/>
+<label x="-17.78" y="170.18" size="1.778" layer="95"/>
 </segment>
 </net>
@@
 <pinref part="R6" gate="G$1" pin="1"/>
 <junction x="-7.62" y="172.72"/>
+<wire x1="-7.62" y1="172.72" x2="-15.24" y2="172.72" width="0.1524" layer="91"/>
+<pinref part="TP1" gate="G$1" pin="TP"/>
+<wire x1="-15.24" y1="172.72" x2="-15.24" y2="175.26" width="0.1524" layer="91"/>
+<junction x="-15.24" y="175.26"/>
 </segment>
 </net>
@@
 <junction x="22.86" y="160.02"/>
 <junction x="22.86" y="165.1"/>
+<wire x1="22.86" y1="160.02" x2="22.86" y2="154.94" width="0.1524" layer="91"/>
+<pinref part="TP2" gate="G$1" pin="TP"/>
+<wire x1="22.86" y1="154.94" x2="20.32" y2="154.94" width="0.1524" layer="91"/>
+<junction x="20.32" y="154.94"/>
 </segment>
 </net>
@@
 </segment>
 </net>
+<net name="N$66" class="0">
+<segment>
+<pinref part="U3" gate="G$1" pin="MISO"/>
+<pinref part="R9" gate="G$1" pin="1"/>
+<junction x="-7.62" y="165.1"/>
+</segment>
+</net>

Commit message: up
Connections:
- net N$30: now also X6-9.S, X7-9.S
- net N$32: no longer X6-9.S, X7-9.S
Changed lines of the file:
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@@
 <pinref part="F1" gate="G$1" pin="1"/>
-</segment>
-<segment>
-<wire x1="144.78" y1="160.02" x2="134.62" y2="160.02" width="0.1524" layer="91"/>
-<pinref part="X6" gate="-9" pin="S"/>
-<junction x="144.78" y="160.02"/>
-</segment>
-<segment>
-<wire x1="162.56" y1="127" x2="152.4" y2="127" width="0.1524" layer="91"/>
-<pinref part="X7" gate="-9" pin="S"/>
-<junction x="162.56" y="127"/>
 </segment>
 </net>
@@
 <junction x="187.96" y="170.18"/>
 </segment>
-</net>
+<segment>
+<wire x1="144.78" y1="160.02" x2="134.62" y2="160.02" width="0.1524" layer="91"/>
+<pinref part="X6" gate="-9" pin="S"/>
+<junction x="144.78" y="160.02"/>
+</segment>
+<segment>
+<wire x1="162.56" y1="127" x2="152.4" y2="127" width="0.1524" layer="91"/>
+<pinref part="X7" gate="-9" pin="S"/>
+<junction x="162.56" y="127"/>
+</segment>
+</net>
