File: tic12400.sch (EAGLE design)
At the start: 49 parts, among them Q1 CSTCR6M00G53Z, U1 TIC12400DCPR, U2 MCZ33996EK, U3 MCP2210-I/SO, X1 22-23-2031, X2 INPUT1, X3 INPUT2, X4 INPUT3, X5 22-23-2031, X6 OUTPUT1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

Commit message: up
Parts:
- added OS1: OSC-OE-CFPS-73, IQD-Frequency-Products:OSC-OE-CFPS-73
Connections:
- removed net N$52: C15.1, U3.VUSB
- net GND: now also OS1.VSS
- net N$57: now also OS1.OUT
- net VDD: now also C15.1, OS1.CON, OS1.VDD, U3.VUSB
Changed lines of the file:
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@@
 <part name="TP3" library="testpad" library_urn="urn:adsk.eagle:library:385" deviceset="PTR1" device="B1,27" package3d_urn="urn:adsk.eagle:package:27944/2"/>
 <part name="GND35" library="supply1" library_urn="urn:adsk.eagle:library:371" deviceset="GND" device=""/>
+<part name="VDD13" library="supply1" library_urn="urn:adsk.eagle:library:371" deviceset="VDD" device=""/>
+<part name="OS1" library="IQD-Frequency-Products" library_urn="urn:adsk.eagle:library:90" deviceset="OSC-OE" device="-CFPS-73" package3d_urn="urn:adsk.eagle:package:3365/1"/>
+<part name="GND36" library="supply1" library_urn="urn:adsk.eagle:library:371" deviceset="GND" device=""/>
+<part name="VDD14" library="supply1" library_urn="urn:adsk.eagle:library:371" deviceset="VDD" device=""/>
+<part name="VDD15" library="supply1" library_urn="urn:adsk.eagle:library:371" deviceset="VDD" device=""/>
 </parts>
 <sheets>
@@
 <instance part="GND35" gate="1" x="76.2" y="167.64" smashed="yes">
 <attribute name="VALUE" x="73.66" y="165.1" size="1.778" layer="96"/>
+</instance>
+<instance part="VDD13" gate="G$1" x="30.48" y="175.26" smashed="yes" rot="R180">
+<attribute name="VALUE" x="33.02" y="177.8" size="1.778" layer="96" rot="R270"/>
+</instance>
+<instance part="OS1" gate="A" x="83.82" y="190.5" smashed="yes">
+<attribute name="NAME" x="76.2" y="198.755" size="1.778" layer="95"/>
+<attribute name="VALUE" x="76.2" y="180.34" size="1.778" layer="96"/>
+</instance>
+<instance part="GND36" gate="1" x="71.12" y="182.88" smashed="yes">
+<attribute name="VALUE" x="68.58" y="180.34" size="1.778" layer="96"/>
+</instance>
+<instance part="VDD14" gate="G$1" x="71.12" y="193.04" smashed="yes" rot="R180">
+<attribute name="VALUE" x="73.66" y="195.58" size="1.778" layer="96" rot="R270"/>
+</instance>
+<instance part="VDD15" gate="G$1" x="99.06" y="195.58" smashed="yes" rot="R270">
+<attribute name="VALUE" x="96.52" y="198.12" size="1.778" layer="96"/>
 </instance>
 </instances>
@@
 <junction x="76.2" y="170.18"/>
 </segment>
+<segment>
+<pinref part="OS1" gate="A" pin="VSS"/>
+<pinref part="GND36" gate="1" pin="GND"/>
+<junction x="71.12" y="185.42"/>
+</segment>
 </net>
 <net name="N$2" class="0">
@@
 <pinref part="U3" gate="G$1" pin="MOSI"/>
 <junction x="-7.62" y="162.56"/>
-</segment>
-</net>
-<net name="N$52" class="0">
-<segment>
-<pinref part="U3" gate="G$1" pin="VUSB"/>
-<wire x1="22.86" y1="177.8" x2="38.1" y2="177.8" width="0.1524" layer="91"/>
-<pinref part="C15" gate="G$1" pin="1"/>
-<junction x="22.86" y="177.8"/>
-<junction x="38.1" y="177.8"/>
 </segment>
 </net>
@@
 <junction x="10.16" y="58.42"/>
 </segment>
+<segment>
+<pinref part="U3" gate="G$1" pin="VUSB"/>
+<wire x1="22.86" y1="177.8" x2="30.48" y2="177.8" width="0.1524" layer="91"/>
+<pinref part="C15" gate="G$1" pin="1"/>
+<junction x="22.86" y="177.8"/>
+<junction x="38.1" y="177.8"/>
+<pinref part="VDD13" gate="G$1" pin="VDD"/>
+<wire x1="30.48" y1="177.8" x2="38.1" y2="177.8" width="0.1524" layer="91"/>
+<junction x="30.48" y="177.8"/>
+</segment>
+<segment>
+<pinref part="OS1" gate="A" pin="VDD"/>
+<pinref part="VDD14" gate="G$1" pin="VDD"/>
+<junction x="71.12" y="195.58"/>
+</segment>
+<segment>
+<pinref part="OS1" gate="A" pin="CON"/>
+<pinref part="VDD15" gate="G$1" pin="VDD"/>
+<junction x="96.52" y="195.58"/>
+</segment>
 </net>
 <net name="N$55" class="0">
@@
 <junction x="38.1" y="160.02"/>
 <junction x="22.86" y="167.64"/>
-</segment>
-</net>
+<label x="25.4" y="170.18" size="1.778" layer="95"/>
+</segment>
+<segment>
+<wire x1="101.6" y1="190.5" x2="96.52" y2="190.5" width="0.1524" layer="91"/>
+<pinref part="OS1" gate="A" pin="OUT"/>
+<label x="104.14" y="187.96" size="1.778" layer="95"/>
+<junction x="96.52" y="190.5"/>
+</segment>
+</net>

Commit message: up
Parts:
- added TP4: PTR1B1,27, testpad:PTR1B1,27
Connections:
- new net N$52: C15.1, U3.VUSB
- net N$57: now also TP4.TP
- net VDD: no longer C15.1, U3.VUSB
Changed lines of the file:
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@@
 <part name="TP3" library="testpad" library_urn="urn:adsk.eagle:library:385" deviceset="PTR1" device="B1,27" package3d_urn="urn:adsk.eagle:package:27944/2"/>
 <part name="GND35" library="supply1" library_urn="urn:adsk.eagle:library:371" deviceset="GND" device=""/>
-<part name="VDD13" library="supply1" library_urn="urn:adsk.eagle:library:371" deviceset="VDD" device=""/>
 <part name="OS1" library="IQD-Frequency-Products" library_urn="urn:adsk.eagle:library:90" deviceset="OSC-OE" device="-CFPS-73" package3d_urn="urn:adsk.eagle:package:3365/1"/>
 <part name="GND36" library="supply1" library_urn="urn:adsk.eagle:library:371" deviceset="GND" device=""/>
 <part name="VDD14" library="supply1" library_urn="urn:adsk.eagle:library:371" deviceset="VDD" device=""/>
 <part name="VDD15" library="supply1" library_urn="urn:adsk.eagle:library:371" deviceset="VDD" device=""/>
+<part name="TP4" library="testpad" library_urn="urn:adsk.eagle:library:385" deviceset="PTR1" device="B1,27" package3d_urn="urn:adsk.eagle:package:27944/2"/>
 </parts>
 <sheets>
@@
 <attribute name="VALUE" x="73.66" y="165.1" size="1.778" layer="96"/>
 </instance>
-<instance part="VDD13" gate="G$1" x="30.48" y="175.26" smashed="yes" rot="R180">
-<attribute name="VALUE" x="33.02" y="177.8" size="1.778" layer="96" rot="R270"/>
-</instance>
 <instance part="OS1" gate="A" x="83.82" y="190.5" smashed="yes">
 <attribute name="NAME" x="76.2" y="198.755" size="1.778" layer="95"/>
@@
 <instance part="VDD15" gate="G$1" x="99.06" y="195.58" smashed="yes" rot="R270">
 <attribute name="VALUE" x="96.52" y="198.12" size="1.778" layer="96"/>
+</instance>
+<instance part="TP4" gate="G$1" x="104.14" y="190.5" smashed="yes" rot="R90">
+<attribute name="NAME" x="110.49" y="189.484" size="1.778" layer="95" rot="R180"/>
+<attribute name="TP_SIGNAL_NAME" x="106.68" y="191.77" size="1.778" layer="97" rot="R90"/>
 </instance>
 </instances>
@@
 </segment>
 <segment>
-<pinref part="U3" gate="G$1" pin="VUSB"/>
-<wire x1="22.86" y1="177.8" x2="30.48" y2="177.8" width="0.1524" layer="91"/>
-<pinref part="C15" gate="G$1" pin="1"/>
-<junction x="22.86" y="177.8"/>
-<junction x="38.1" y="177.8"/>
-<pinref part="VDD13" gate="G$1" pin="VDD"/>
-<wire x1="30.48" y1="177.8" x2="38.1" y2="177.8" width="0.1524" layer="91"/>
-<junction x="30.48" y="177.8"/>
-</segment>
-<segment>
 <pinref part="OS1" gate="A" pin="VDD"/>
 <pinref part="VDD14" gate="G$1" pin="VDD"/>
@@
 <wire x1="101.6" y1="190.5" x2="96.52" y2="190.5" width="0.1524" layer="91"/>
 <pinref part="OS1" gate="A" pin="OUT"/>
-<label x="104.14" y="187.96" size="1.778" layer="95"/>
+<label x="99.06" y="187.96" size="1.778" layer="95"/>
 <junction x="96.52" y="190.5"/>
+<pinref part="TP4" gate="G$1" pin="TP"/>
+<junction x="101.6" y="190.5"/>
 </segment>
 </net>
@@
 </segment>
 </net>
+<net name="N$52" class="1">
+<segment>
+<pinref part="U3" gate="G$1" pin="VUSB"/>
+<pinref part="C15" gate="G$1" pin="1"/>
+<junction x="22.86" y="177.8"/>
+<junction x="38.1" y="177.8"/>
+<wire x1="22.86" y1="177.8" x2="38.1" y2="177.8" width="0.1524" layer="91"/>
+</segment>
+</net>

Commit message: up
Parts:
- removed LED1: SPI ACT, led:LEDCHIP-LED0805
- added LED3: SPI ACT, led:LEDCHIP-LED0805
Connections:
- net GND: no longer LED1.C
- net N$33: no longer SV1.4, SV2.4, U2.!CS
- net N$59: now also LED3.C; no longer LED1.A
- net N$65: now also SV1.4, SV2.4, U2.!CS
- net VDD: now also LED3.A
Changed lines of the file:
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@@
 <part name="Q1" library="murata-filter" library_urn="urn:adsk.eagle:library:303" deviceset="CSTCR" device="" package3d_urn="urn:adsk.eagle:package:21145/1" technology="6M00G53Z"/>
 <part name="GND31" library="supply1" library_urn="urn:adsk.eagle:library:371" deviceset="GND" device=""/>
-<part name="LED1" library="led" library_urn="urn:adsk.eagle:library:259" deviceset="LED" device="CHIP-LED0805" package3d_urn="urn:adsk.eagle:package:15818/2" value="SPI ACT"/>
 <part name="LED2" library="led" library_urn="urn:adsk.eagle:library:259" deviceset="LED" device="CHIP-LED0805" package3d_urn="urn:adsk.eagle:package:15818/2" value="POWER"/>
 <part name="R7" library="rcl" library_urn="urn:adsk.eagle:library:334" deviceset="R-US_" device="R0805" package3d_urn="urn:adsk.eagle:package:23553/2" value="390"/>
@@
 <part name="GND32" library="supply1" library_urn="urn:adsk.eagle:library:371" deviceset="GND" device=""/>
 <part name="R8" library="rcl" library_urn="urn:adsk.eagle:library:334" deviceset="R-US_" device="R0805" package3d_urn="urn:adsk.eagle:package:23553/2" value="390"/>
-<part name="GND33" library="supply1" library_urn="urn:adsk.eagle:library:371" deviceset="GND" device=""/>
 <part name="SV3" library="con-lsta" library_urn="urn:adsk.eagle:library:161" deviceset="FE10-1" device="" package3d_urn="urn:adsk.eagle:package:8192/1" value="MCP2210_GPIO"/>
 <part name="GND34" library="supply1" library_urn="urn:adsk.eagle:library:371" deviceset="GND" device=""/>
@@
 <part name="VDD15" library="supply1" library_urn="urn:adsk.eagle:library:371" deviceset="VDD" device=""/>
 <part name="TP4" library="testpad" library_urn="urn:adsk.eagle:library:385" deviceset="PTR1" device="B1,27" package3d_urn="urn:adsk.eagle:package:27944/2"/>
+<part name="LED3" library="led" library_urn="urn:adsk.eagle:library:259" deviceset="LED" device="CHIP-LED0805" package3d_urn="urn:adsk.eagle:package:15818/2" value="SPI ACT"/>
+<part name="VDD13" library="supply1" library_urn="urn:adsk.eagle:library:371" deviceset="VDD" device=""/>
 </parts>
 <sheets>
@@
 <attribute name="VALUE" x="33.02" y="147.32" size="1.778" layer="96"/>
 </instance>
-<instance part="LED1" gate="G$1" x="-12.7" y="124.46" smashed="yes">
-<attribute name="NAME" x="-9.144" y="119.888" size="1.778" layer="95" rot="R90"/>
-<attribute name="VALUE" x="-6.985" y="119.888" size="1.778" layer="96" rot="R90"/>
-</instance>
 <instance part="LED2" gate="G$1" x="10.16" y="111.76" smashed="yes">
 <attribute name="NAME" x="13.716" y="107.188" size="1.778" layer="95" rot="R90"/>
@@
 <attribute name="VALUE" x="-16.002" y="135.89" size="1.778" layer="96" rot="R270"/>
 </instance>
-<instance part="GND33" gate="1" x="-12.7" y="116.84" smashed="yes">
-<attribute name="VALUE" x="-15.24" y="114.3" size="1.778" layer="96"/>
-</instance>
 <instance part="SV3" gate="G$1" x="58.42" y="101.6" smashed="yes" rot="R90">
 <attribute name="VALUE" x="73.66" y="100.33" size="1.778" layer="96" rot="R90"/>
@@
 <attribute name="NAME" x="110.49" y="189.484" size="1.778" layer="95" rot="R180"/>
 <attribute name="TP_SIGNAL_NAME" x="106.68" y="191.77" size="1.778" layer="97" rot="R90"/>
+</instance>
+<instance part="LED3" gate="G$1" x="-12.7" y="121.92" smashed="yes" rot="R180">
+<attribute name="NAME" x="-16.256" y="126.492" size="1.778" layer="95" rot="R270"/>
+<attribute name="VALUE" x="-18.415" y="126.492" size="1.778" layer="96" rot="R270"/>
+</instance>
+<instance part="VDD13" gate="G$1" x="-12.7" y="116.84" smashed="yes" rot="R180">
+<attribute name="VALUE" x="-10.16" y="119.38" size="1.778" layer="96" rot="R270"/>
 </instance>
 </instances>
@@
 </segment>
 <segment>
-<pinref part="LED1" gate="G$1" pin="C"/>
-<pinref part="GND33" gate="1" pin="GND"/>
-<junction x="-12.7" y="119.38"/>
-</segment>
-<segment>
 <pinref part="SV3" gate="G$1" pin="10"/>
 <pinref part="GND34" gate="1" pin="GND"/>
@@
 </net>
 <net name="N$33" class="0">
-<segment>
-<pinref part="SV1" gate="1" pin="4"/>
-<pinref part="SV2" gate="G$1" pin="4"/>
-<wire x1="63.5" y1="20.32" x2="63.5" y2="43.18" width="0.1524" layer="91"/>
-<wire x1="63.5" y1="43.18" x2="63.5" y2="48.26" width="0.1524" layer="91"/>
-<junction x="63.5" y="43.18"/>
-</segment>
-<segment>
-<wire x1="187.96" y1="160.02" x2="182.88" y2="160.02" width="0.1524" layer="91"/>
-<pinref part="U2" gate="G$1" pin="!CS"/>
-<junction x="187.96" y="160.02"/>
-<label x="157.48" y="160.02" size="1.778" layer="95"/>
-</segment>
 <segment>
 <wire x1="27.94" y1="142.24" x2="22.86" y2="142.24" width="0.1524" layer="91"/>
@@
 <label x="-12.7" y="109.22" size="1.778" layer="95"/>
 <junction x="-2.54" y="109.22"/>
+<junction x="-2.54" y="114.3"/>
 </segment>
 <segment>
@@
 <pinref part="VDD15" gate="G$1" pin="VDD"/>
 <junction x="96.52" y="195.58"/>
+</segment>
+<segment>
+<pinref part="LED3" gate="G$1" pin="A"/>
+<pinref part="VDD13" gate="G$1" pin="VDD"/>
+<junction x="-12.7" y="119.38"/>
 </segment>
 </net>
@@
 </segment>
 </net>
-<net name="N$59" class="0">
-<segment>
-<pinref part="LED1" gate="G$1" pin="A"/>
-<pinref part="R8" gate="G$1" pin="2"/>
-<junction x="-12.7" y="127"/>
-</segment>
-</net>
 <net name="N$60" class="0">
 <segment>
@@
 <junction x="50.8" y="109.22"/>
 </segment>
+<segment>
+<wire x1="180.34" y1="160.02" x2="187.96" y2="160.02" width="0.1524" layer="91"/>
+<pinref part="U2" gate="G$1" pin="!CS"/>
+<junction x="187.96" y="160.02"/>
+</segment>
+<segment>
+<wire x1="63.5" y1="43.18" x2="63.5" y2="50.8" width="0.1524" layer="91"/>
+<pinref part="SV2" gate="G$1" pin="4"/>
+<junction x="63.5" y="43.18"/>
+</segment>
+<segment>
+<wire x1="63.5" y1="20.32" x2="63.5" y2="27.94" width="0.1524" layer="91"/>
+<pinref part="SV1" gate="1" pin="4"/>
+<junction x="63.5" y="20.32"/>
+</segment>
 </net>
 <net name="N$66" class="0">
@@
 </segment>
 </net>
+<net name="N$59" class="0">
+<segment>
+<pinref part="R8" gate="G$1" pin="2"/>
+<pinref part="LED3" gate="G$1" pin="C"/>
+<junction x="-12.7" y="127"/>
+</segment>
+</net>

Commit message: up
Parts:
- added C17: 0.1, rcl:C-USC0805
Connections:
- net GND: now also C17.2
- net N$52: now also C17.1, OS1.CON, OS1.VDD
- net N$54: now also U2.!RST
- net N$6: no longer U2.!RST
- net VDD: no longer OS1.CON, OS1.VDD
Changed lines of the file:
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@@
 <part name="OS1" library="IQD-Frequency-Products" library_urn="urn:adsk.eagle:library:90" deviceset="OSC-OE" device="-CFPS-73" package3d_urn="urn:adsk.eagle:package:3365/1"/>
 <part name="GND36" library="supply1" library_urn="urn:adsk.eagle:library:371" deviceset="GND" device=""/>
-<part name="VDD14" library="supply1" library_urn="urn:adsk.eagle:library:371" deviceset="VDD" device=""/>
-<part name="VDD15" library="supply1" library_urn="urn:adsk.eagle:library:371" deviceset="VDD" device=""/>
 <part name="TP4" library="testpad" library_urn="urn:adsk.eagle:library:385" deviceset="PTR1" device="B1,27" package3d_urn="urn:adsk.eagle:package:27944/2"/>
 <part name="LED3" library="led" library_urn="urn:adsk.eagle:library:259" deviceset="LED" device="CHIP-LED0805" package3d_urn="urn:adsk.eagle:package:15818/2" value="SPI ACT"/>
 <part name="VDD13" library="supply1" library_urn="urn:adsk.eagle:library:371" deviceset="VDD" device=""/>
+<part name="C17" library="rcl" library_urn="urn:adsk.eagle:library:334" deviceset="C-US" device="C0805" package3d_urn="urn:adsk.eagle:package:23617/2" value="0.1"/>
+<part name="GND33" library="supply1" library_urn="urn:adsk.eagle:library:371" deviceset="GND" device=""/>
 </parts>
 <sheets>
@@
 <attribute name="VALUE" x="68.58" y="180.34" size="1.778" layer="96"/>
 </instance>
-<instance part="VDD14" gate="G$1" x="71.12" y="193.04" smashed="yes" rot="R180">
-<attribute name="VALUE" x="73.66" y="195.58" size="1.778" layer="96" rot="R270"/>
-</instance>
-<instance part="VDD15" gate="G$1" x="99.06" y="195.58" smashed="yes" rot="R270">
-<attribute name="VALUE" x="96.52" y="198.12" size="1.778" layer="96"/>
-</instance>
 <instance part="TP4" gate="G$1" x="104.14" y="190.5" smashed="yes" rot="R90">
 <attribute name="NAME" x="110.49" y="189.484" size="1.778" layer="95" rot="R180"/>
@@
 <instance part="VDD13" gate="G$1" x="-12.7" y="116.84" smashed="yes" rot="R180">
 <attribute name="VALUE" x="-10.16" y="119.38" size="1.778" layer="96" rot="R270"/>
+</instance>
+<instance part="C17" gate="G$1" x="33.02" y="175.26" smashed="yes">
+<attribute name="NAME" x="34.036" y="175.895" size="1.778" layer="95"/>
+<attribute name="VALUE" x="34.036" y="171.069" size="1.778" layer="96"/>
+</instance>
+<instance part="GND33" gate="1" x="33.02" y="167.64" smashed="yes">
+<attribute name="VALUE" x="30.48" y="165.1" size="1.778" layer="96"/>
 </instance>
 </instances>
@@
 <pinref part="U1" gate="G$1" pin="RESET"/>
 <junction x="198.12" y="60.96"/>
-</segment>
-<segment>
-<wire x1="187.96" y1="162.56" x2="172.72" y2="162.56" width="0.1524" layer="91"/>
-<pinref part="U2" gate="G$1" pin="!RST"/>
-<junction x="187.96" y="162.56"/>
 </segment>
 </net>
@@
 <pinref part="C15" gate="G$1" pin="2"/>
 <pinref part="GND28" gate="1" pin="GND"/>
+<junction x="38.1" y="170.18"/>
 </segment>
 <segment>
@@
 <pinref part="GND36" gate="1" pin="GND"/>
 <junction x="71.12" y="185.42"/>
+</segment>
+<segment>
+<pinref part="C17" gate="G$1" pin="2"/>
+<pinref part="GND33" gate="1" pin="GND"/>
+<junction x="33.02" y="170.18"/>
 </segment>
 </net>
@@
 <wire x1="-15.24" y1="172.72" x2="-15.24" y2="175.26" width="0.1524" layer="91"/>
 <junction x="-15.24" y="175.26"/>
+</segment>
+<segment>
+<wire x1="187.96" y1="162.56" x2="180.34" y2="162.56" width="0.1524" layer="91"/>
+<pinref part="U2" gate="G$1" pin="!RST"/>
 </segment>
 </net>
@@
 </segment>
 <segment>
-<pinref part="OS1" gate="A" pin="VDD"/>
-<pinref part="VDD14" gate="G$1" pin="VDD"/>
-<junction x="71.12" y="195.58"/>
-</segment>
-<segment>
-<pinref part="OS1" gate="A" pin="CON"/>
-<pinref part="VDD15" gate="G$1" pin="VDD"/>
-<junction x="96.52" y="195.58"/>
-</segment>
-<segment>
 <pinref part="LED3" gate="G$1" pin="A"/>
 <pinref part="VDD13" gate="G$1" pin="VDD"/>
@@
 <junction x="22.86" y="177.8"/>
 <junction x="38.1" y="177.8"/>
-<wire x1="22.86" y1="177.8" x2="38.1" y2="177.8" width="0.1524" layer="91"/>
-</segment>
-</net>
+<wire x1="22.86" y1="177.8" x2="33.02" y2="177.8" width="0.1524" layer="91"/>
+<pinref part="C17" gate="G$1" pin="1"/>
+<wire x1="33.02" y1="177.8" x2="38.1" y2="177.8" width="0.1524" layer="91"/>
+<junction x="33.02" y="177.8"/>
+<label x="43.18" y="175.26" size="1.778" layer="95"/>
+</segment>
+<segment>
+<wire x1="96.52" y1="195.58" x2="106.68" y2="195.58" width="0.1524" layer="91"/>
+<pinref part="OS1" gate="A" pin="CON"/>
+<label x="99.06" y="195.58" size="1.778" layer="95"/>
+<junction x="96.52" y="195.58"/>
+</segment>
+<segment>
+<wire x1="60.96" y1="195.58" x2="71.12" y2="195.58" width="0.1524" layer="91"/>
+<pinref part="OS1" gate="A" pin="VDD"/>
+<junction x="71.12" y="195.58"/>
+<label x="66.04" y="193.04" size="1.778" layer="95"/>
+</segment>
+</net>
