File: imu/pic32mk/imu.brd (EAGLE design)
At the start: 160 x 100 mm, 6 parts

Commit message: up
Parts:
- added SV7: J601, con-lstb:MA17-2W
- added SV8: LCD, con-lstb:MA10-1
Connections:
- new net N$1: SV7.2, SV8.3
- new net N$3: SV7.12, SV8.2
- new net N$4: SV7.13, SV8.5
- new net N$5: SV7.14, SV8.4
- new net N$6: SV7.16, SV8.6
- net +3V3: now also SV8.7
- net GND: now also SV8.8
Routing:
- net N$1: track 0.00 -> 57.3 mm
- net N$3: track 0.00 -> 45.6 mm
- net +3V3: track 64.7 -> 108.7 mm
- net N$5: track 0.00 -> 40.8 mm
- net N$4: track 0.00 -> 38.6 mm
- net GND: track 116.1 -> 152.3 mm
- net N$6: track 0.00 -> 36.1 mm
Changed lines of the file:
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@@
 <attribute name="VALUE" x="89.535" y="58.801" size="1.27" layer="27" ratio="10"/>
+</element>
+<element name="SV7" library="con-lstb" library_urn="urn:adsk.eagle:library:162" package="MA17-2W" package3d_urn="urn:adsk.eagle:package:8356/1" value="J601" x="67.31" y="86.36" smashed="yes">
+<attribute name="MF" value="" x="67.31" y="86.36" size="1.778" layer="27" display="off"/>
+<attribute name="MPN" value="" x="67.31" y="86.36" size="1.778" layer="27" display="off"/>
+<attribute name="NAME" x="45.847" y="82.55" size="1.27" layer="25" ratio="10"/>
+<attribute name="OC_FARNELL" value="unknown" x="67.31" y="86.36" size="1.778" layer="27" display="off"/>
+<attribute name="OC_NEWARK" value="unknown" x="67.31" y="86.36" size="1.778" layer="27" display="off"/>
+<attribute name="POPULARITY" value="0" x="67.31" y="86.36" size="1.778" layer="27" display="off"/>
+<attribute name="VALUE" x="54.61" y="82.55" size="1.27" layer="27" ratio="10"/>
+</element>
+<element name="SV8" library="con-lstb" library_urn="urn:adsk.eagle:library:162" package="MA10-1" package3d_urn="urn:adsk.eagle:package:8346/1" value="LCD" x="100.33" y="85.09" smashed="yes" rot="R90">
+<attribute name="MF" value="" x="100.33" y="85.09" size="1.778" layer="27" rot="R90" display="off"/>
+<attribute name="MPN" value="" x="100.33" y="85.09" size="1.778" layer="27" rot="R90" display="off"/>
+<attribute name="NAME" x="98.679" y="72.39" size="1.27" layer="25" ratio="10" rot="R90"/>
+<attribute name="OC_FARNELL" value="unknown" x="100.33" y="85.09" size="1.778" layer="27" rot="R90" display="off"/>
+<attribute name="OC_NEWARK" value="unknown" x="100.33" y="85.09" size="1.778" layer="27" rot="R90" display="off"/>
+<attribute name="POPULARITY" value="4" x="100.33" y="85.09" size="1.778" layer="27" rot="R90" display="off"/>
+<attribute name="VALUE" x="104.521" y="86.36" size="1.27" layer="27" ratio="10" rot="R90"/>
 </element>
 </elements>
@@
 <contactref element="SV4" pad="3"/>
 <contactref element="SV6" pad="1"/>
-<wire x1="106.68" y1="35.6616" x2="112.9284" y2="35.6616" width="0.1524" layer="1"/>
-<wire x1="85.1916" y1="57.15" x2="106.68" y2="35.6616" width="0.1524" layer="1"/>
-<wire x1="112.9284" y1="35.6616" x2="113.03" y2="35.56" width="0.1524" layer="1"/>
-<wire x1="85.1916" y1="57.15" x2="85.09" y2="57.15" width="0.1524" layer="1"/>
+<contactref element="SV8" pad="8"/>
 <wire x1="54.7116" y1="38.1" x2="54.7116" y2="35.6616" width="0.1524" layer="1"/>
 <wire x1="54.7116" y1="35.6616" x2="54.61" y2="35.56" width="0.1524" layer="1"/>
@@
 <wire x1="76.2" y1="14.0208" x2="83.82" y2="14.0208" width="0.1524" layer="1"/>
 <wire x1="54.7116" y1="35.5092" x2="76.2" y2="14.0208" width="0.1524" layer="1"/>
+<wire x1="54.7116" y1="35.5092" x2="54.61" y2="35.56" width="0.1524" layer="1"/>
+<wire x1="106.68" y1="35.6616" x2="105.3084" y2="37.0332" width="0.1524" layer="1"/>
+<wire x1="105.3084" y1="37.0332" x2="85.1916" y2="57.15" width="0.1524" layer="1"/>
+<wire x1="112.9284" y1="35.6616" x2="106.68" y2="35.6616" width="0.1524" layer="1"/>
+<wire x1="112.9284" y1="35.6616" x2="113.03" y2="35.56" width="0.1524" layer="1"/>
+<wire x1="100.4316" y1="90.9828" x2="100.4316" y2="91.44" width="0.1524" layer="1"/>
+<wire x1="102.108" y1="89.3064" x2="100.4316" y2="90.9828" width="0.1524" layer="1"/>
+<wire x1="102.108" y1="73.152" x2="102.108" y2="89.3064" width="0.1524" layer="1"/>
+<wire x1="87.9348" y1="58.9788" x2="102.108" y2="73.152" width="0.1524" layer="1"/>
+<wire x1="87.0204" y1="58.9788" x2="87.9348" y2="58.9788" width="0.1524" layer="1"/>
+<wire x1="85.1916" y1="57.15" x2="87.0204" y2="58.9788" width="0.1524" layer="1"/>
+<wire x1="100.4316" y1="91.44" x2="100.33" y2="91.44" width="0.1524" layer="1"/>
+<wire x1="85.1916" y1="57.15" x2="85.09" y2="57.15" width="0.1524" layer="1"/>
+<wire x1="83.82" y1="15.0876" x2="83.82" y2="14.0208" width="0.1524" layer="1"/>
+<wire x1="85.344" y1="16.6116" x2="83.82" y2="15.0876" width="0.1524" layer="1"/>
+<wire x1="85.344" y1="17.0688" x2="85.344" y2="16.6116" width="0.1524" layer="1"/>
+<wire x1="105.3084" y1="37.0332" x2="85.344" y2="17.0688" width="0.1524" layer="1"/>
 <wire x1="83.82" y1="14.0208" x2="83.82" y2="13.97" width="0.1524" layer="1"/>
-<wire x1="54.7116" y1="35.5092" x2="54.61" y2="35.56" width="0.1524" layer="1"/>
-<wire x1="73.7616" y1="57.15" x2="85.09" y2="57.15" width="0.1524" layer="16"/>
-<wire x1="54.7116" y1="38.1" x2="73.7616" y2="57.15" width="0.1524" layer="16"/>
-<wire x1="54.7116" y1="38.1" x2="54.61" y2="38.1" width="0.1524" layer="16"/>
 </signal>
 <signal name="+3V3">
 <contactref element="SV4" pad="7"/>
 <contactref element="SV1" pad="8"/>
-<wire x1="69.7992" y1="33.0708" x2="112.9284" y2="33.0708" width="0.1524" layer="1"/>
-<wire x1="54.61" y1="48.26" x2="69.7992" y2="33.0708" width="0.1524" layer="1"/>
-<wire x1="112.9284" y1="33.0708" x2="113.03" y2="33.02" width="0.1524" layer="1"/>
+<contactref element="SV8" pad="7"/>
+<wire x1="112.9284" y1="33.3756" x2="112.9284" y2="33.0708" width="0.1524" layer="16"/>
+<wire x1="102.108" y1="44.196" x2="112.9284" y2="33.3756" width="0.1524" layer="16"/>
+<wire x1="102.108" y1="87.1728" x2="102.108" y2="48.3108" width="0.1524" layer="16"/>
+<wire x1="102.108" y1="48.3108" x2="102.108" y2="44.196" width="0.1524" layer="16"/>
+<wire x1="100.4316" y1="88.8492" x2="102.108" y2="87.1728" width="0.1524" layer="16"/>
+<wire x1="112.9284" y1="33.0708" x2="113.03" y2="33.02" width="0.1524" layer="16"/>
+<wire x1="100.4316" y1="88.8492" x2="100.33" y2="88.9" width="0.1524" layer="16"/>
+<wire x1="102.108" y1="48.3108" x2="54.7116" y2="48.3108" width="0.1524" layer="16"/>
+<wire x1="54.7116" y1="48.3108" x2="54.61" y2="48.26" width="0.1524" layer="16"/>
 </signal>
 <signal name="SLC">
@@
 <wire x1="92.8116" y1="57.15" x2="92.71" y2="57.15" width="0.1524" layer="1"/>
 </signal>
+<signal name="N$1">
+<contactref element="SV8" pad="3"/>
+<contactref element="SV7" pad="2"/>
+<wire x1="56.8452" y1="78.7908" x2="100.2792" y2="78.7908" width="0.1524" layer="1"/>
+<wire x1="50.5968" y1="85.0392" x2="56.8452" y2="78.7908" width="0.1524" layer="1"/>
+<wire x1="50.5968" y1="85.4964" x2="50.5968" y2="85.0392" width="0.1524" layer="1"/>
+<wire x1="49.53" y1="86.5632" x2="50.5968" y2="85.4964" width="0.1524" layer="1"/>
+<wire x1="48.1584" y1="86.5632" x2="49.53" y2="86.5632" width="0.1524" layer="1"/>
+<wire x1="47.0916" y1="87.63" x2="48.1584" y2="86.5632" width="0.1524" layer="1"/>
+<wire x1="100.2792" y1="78.7908" x2="100.33" y2="78.74" width="0.1524" layer="1"/>
+<wire x1="47.0916" y1="87.63" x2="46.99" y2="87.63" width="0.1524" layer="1"/>
+</signal>
+<signal name="N$3">
+<contactref element="SV8" pad="2"/>
+<contactref element="SV7" pad="12"/>
+<wire x1="72.2376" y1="76.2" x2="100.33" y2="76.2" width="0.1524" layer="16"/>
+<wire x1="63.246" y1="85.1916" x2="72.2376" y2="76.2" width="0.1524" layer="16"/>
+<wire x1="63.246" y1="85.4964" x2="63.246" y2="85.1916" width="0.1524" layer="16"/>
+<wire x1="62.1792" y1="86.5632" x2="63.246" y2="85.4964" width="0.1524" layer="16"/>
+<wire x1="60.8076" y1="86.5632" x2="62.1792" y2="86.5632" width="0.1524" layer="16"/>
+<wire x1="59.7408" y1="87.63" x2="60.8076" y2="86.5632" width="0.1524" layer="16"/>
+<wire x1="59.7408" y1="87.63" x2="59.69" y2="87.63" width="0.1524" layer="16"/>
+</signal>
+<signal name="N$4">
+<contactref element="SV8" pad="5"/>
+<contactref element="SV7" pad="13"/>
+<wire x1="63.5508" y1="83.82" x2="100.33" y2="83.82" width="0.1524" layer="1"/>
+<wire x1="62.3316" y1="85.0392" x2="63.5508" y2="83.82" width="0.1524" layer="1"/>
+<wire x1="62.3316" y1="85.0392" x2="62.23" y2="85.09" width="0.1524" layer="1"/>
+</signal>
+<signal name="N$5">
+<contactref element="SV8" pad="4"/>
+<contactref element="SV7" pad="14"/>
+<wire x1="92.8116" y1="81.3816" x2="100.2792" y2="81.3816" width="0.1524" layer="16"/>
+<wire x1="87.63" y1="86.5632" x2="92.8116" y2="81.3816" width="0.1524" layer="16"/>
+<wire x1="63.3984" y1="86.5632" x2="87.63" y2="86.5632" width="0.1524" layer="16"/>
+<wire x1="62.3316" y1="87.63" x2="63.3984" y2="86.5632" width="0.1524" layer="16"/>
+<wire x1="100.2792" y1="81.3816" x2="100.33" y2="81.28" width="0.1524" layer="16"/>
+<wire x1="62.3316" y1="87.63" x2="62.23" y2="87.63" width="0.1524" layer="16"/>
+</signal>
+<signal name="N$6">
+<contactref element="SV8" pad="6"/>
+<contactref element="SV7" pad="16"/>
+<wire x1="65.9892" y1="86.4108" x2="100.2792" y2="86.4108" width="0.1524" layer="1"/>
+<wire x1="64.77" y1="87.63" x2="65.9892" y2="86.4108" width="0.1524" layer="1"/>
+<wire x1="100.2792" y1="86.4108" x2="100.33" y2="86.36" width="0.1524" layer="1"/>
+</signal>
 </signals>

Commit message: up
Parts:
- added C1, C3: 0.1uf, rcl:C0805
- added C2: 10uf, rcl:C0805
- added SJ1: SPI 3wire, jumper:SJ
- added U1, U2: BMX160, BMX160:PQFN50P250X300X100-14N
Connections:
- new net N$7: SJ1.1, SV3.6, U1.14, U2.14
- new net N$8: SV1.2, U1.9
- new net N$9: SV1.1, U1.4
- net +3V3: now also C1.1, C2.1, C3.1, U1.5, U1.8, U2.5, U2.8
- net CS_AG: now also U1.12
- net CS_M: now also U2.12
- net GND: now also C1.2, C2.2, C3.2, U1.2, U1.3, U1.6, U1.7, U2.2, U2.3, U2.6, U2.7
- net SDIO: now also SJ1.2, U1.1, U2.1; no longer SV3.6
- net SLC: now also U1.13, U2.13
Routing:
- net SDIO: track 30.9 -> 93.4 mm, vias 0 -> 2
- net N$7: track 0.00 -> 59.4 mm, vias 0 -> 2
- net SLC: track 28.3 -> 65.4 mm, vias 0 -> 3
- net CS_M: track 30.8 -> 63.3 mm
- net CS_AG: track 24.8 -> 56.8 mm
- net N$9: track 0.00 -> 31.0 mm
- net +3V3: track 108.7 -> 136.6 mm, vias 0 -> 2
- net N$8: track 0.00 -> 23.9 mm
- net GND: track 152.3 -> 175.8 mm, vias 0 -> 2
- net N$3: track 45.6 -> 50.9 mm
- net N$5: track 40.8 -> 44.1 mm
- net N$2: track 52.0 -> 52.6 mm
- added copper zone on layer 16, net GND
