File: imu/pic32mk/imu.sch (EAGLE design)
At the start: 6 parts

Commit message: up
Parts:
- added SV7: J601, con-lstb:MA17-2W
- added SV8: LCD, con-lstb:MA10-1
Connections:
- new net N$1: SV7.2, SV8.3
- new net N$3: SV7.12, SV8.2
- new net N$4: SV7.13, SV8.5
- new net N$5: SV7.14, SV8.4
- new net N$6: SV7.16, SV8.6
- net +3V3: now also SV8.7
- net GND: now also SV8.8
Changed lines of the file:
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@@
 <part name="SV6" library="con-lstb" library_urn="urn:adsk.eagle:library:162" deviceset="MA04-1" device="" package3d_urn="urn:adsk.eagle:package:8337/1" value="DPINS"/>
 <part name="GND2" library="supply1" library_urn="urn:adsk.eagle:library:371" deviceset="GND" device=""/>
+<part name="SV7" library="con-lstb" library_urn="urn:adsk.eagle:library:162" deviceset="MA17-2W" device="" package3d_urn="urn:adsk.eagle:package:8356/1" value="J601"/>
+<part name="SV8" library="con-lstb" library_urn="urn:adsk.eagle:library:162" deviceset="MA10-1" device="" package3d_urn="urn:adsk.eagle:package:8346/1" value="LCD"/>
+<part name="GND3" library="supply1" library_urn="urn:adsk.eagle:library:371" deviceset="GND" device=""/>
+<part name="+3V2" library="supply1" library_urn="urn:adsk.eagle:library:371" deviceset="+3V3" device=""/>
 </parts>
 <sheets>
@@
 <instance part="GND2" gate="1" x="20.32" y="15.24" smashed="yes">
 <attribute name="VALUE" x="17.78" y="12.7" size="1.778" layer="96"/>
+</instance>
+<instance part="SV7" gate="1" x="154.94" y="27.94" smashed="yes">
+<attribute name="VALUE" x="151.13" y="2.54" size="1.778" layer="96"/>
+<attribute name="NAME" x="151.13" y="51.562" size="1.778" layer="95"/>
+</instance>
+<instance part="SV8" gate="1" x="127" y="-7.62" smashed="yes">
+<attribute name="VALUE" x="125.73" y="-22.86" size="1.778" layer="96"/>
+<attribute name="NAME" x="125.73" y="8.382" size="1.778" layer="95"/>
+</instance>
+<instance part="GND3" gate="1" x="167.64" y="-2.54" smashed="yes">
+<attribute name="VALUE" x="165.1" y="-5.08" size="1.778" layer="96"/>
+</instance>
+<instance part="+3V2" gate="G$1" x="162.56" y="-5.08" smashed="yes" rot="R180">
+<attribute name="VALUE" x="165.1" y="0" size="1.778" layer="96" rot="R270"/>
 </instance>
 </instances>
@@
 <junction x="20.32" y="17.78"/>
 </segment>
+<segment>
+<pinref part="SV8" gate="1" pin="8"/>
+<wire x1="134.62" y1="0" x2="167.64" y2="0" width="0.1524" layer="91"/>
+<pinref part="GND3" gate="1" pin="GND"/>
+<junction x="134.62" y="0"/>
+<junction x="167.64" y="0"/>
+</segment>
 </net>
 <net name="+3V3" class="0">
@@
 <junction x="48.26" y="10.16"/>
 <junction x="111.76" y="30.48"/>
+</segment>
+<segment>
+<pinref part="SV8" gate="1" pin="7"/>
+<wire x1="134.62" y1="-2.54" x2="162.56" y2="-2.54" width="0.1524" layer="91"/>
+<pinref part="+3V2" gate="G$1" pin="+3V3"/>
+<junction x="134.62" y="-2.54"/>
+<junction x="162.56" y="-2.54"/>
 </segment>
 </net>
@@
 </segment>
 </net>
+<net name="N$1" class="0">
+<segment>
+<pinref part="SV8" gate="1" pin="3"/>
+<wire x1="134.62" y1="-12.7" x2="144.78" y2="-12.7" width="0.1524" layer="91"/>
+<wire x1="144.78" y1="-12.7" x2="144.78" y2="7.62" width="0.1524" layer="91"/>
+<pinref part="SV7" gate="1" pin="2"/>
+<wire x1="144.78" y1="7.62" x2="147.32" y2="7.62" width="0.1524" layer="91"/>
+<junction x="134.62" y="-12.7"/>
+<junction x="147.32" y="7.62"/>
+</segment>
+</net>
+<net name="N$3" class="0">
+<segment>
+<pinref part="SV8" gate="1" pin="2"/>
+<wire x1="134.62" y1="-15.24" x2="142.24" y2="-15.24" width="0.1524" layer="91"/>
+<wire x1="142.24" y1="-15.24" x2="142.24" y2="20.32" width="0.1524" layer="91"/>
+<pinref part="SV7" gate="1" pin="12"/>
+<wire x1="142.24" y1="20.32" x2="147.32" y2="20.32" width="0.1524" layer="91"/>
+<junction x="134.62" y="-15.24"/>
+<junction x="147.32" y="20.32"/>
+</segment>
+</net>
+<net name="N$4" class="0">
+<segment>
+<pinref part="SV8" gate="1" pin="5"/>
+<wire x1="134.62" y1="-7.62" x2="172.72" y2="-7.62" width="0.1524" layer="91"/>
+<wire x1="172.72" y1="-7.62" x2="172.72" y2="22.86" width="0.1524" layer="91"/>
+<pinref part="SV7" gate="1" pin="13"/>
+<wire x1="172.72" y1="22.86" x2="162.56" y2="22.86" width="0.1524" layer="91"/>
+<junction x="134.62" y="-7.62"/>
+<junction x="162.56" y="22.86"/>
+</segment>
+</net>
+<net name="N$5" class="0">
+<segment>
+<pinref part="SV8" gate="1" pin="4"/>
+<wire x1="134.62" y1="-10.16" x2="139.7" y2="-10.16" width="0.1524" layer="91"/>
+<pinref part="SV7" gate="1" pin="14"/>
+<wire x1="139.7" y1="-10.16" x2="139.7" y2="22.86" width="0.1524" layer="91"/>
+<wire x1="139.7" y1="22.86" x2="147.32" y2="22.86" width="0.1524" layer="91"/>
+<junction x="134.62" y="-10.16"/>
+<junction x="147.32" y="22.86"/>
+</segment>
+</net>
+<net name="N$6" class="0">
+<segment>
+<pinref part="SV8" gate="1" pin="6"/>
+<wire x1="134.62" y1="-5.08" x2="137.16" y2="-5.08" width="0.1524" layer="91"/>
+<wire x1="137.16" y1="-5.08" x2="137.16" y2="25.4" width="0.1524" layer="91"/>
+<pinref part="SV7" gate="1" pin="16"/>
+<wire x1="137.16" y1="25.4" x2="147.32" y2="25.4" width="0.1524" layer="91"/>
+<junction x="134.62" y="-5.08"/>
+<junction x="147.32" y="25.4"/>
+</segment>
+</net>

Commit message: up
Parts:
- added C1, C3: 0.1uf, rcl:C-USC0805
- added C2: 10uf, rcl:C-USC0805
- added SJ1: SPI 3wire, jumper:SJ
- added U1, U2: BMX160, BMX160:BMX160
Connections:
- new net N$7: SJ1.1, SV3.6, U1.SDX, U2.SDX
- new net N$8: SV1.2, U1.INT2
- new net N$9: SV1.1, U1.INT1
- net +3V3: now also C1.1, C2.1, C3.1, U1.VDD, U1.VDDIO, U2.VDD, U2.VDDIO
- net CS_AG: now also U1.CSB
- net CS_M: now also U2.CSB
- net GND: now also C1.2, C2.2, C3.2, U1.GND, U1.GNDIO, U2.GND, U2.GNDIO
- net SDIO: now also SJ1.2, U1.SDO, U2.SDO; no longer SV3.6
- net SLC: now also U1.SCX, U2.SCX
